Commit message: [gazebo] tweaked params to grasp the fragment in gazebo

File: repair_urdf/urdf/fragment_stance.urdf (robot description, URDF)
Before this commit: robot fragment_stance, 1 links, 0 joints
Links:
- link fragment_stance: geometry collision box size=0.035 0.035 0.05; visual box size=0.035 0.035 0.05
