Commit message: original state of the softhand_intergration branch

File: repair_urdf/urdf/repair_full.urdf (robot description, URDF)
Before this commit: robot repair_full, 39 links, 38 joints
Links:
- removed link arm_1_tcp
- removed link arm_2_tcp
- added link left_hand_v1s_index_distal_link, mass 0.1; collision mesh filename=package://softhands_description/meshes/softhands/v1.0/commo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; visual mesh filename=package://softhands_description/meshes/softhands/v1.0/commo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
- added link left_hand_v1s_index_knuckle_link, mass 0.09; collision mesh filename=package://softhands_description/meshes/softhands/v1.0/commo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; visual mesh filename=package://softhands_description/meshes/softhands/v1.0/commo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
- added link left_hand_v1s_index_middle_link, mass 0.05; collision mesh filename=package://softhands_description/meshes/softhands/v1.0/commo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; visual mesh filename=package://softhands_description/meshes/softhands/v1.0/commo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
- added link left_hand_v1s_index_proximal_link, mass 0.05; collision mesh filename=package://softhands_description/meshes/softhands/v1.0/commo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; visual mesh filename=package://softhands_description/meshes/softhands/v1.0/commo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
- added link left_hand_v1s_little_distal_link, mass 0.1; collision mesh filename=package://softhands_description/meshes/softhands/v1.0/commo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; visual mesh filename=package://softhands_description/meshes/softhands/v1.0/commo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
- added link left_hand_v1s_little_knuckle_link, mass 0.09; collision mesh filename=package://softhands_description/meshes/softhands/v1.0/commo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; visual mesh filename=package://softhands_description/meshes/softhands/v1.0/commo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
- added link left_hand_v1s_little_middle_link, mass 0.05; collision mesh filename=package://softhands_description/meshes/softhands/v1.0/commo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; visual mesh filename=package://softhands_description/meshes/softhands/v1.0/commo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
- added link left_hand_v1s_little_proximal_link, mass 0.05; collision mesh filename=package://softhands_description/meshes/softhands/v1.0/commo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; visual mesh filename=package://softhands_description/meshes/softhands/v1.0/commo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
- added link left_hand_v1s_middle_distal_link, mass 0.1; collision mesh filename=package://softhands_description/meshes/softhands/v1.0/commo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; visual mesh filename=package://softhands_description/meshes/softhands/v1.0/commo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
- added link left_hand_v1s_middle_knuckle_link, mass 0.09; collision mesh filename=package://softhands_description/meshes/softhands/v1.0/commo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; visual mesh filename=package://softhands_description/meshes/softhands/v1.0/commo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
- added link left_hand_v1s_middle_middle_link, mass 0.05; collision mesh filename=package://softhands_description/meshes/softhands/v1.0/commo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; visual mesh filename=package://softhands_description/meshes/softhands/v1.0/commo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
- added link left_hand_v1s_middle_proximal_link, mass 0.05; collision mesh filename=package://softhands_description/meshes/softhands/v1.0/commo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; visual mesh filename=package://softhands_description/meshes/softhands/v1.0/commo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
- added link left_hand_v1s_palm_base
- added link left_hand_v1s_palm_link, mass 2.28; collision mesh filename=package://softhands_description/meshes/softhands/v1.0/left/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; collision mesh filename=package://softhands_description/meshes/softhands/v1.0/right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
- added link left_hand_v1s_ring_distal_link, mass 0.1; collision mesh filename=package://softhands_description/meshes/softhands/v1.0/commo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; visual mesh filename=package://softhands_description/meshes/softhands/v1.0/commo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
- added link left_hand_v1s_ring_knuckle_link, mass 0.09; collision mesh filename=package://softhands_description/meshes/softhands/v1.0/commo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; visual mesh filename=package://softhands_description/meshes/softhands/v1.0/commo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
- added link left_hand_v1s_ring_middle_link, mass 0.05; collision mesh filename=package://softhands_description/meshes/softhands/v1.0/commo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; visual mesh filename=package://softhands_description/meshes/softhands/v1.0/commo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
- added link left_hand_v1s_ring_proximal_link, mass 0.05; collision mesh filename=package://softhands_description/meshes/softhands/v1.0/commo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; visual mesh filename=package://softhands_description/meshes/softhands/v1.0/commo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
- added link left_hand_v1s_thumb_distal_link, mass 0.1; collision mesh filename=package://softhands_description/meshes/softhands/v1.0/commo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; visual mesh filename=package://softhands_description/meshes/softhands/v1.0/commo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
- added link left_hand_v1s_thumb_knuckle_link, mass 0.09; collision mesh filename=package://softhands_description/meshes/softhands/v1.0/left/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; visual mesh filename=package://softhands_description/meshes/softhands/v1.0/left/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
- added link left_hand_v1s_thumb_proximal_link, mass 0.05; collision mesh filename=package://softhands_description/meshes/softhands/v1.0/commo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; visual mesh filename=package://softhands_description/meshes/softhands/v1.0/commo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
- added link right_hand_v1s_index_distal_link, mass 0.1; collision mesh filename=package://softhands_description/meshes/softhands/v1.0/commo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; visual mesh filename=package://softhands_description/meshes/softhands/v1.0/commo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
- added link right_hand_v1s_index_knuckle_link, mass 0.09; collision mesh filename=package://softhands_description/meshes/softhands/v1.0/commo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; visual mesh filename=package://softhands_description/meshes/softhands/v1.0/commo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
- added link right_hand_v1s_index_middle_link, mass 0.05; collision mesh filename=package://softhands_description/meshes/softhands/v1.0/commo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; visual mesh filename=package://softhands_description/meshes/softhands/v1.0/commo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
- added link right_hand_v1s_index_proximal_link, mass 0.05; collision mesh filename=package://softhands_description/meshes/softhands/v1.0/commo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; visual mesh filename=package://softhands_description/meshes/softhands/v1.0/commo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
- added link right_hand_v1s_little_distal_link, mass 0.1; collision mesh filename=package://softhands_description/meshes/softhands/v1.0/commo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; visual mesh filename=package://softhands_description/meshes/softhands/v1.0/commo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
- added link right_hand_v1s_little_knuckle_link, mass 0.09; collision mesh filename=package://softhands_description/meshes/softhands/v1.0/commo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; visual mesh filename=package://softhands_description/meshes/softhands/v1.0/commo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
- added link right_hand_v1s_little_middle_link, mass 0.05; collision mesh filename=package://softhands_description/meshes/softhands/v1.0/commo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; visual mesh filename=package://softhands_description/meshes/softhands/v1.0/commo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
- added link right_hand_v1s_little_proximal_link, mass 0.05; collision mesh filename=package://softhands_description/meshes/softhands/v1.0/commo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; visual mesh filename=package://softhands_description/meshes/softhands/v1.0/commo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
- added link right_hand_v1s_middle_distal_link, mass 0.1; collision mesh filename=package://softhands_description/meshes/softhands/v1.0/commo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; visual mesh filename=package://softhands_description/meshes/softhands/v1.0/commo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
- added link right_hand_v1s_middle_knuckle_link, mass 0.09; collision mesh filename=package://softhands_description/meshes/softhands/v1.0/commo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; visual mesh filename=package://softhands_description/meshes/softhands/v1.0/commo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
- added link right_hand_v1s_middle_middle_link, mass 0.05; collision mesh filename=package://softhands_description/meshes/softhands/v1.0/commo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; visual mesh filename=package://softhands_description/meshes/softhands/v1.0/commo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
- added link right_hand_v1s_middle_proximal_link, mass 0.05; collision mesh filename=package://softhands_description/meshes/softhands/v1.0/commo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; visual mesh filename=package://softhands_description/meshes/softhands/v1.0/commo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
- added link right_hand_v1s_palm_base
- added link right_hand_v1s_palm_link, mass 2.28; collision mesh filename=package://softhands_description/meshes/softhands/v1.0/right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; collision mesh filename=package://softhands_description/meshes/softhands/v1.0/right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
- added link right_hand_v1s_ring_distal_link, mass 0.1; collision mesh filename=package://softhands_description/meshes/softhands/v1.0/commo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; visual mesh filename=package://softhands_description/meshes/softhands/v1.0/commo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
- added link right_hand_v1s_ring_knuckle_link, mass 0.09; collision mesh filename=package://softhands_description/meshes/softhands/v1.0/commo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; visual mesh filename=package://softhands_description/meshes/softhands/v1.0/commo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
- added link right_hand_v1s_ring_middle_link, mass 0.05; collision mesh filename=package://softhands_description/meshes/softhands/v1.0/commo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; visual mesh filename=package://softhands_description/meshes/softhands/v1.0/commo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
- added link right_hand_v1s_ring_proximal_link, mass 0.05; collision mesh filename=package://softhands_description/meshes/softhands/v1.0/commo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; visual mesh filename=package://softhands_description/meshes/softhands/v1.0/commo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
- added link right_hand_v1s_thumb_distal_link, mass 0.1; collision mesh filename=package://softhands_description/meshes/softhands/v1.0/commo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; visual mesh filename=package://softhands_description/meshes/softhands/v1.0/commo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
- added link right_hand_v1s_thumb_knuckle_link, mass 0.09; collision mesh filename=package://softhands_description/meshes/softhands/v1.0/right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; visual mesh filename=package://softhands_description/meshes/softhands/v1.0/right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
- added link right_hand_v1s_thumb_proximal_link, mass 0.05; collision mesh filename=package://softhands_description/meshes/softhands/v1.0/commo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; visual mesh filename=package://softhands_description/meshes/softhands/v1.0/commo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
- link leg1_link: mass 0.1 -> None
- link leg2_link: mass 0.1 -> None
- link leg3_link: mass 0.1 -> None
- link leg4_link: mass 0.1 -> None
- link obar1_link: mass 0.1 -> None
- link obar2_link: mass 0.1 -> None
- link obar3_link: mass 0.1 -> None
- link obar4_link: mass 0.1 -> None
- link sliding_guide_link: mass 0.1 -> None
- link table_top_link: mass 0.1 -> None
- link vbar1_link: mass 0.1 -> None
- link vbar2_link: mass 0.1 -> None
- link vbar3_link: mass 0.1 -> None
- link vbar4_link: mass 0.1 -> None
Joints:
- removed joint arm_1_tcp_joint
- removed joint arm_2_tcp_joint
- added joint left_hand_base_joint: type fixed, parent arm_2_link_7, child left_hand_v1s_palm_base, origin xyz=0 -0.013900 -0.015 rpy=0 0 0
- added joint left_hand_v1s_index_distal_joint: type revolute, parent left_hand_v1s_index_middle_link, child left_hand_v1s_index_distal_link, origin xyz=0.020 0 0 rpy=0 0 0, axis 0 -1 0, limit lower=-1.57 upper=1.57 effort=30 velocity=1.0
- added joint left_hand_v1s_index_knuckle_joint: type revolute, parent left_hand_v1s_palm_link, child left_hand_v1s_index_knuckle_link, origin xyz=-0.0033 -0.0195 0.0936994 rpy=-1.5707963267948966 -1.4835299330931884 -1.5707963267948966, axis 0 0 -1, limit lower=-1.57 upper=1.57 effort=30 velocity=1.0
- added joint left_hand_v1s_index_middle_joint: type revolute, parent left_hand_v1s_index_proximal_link, child left_hand_v1s_index_middle_link, origin xyz=0.020 0 0 rpy=0 0 0, axis 0 -1 0, limit lower=-1.57 upper=1.57 effort=30 velocity=1.0
- added joint left_hand_v1s_index_proximal_joint: type revolute, parent left_hand_v1s_index_knuckle_link, child left_hand_v1s_index_proximal_link, origin xyz=0.020 0 0 rpy=0 0 0, axis 0 -1 0, limit lower=-1.57 upper=1.57 effort=30 velocity=1.0
- added joint left_hand_v1s_little_distal_joint: type revolute, parent left_hand_v1s_little_middle_link, child left_hand_v1s_little_distal_link, origin xyz=0.020 0 0 rpy=0 0 0, axis 0 -1 0, limit lower=-1.57 upper=1.57 effort=30 velocity=1.0
- added joint left_hand_v1s_little_knuckle_joint: type revolute, parent left_hand_v1s_palm_link, child left_hand_v1s_little_knuckle_link, origin xyz=-0.0033 0.039 0.0836994 rpy=1.5707963267948966 -1.4835299330931884 1.5707963267948966, axis 0 0 -1, limit lower=-1.57 upper=1.57 effort=30 velocity=1.0
- added joint left_hand_v1s_little_middle_joint: type revolute, parent left_hand_v1s_little_proximal_link, child left_hand_v1s_little_middle_link, origin xyz=0.020 0 0 rpy=0 0 0, axis 0 -1 0, limit lower=-1.57 upper=1.57 effort=30 velocity=1.0
- added joint left_hand_v1s_little_proximal_joint: type revolute, parent left_hand_v1s_little_knuckle_link, child left_hand_v1s_little_proximal_link, origin xyz=0.020 0 0 rpy=0 0 0, axis 0 -1 0, limit lower=-1.57 upper=1.57 effort=30 velocity=1.0
- added joint left_hand_v1s_middle_distal_joint: type revolute, parent left_hand_v1s_middle_middle_link, child left_hand_v1s_middle_distal_link, origin xyz=0.020 0 0 rpy=0 0 0, axis 0 -1 0, limit lower=-1.57 upper=1.57 effort=30 velocity=1.0
- added joint left_hand_v1s_middle_knuckle_joint: type revolute, parent left_hand_v1s_palm_link, child left_hand_v1s_middle_knuckle_link, origin xyz=-0.0033 0.0 0.100699 rpy=3.1415 -1.5707963267948966 0.0, axis 0 0 -1, limit lower=-1.57 upper=1.57 effort=30 velocity=1.0
- added joint left_hand_v1s_middle_middle_joint: type revolute, parent left_hand_v1s_middle_proximal_link, child left_hand_v1s_middle_middle_link, origin xyz=0.020 0 0 rpy=0 0 0, axis 0 -1 0, limit lower=-1.57 upper=1.57 effort=30 velocity=1.0
- added joint left_hand_v1s_middle_proximal_joint: type revolute, parent left_hand_v1s_middle_knuckle_link, child left_hand_v1s_middle_proximal_link, origin xyz=0.020 0 0 rpy=0 0 0, axis 0 -1 0, limit lower=-1.57 upper=1.57 effort=30 velocity=1.0
- added joint left_hand_v1s_palm_joint: type fixed, parent left_hand_v1s_palm_base, child left_hand_v1s_palm_link, origin xyz=0.002 0.00695 0.0535 rpy=0 0 0
- added joint left_hand_v1s_ring_distal_joint: type revolute, parent left_hand_v1s_ring_middle_link, child left_hand_v1s_ring_distal_link, origin xyz=0.020 0 0 rpy=0 0 0, axis 0 -1 0, limit lower=-1.57 upper=1.57 effort=30 velocity=1.0
- added joint left_hand_v1s_ring_knuckle_joint: type revolute, parent left_hand_v1s_palm_link, child left_hand_v1s_ring_knuckle_link, origin xyz=-0.0033 0.0195 0.0936994 rpy=1.5707963267948966 -1.5184364298870514 1.5707963267948966, axis 0 0 -1, limit lower=-1.57 upper=1.57 effort=30 velocity=1.0
- added joint left_hand_v1s_ring_middle_joint: type revolute, parent left_hand_v1s_ring_proximal_link, child left_hand_v1s_ring_middle_link, origin xyz=0.020 0 0 rpy=0 0 0, axis 0 -1 0, limit lower=-1.57 upper=1.57 effort=30 velocity=1.0
- added joint left_hand_v1s_ring_proximal_joint: type revolute, parent left_hand_v1s_ring_knuckle_link, child left_hand_v1s_ring_proximal_link, origin xyz=0.020 0 0 rpy=0 0 0, axis 0 -1 0, limit lower=-1.57 upper=1.57 effort=30 velocity=1.0
- added joint left_hand_v1s_thumb_distal_joint: type continuous, parent left_hand_v1s_thumb_proximal_link, child left_hand_v1s_thumb_distal_link, origin xyz=0.020 0 0.0 rpy=0 0 0, axis 0 -1 0
- added joint left_hand_v1s_thumb_knuckle_joint: type continuous, parent left_hand_v1s_palm_link, child left_hand_v1s_thumb_knuckle_link, origin xyz=0.005669722 -0.029616 0.055314 rpy=0.0 -0.38397275793662144 -1.5707963267948966, axis 0 0 1
- added joint left_hand_v1s_thumb_proximal_joint: type continuous, parent left_hand_v1s_thumb_knuckle_link, child left_hand_v1s_thumb_proximal_link, origin xyz=0.033500000 0.0033 0.0 rpy=-0.426627741408745 0 0.0, axis 0 -1 0
- added joint right_hand_base_joint: type fixed, parent arm_1_link_7, child right_hand_v1s_palm_base, origin xyz=0 0 -0.015 rpy=0 0.0 3.14159265359
- added joint right_hand_v1s_index_distal_joint: type revolute, parent right_hand_v1s_index_middle_link, child right_hand_v1s_index_distal_link, origin xyz=0.020 0 0 rpy=0 0 0, axis 0 -1 0, limit lower=-1.57 upper=1.57 effort=30 velocity=1.0
- added joint right_hand_v1s_index_knuckle_joint: type revolute, parent right_hand_v1s_palm_link, child right_hand_v1s_index_knuckle_link, origin xyz=-0.0033 0.0195 0.0936994 rpy=1.5707963267948966 -1.4835299330931884 1.5707963267948966, axis 0 0 1, limit lower=-1.57 upper=1.57 effort=30 velocity=1.0
- added joint right_hand_v1s_index_middle_joint: type revolute, parent right_hand_v1s_index_proximal_link, child right_hand_v1s_index_middle_link, origin xyz=0.020 0 0 rpy=0 0 0, axis 0 -1 0, limit lower=-1.57 upper=1.57 effort=30 velocity=1.0
- added joint right_hand_v1s_index_proximal_joint: type revolute, parent right_hand_v1s_index_knuckle_link, child right_hand_v1s_index_proximal_link, origin xyz=0.020 0 0 rpy=0 0 0, axis 0 -1 0, limit lower=-1.57 upper=1.57 effort=30 velocity=1.0
- added joint right_hand_v1s_little_distal_joint: type revolute, parent right_hand_v1s_little_middle_link, child right_hand_v1s_little_distal_link, origin xyz=0.020 0 0 rpy=0 0 0, axis 0 -1 0, limit lower=-1.57 upper=1.57 effort=30 velocity=1.0
- added joint right_hand_v1s_little_knuckle_joint: type revolute, parent right_hand_v1s_palm_link, child right_hand_v1s_little_knuckle_link, origin xyz=-0.0033 -0.039 0.0836994 rpy=-1.5707963267948966 -1.4835299330931884 -1.5707963267948966, axis 0 0 1, limit lower=-1.57 upper=1.57 effort=30 velocity=1.0
- added joint right_hand_v1s_little_middle_joint: type revolute, parent right_hand_v1s_little_proximal_link, child right_hand_v1s_little_middle_link, origin xyz=0.020 0 0 rpy=0 0 0, axis 0 -1 0, limit lower=-1.57 upper=1.57 effort=30 velocity=1.0
- added joint right_hand_v1s_little_proximal_joint: type revolute, parent right_hand_v1s_little_knuckle_link, child right_hand_v1s_little_proximal_link, origin xyz=0.020 0 0 rpy=0 0 0, axis 0 -1 0, limit lower=-1.57 upper=1.57 effort=30 velocity=1.0
- added joint right_hand_v1s_middle_distal_joint: type revolute, parent right_hand_v1s_middle_middle_link, child right_hand_v1s_middle_distal_link, origin xyz=0.020 0 0 rpy=0 0 0, axis 0 -1 0, limit lower=-1.57 upper=1.57 effort=30 velocity=1.0
- added joint right_hand_v1s_middle_knuckle_joint: type revolute, parent right_hand_v1s_palm_link, child right_hand_v1s_middle_knuckle_link, origin xyz=-0.003300000 0.0 0.100699 rpy=3.141592 -1.5707963267948966 0.0, axis 0 0 1, limit lower=-1.57 upper=1.57 effort=30 velocity=1.0
- added joint right_hand_v1s_middle_middle_joint: type revolute, parent right_hand_v1s_middle_proximal_link, child right_hand_v1s_middle_middle_link, origin xyz=0.020 0 0 rpy=0 0 0, axis 0 -1 0, limit lower=-1.57 upper=1.57 effort=30 velocity=1.0
- added joint right_hand_v1s_middle_proximal_joint: type revolute, parent right_hand_v1s_middle_knuckle_link, child right_hand_v1s_middle_proximal_link, origin xyz=0.020 0 0 rpy=0 0 0, axis 0 -1 0, limit lower=-1.57 upper=1.57 effort=30 velocity=1.0
- added joint right_hand_v1s_palm_joint: type fixed, parent right_hand_v1s_palm_base, child right_hand_v1s_palm_link, origin xyz=0.002 0.00695 0.0535 rpy=0 0 0
- added joint right_hand_v1s_ring_distal_joint: type revolute, parent right_hand_v1s_ring_middle_link, child right_hand_v1s_ring_distal_link, origin xyz=0.020 0 0 rpy=0 0 0, axis 0 -1 0, limit lower=-1.57 upper=1.57 effort=30 velocity=1.0
- added joint right_hand_v1s_ring_knuckle_joint: type revolute, parent right_hand_v1s_palm_link, child right_hand_v1s_ring_knuckle_link, origin xyz=-0.0033 -0.0195 0.0936994 rpy=-1.5707963267948966 -1.5184364298870514 -1.5707963267948966, axis 0 0 1, limit lower=-1.57 upper=1.57 effort=30 velocity=1.0
- added joint right_hand_v1s_ring_middle_joint: type revolute, parent right_hand_v1s_ring_proximal_link, child right_hand_v1s_ring_middle_link, origin xyz=0.020 0 0 rpy=0 0 0, axis 0 -1 0, limit lower=-1.57 upper=1.57 effort=30 velocity=1.0
- added joint right_hand_v1s_ring_proximal_joint: type revolute, parent right_hand_v1s_ring_knuckle_link, child right_hand_v1s_ring_proximal_link, origin xyz=0.020 0 0 rpy=0 0 0, axis 0 -1 0, limit lower=-1.57 upper=1.57 effort=30 velocity=1.0
- added joint right_hand_v1s_thumb_distal_joint: type continuous, parent right_hand_v1s_thumb_proximal_link, child right_hand_v1s_thumb_distal_link, origin xyz=0.020 0 0.0 rpy=0 0 0, axis 0 -1 0
- added joint right_hand_v1s_thumb_knuckle_joint: type continuous, parent right_hand_v1s_palm_link, child right_hand_v1s_thumb_knuckle_link, origin xyz=0.00566972 0.0296160 0.0553140 rpy=0.0 -0.38397275793662144 1.5707963267948966, axis 0 0 -1
- added joint right_hand_v1s_thumb_proximal_joint: type continuous, parent right_hand_v1s_thumb_knuckle_link, child right_hand_v1s_thumb_proximal_link, origin xyz=0.033500000 -0.0033 0.0 rpy=0.426627741408745 0 0.0, axis 0 -1 0
- joint arm_1_joint_7: origin xyz=0.18 0 0 rpy=1.57079632679 0 1.57079632679 -> xyz=0.08 0 0 rpy=1.57079632679 0 1.57079632679
- joint arm_2_joint_7: origin xyz=0.18 0 0 rpy=-1.57079632679 3.14159265359 -1.57079632679 -> xyz=0.08 0 0 rpy=-1.57079632679 3.14159265359 -1.57079632679
