Commit message: original state of the softhand_intergration branch

File: repair_urdf/urdf/repair_full.urdf.xacro (robot description, xacro)
@@ -15,8 +15,13 @@
 <xacro:arg name="use_updated_wrist" default="false" />
 <xacro:arg name="gz_self_collide" default="true" />
+<xacro:arg name="xbot" default="true" />
+<xacro:arg name="fixed_hands" default="false" />
 <xacro:include filename="$(find repair_urdf)/urdf/repair_arm.urdf.xacro"/>
 <xacro:include filename="$(find repair_urdf)/urdf/repair_cage.urdf.xacro"/>
 <xacro:include filename="$(find repair_urdf)/urdf/repair_opt_mount_params.urdf.xacro"/>
 <xacro:include filename="$(find repair_urdf)/urdf/materials.gazebo.xacro"/>
+<xacro:if value="$(arg xbot)">
+    <xacro:include filename="$(find repair_urdf)/urdf/xbot2.gazebo.xacro"/>
+</xacro:if>
 <xacro:if value="$(arg load_sol)">
     <joint name="x_joint" type="prismatic">
@@ -27,14 +32,4 @@
         <limit lower="${- cage_depth/2 + x_joint_limit_margin}" upper= "${cage_depth/2 - x_joint_limit_margin}" effort="1000.0" velocity="20.0"/>
     </joint>
-    <transmission name="trans_x_joint">
-        <type>transmission_interface/SimpleTransmission</type>
-        <joint name="x_joint">
-            <hardwareInterface>hardware_interface/PositionJointInterface</hardwareInterface>
-        </joint>
-        <actuator name="x_joint_motor">
-            <hardwareInterface>hardware_interface/PositionJointInterface</hardwareInterface>
-            <mechanicalReduction>1</mechanicalReduction>
-        </actuator>
-    </transmission>
     <link name="base_link">
         <!-- torso inertias + stuff attached to the sliding guide -->
@@ -94,14 +89,4 @@
         <limit lower="${- cage_depth/2 + x_joint_limit_margin}" upper= "${cage_depth/2 - x_joint_limit_margin}" effort="1000.0" velocity="20.0"/>
     </joint>
-    <transmission name="trans_x_joint">
-        <type>transmission_interface/SimpleTransmission</type>
-        <joint name="x_joint">
-            <hardwareInterface>hardware_interface/PositionJointInterface</hardwareInterface>
-        </joint>
-        <actuator name="x_joint_motor">
-            <hardwareInterface>hardware_interface/PositionJointInterface</hardwareInterface>
-            <mechanicalReduction>1</mechanicalReduction>
-        </actuator>
-    </transmission>
     <link name="dummy_link">
     </link>
@@ -170,9 +155,9 @@
 </xacro:unless>
 <xacro:repair_arm base_link="r_arm_mount_frame" id="1" is_sliding_wrist="$(arg is_sliding_wrist)"
-gen_coll="$(arg gen_coll)" load_sol="$(arg load_sol)" use_updated_wrist = "$(arg use_updated_wrist)"
-gz_self_collide = "$(arg gz_self_collide)" />
+gen_coll="$(arg gen_coll)" load_sol="$(arg load_sol)" use_updated_wrist ="$(arg use_updated_wrist)"
+gz_self_collide ="$(arg gz_self_collide)" fixed_hands ="$(arg fixed_hands)" />
 <xacro:repair_arm base_link="l_arm_mount_frame" id="2" is_sliding_wrist="$(arg is_sliding_wrist)"
-gen_coll="$(arg gen_coll)" load_sol="$(arg load_sol)" use_updated_wrist = "$(arg use_updated_wrist)"
-gz_self_collide = "$(arg gz_self_collide)" />
+gen_coll="$(arg gen_coll)" load_sol="$(arg load_sol)" use_updated_wrist ="$(arg use_updated_wrist)"
+gz_self_collide ="$(arg gz_self_collide)" fixed_hands ="$(arg fixed_hands)" />
 <xacro:repair_arm_materials id="1" />
 <xacro:repair_arm_materials id="2" />

Commit message: added the movet_config package and added transmission to urdf

File: repair_urdf/urdf/repair_arm.urdf.xacro (robot description, xacro)
@@ -16,4 +16,6 @@
 <xacro:property name="sm_tau_max" value="200.0" />
 <xacro:include filename="$(find repair_urdf)/urdf/repair_arm_coll_params.urdf.xacro"/>
+<xacro:include filename="$(find repair_urdf)/urdf/repair.transmission.xacro" />
+<xacro:include filename="$(find repair_urdf)/urdf/common.gazebo.xacro" />
 <xacro:macro name="repair_arm" params="id base_link is_sliding_wrist gen_coll load_sol use_updated_wrist gz_self_collide fixed_hands" >
 <xacro:if value="${gen_coll == True}">
@@ -387,4 +389,5 @@
     </gazebo>
 </xacro:if>
+<xacro:repair_arm_transmission id="${id}" />
 </xacro:macro>
 </robot>

File: repair_urdf/urdf/repair_full.urdf.xacro (robot description, xacro)
@@ -32,4 +32,14 @@
         <limit lower="${- cage_depth/2 + x_joint_limit_margin}" upper= "${cage_depth/2 - x_joint_limit_margin}" effort="1000.0" velocity="20.0"/>
     </joint>
+    <transmission name="trans_x_joint">
+        <type>transmission_interface/SimpleTransmission</type>
+        <joint name="x_joint">
+            <hardwareInterface>hardware_interface/PositionJointInterface</hardwareInterface>
+        </joint>
+        <actuator name="x_joint_motor">
+            <hardwareInterface>hardware_interface/PositionJointInterface</hardwareInterface>
+            <mechanicalReduction>1</mechanicalReduction>
+        </actuator>
+    </transmission>
     <link name="base_link">
         <!-- torso inertias + stuff attached to the sliding guide -->
