Commit message: [hand] modified hand from v2s to v1s

File: repair_urdf/urdf/repair_arm.urdf.xacro (robot description, xacro)
@@ -349,7 +349,13 @@
     </inertial>
 </link>
+<gazebo reference="arm_${id}_link_7">
+    <kp value="1e4" />
+    <kd value="1e2" />
+    <mu1>0.2</mu1>
+	<mu2>0.2</mu2>
+</gazebo>
 <xacro:if value="${id == 1}">
     <xacro:softhands type="right"
-        version="v2.0_simple"
+        version="v1.0_simple"
         parent="arm_${id}_link_7"
         useMimicTag="true"
@@ -362,5 +368,5 @@
 <xacro:unless value="${id == 1}">
     <xacro:softhands type="left"
-        version="v2.0_simple"
+        version="v1.0_simple"
         parent="arm_${id}_link_7"
         useMimicTag="true"

File: repair_urdf/urdf/repair_hand_transmission.xacro (robot description, xacro)
@@ -3,200 +3,200 @@
   <xacro:macro name="repair_hand_transmission" params="id">
     <!-- synergy joint -->
-    <transmission name="trans_${id}_hand_v2s_synergy_joint">
-        <type>transmission_interface/SimpleTransmission</type>
-        <joint name="${id}_hand_v2s_synergy_joint">
+    <transmission name="trans_${id}_hand_v1s_synergy_joint">
+        <type>transmission_interface/SimpleTransmission</type>
+        <joint name="${id}_hand_v1s_synergy_joint">
             <hardwareInterface>hardware_interface/PositionJointInterface</hardwareInterface>
         </joint>
-        <actuator name="${id}_hand_v2s_synergy_joint_motor">
+        <actuator name="${id}_hand_v1s_synergy_joint_motor">
             <!-- <hardwareInterface>hardware_interface/PositionJointInterface</hardwareInterface> -->
             <mechanicalReduction>1</mechanicalReduction>
         </actuator>
     </transmission>
-    <!-- <transmission name="trans_${id}_hand_v2s_index_knuckle_joint">
-        <type>transmission_interface/SimpleTransmission</type>
-        <joint name="${id}_hand_v2s_index_knuckle_joint">
-            <hardwareInterface>hardware_interface/EffortJointInterface</hardwareInterface>
-        </joint>
-        <actuator name="${id}_hand_v2s_index_knuckle_joint_motor">
-            <hardwareInterface>hardware_interface/EffortJointInterface</hardwareInterface>
-            <mechanicalReduction>1</mechanicalReduction>
-        </actuator>
-    </transmission>
-    <transmission name="trans_${id}_hand_v2s_index_proximal_joint">
-        <type>transmission_interface/SimpleTransmission</type>
-        <joint name="${id}_hand_v2s_index_proximal_joint">
-            <hardwareInterface>hardware_interface/EffortJointInterface</hardwareInterface>
-        </joint>
-        <actuator name="${id}_hand_v2s_index_proximal_joint_motor">
-            <hardwareInterface>hardware_interface/EffortJointInterface</hardwareInterface>
-            <mechanicalReduction>1</mechanicalReduction>
-        </actuator>
-    </transmission>
-    <transmission name="trans_${id}_hand_v2s_index_middle_joint">
-        <type>transmission_interface/SimpleTransmission</type>
-        <joint name="${id}_hand_v2s_index_middle_joint">
-            <hardwareInterface>hardware_interface/EffortJointInterface</hardwareInterface>
-        </joint>
-        <actuator name="${id}_hand_v2s_index_middle_joint_motor">
-            <hardwareInterface>hardware_interface/EffortJointInterface</hardwareInterface>
-            <mechanicalReduction>1</mechanicalReduction>
-        </actuator>
-    </transmission>
-    <transmission name="trans_${id}_hand_v2s_index_distal_joint">
-        <type>transmission_interface/SimpleTransmission</type>
-        <joint name="${id}_hand_v2s_index_distal_joint">
-            <hardwareInterface>hardware_interface/EffortJointInterface</hardwareInterface>
-        </joint>
-        <actuator name="${id}_hand_v2s_index_distal_joint_motor">
-            <hardwareInterface>hardware_interface/EffortJointInterface</hardwareInterface>
-            <mechanicalReduction>1</mechanicalReduction>
-        </actuator>
-    </transmission>
-    <transmission name="trans_${id}_hand_v2s_middle_knuckle_joint">
-        <type>transmission_interface/SimpleTransmission</type>
-        <joint name="${id}_hand_v2s_middle_knuckle_joint">
-            <hardwareInterface>hardware_interface/EffortJointInterface</hardwareInterface>
-        </joint>
-        <actuator name="${id}_hand_v2s_middle_knuckle_joint_motor">
-            <hardwareInterface>hardware_interface/EffortJointInterface</hardwareInterface>
-            <mechanicalReduction>1</mechanicalReduction>
-        </actuator>
-    </transmission>
-    <transmission name="trans_${id}_hand_v2s_middle_proximal_joint">
-        <type>transmission_interface/SimpleTransmission</type>
-        <joint name="${id}_hand_v2s_middle_proximal_joint">
-            <hardwareInterface>hardware_interface/EffortJointInterface</hardwareInterface>
-        </joint>
-        <actuator name="${id}_hand_v2s_middle_proximal_joint_motor">
-            <hardwareInterface>hardware_interface/EffortJointInterface</hardwareInterface>
-            <mechanicalReduction>1</mechanicalReduction>
-        </actuator>
-    </transmission>
-    <transmission name="trans_${id}_hand_v2s_middle_middle_joint">
-        <type>transmission_interface/SimpleTransmission</type>
-        <joint name="${id}_hand_v2s_middle_middle_joint">
-            <hardwareInterface>hardware_interface/EffortJointInterface</hardwareInterface>
-        </joint>
-        <actuator name="${id}_hand_v2s_middle_middle_joint_motor">
-            <hardwareInterface>hardware_interface/EffortJointInterface</hardwareInterface>
-            <mechanicalReduction>1</mechanicalReduction>
-        </actuator>
-    </transmission>
-    <transmission name="trans_${id}_hand_v2s_middle_distal_joint">
-        <type>transmission_interface/SimpleTransmission</type>
-        <joint name="${id}_hand_v2s_middle_distal_joint">
-            <hardwareInterface>hardware_interface/EffortJointInterface</hardwareInterface>
-        </joint>
-        <actuator name="${id}_hand_v2s_middle_distal_joint_motor">
-            <hardwareInterface>hardware_interface/EffortJointInterface</hardwareInterface>
-            <mechanicalReduction>1</mechanicalReduction>
-        </actuator>
-    </transmission>
-    <transmission name="trans_${id}_hand_v2s_ring_knuckle_joint">
-        <type>transmission_interface/SimpleTransmission</type>
-        <joint name="${id}_hand_v2s_ring_knuckle_joint">
-            <hardwareInterface>hardware_interface/EffortJointInterface</hardwareInterface>
-        </joint>
-        <actuator name="${id}_hand_v2s_ring_knuckle_joint_motor">
-            <hardwareInterface>hardware_interface/EffortJointInterface</hardwareInterface>
-            <mechanicalReduction>1</mechanicalReduction>
-        </actuator>
-    </transmission>
-    <transmission name="trans_${id}_hand_v2s_ring_proximal_joint">
-        <type>transmission_interface/SimpleTransmission</type>
-        <joint name="${id}_hand_v2s_ring_proximal_joint">
-            <hardwareInterface>hardware_interface/EffortJointInterface</hardwareInterface>
-        </joint>
-        <actuator name="${id}_hand_v2s_ring_proximal_joint_motor">
-            <hardwareInterface>hardware_interface/EffortJointInterface</hardwareInterface>
-            <mechanicalReduction>1</mechanicalReduction>
-        </actuator>
-    </transmission>
-    <transmission name="trans_${id}_hand_v2s_ring_middle_joint">
-        <type>transmission_interface/SimpleTransmission</type>
-        <joint name="${id}_hand_v2s_ring_middle_joint">
-            <hardwareInterface>hardware_interface/EffortJointInterface</hardwareInterface>
-        </joint>
-        <actuator name="${id}_hand_v2s_ring_middle_joint_motor">
-            <hardwareInterface>hardware_interface/EffortJointInterface</hardwareInterface>
-            <mechanicalReduction>1</mechanicalReduction>
-        </actuator>
-    </transmission>
-    <transmission name="trans_${id}_hand_v2s_ring_distal_joint">
-        <type>transmission_interface/SimpleTransmission</type>
-        <joint name="${id}_hand_v2s_ring_distal_joint">
-            <hardwareInterface>hardware_interface/EffortJointInterface</hardwareInterface>
-        </joint>
-        <actuator name="${id}_hand_v2s_ring_distal_joint_motor">
-            <hardwareInterface>hardware_interface/EffortJointInterface</hardwareInterface>
-            <mechanicalReduction>1</mechanicalReduction>
-        </actuator>
-    </transmission>
-    <transmission name="trans_${id}_hand_v2s_little_knuckle_joint">
-        <type>transmission_interface/SimpleTransmission</type>
-        <joint name="${id}_hand_v2s_little_knuckle_joint">
-            <hardwareInterface>hardware_interface/EffortJointInterface</hardwareInterface>
-        </joint>
-        <actuator name="${id}_hand_v2s_little_knuckle_joint_motor">
-            <hardwareInterface>hardware_interface/EffortJointInterface</hardwareInterface>
-            <mechanicalReduction>1</mechanicalReduction>
-        </actuator>
-    </transmission>
-    <transmission name="trans_${id}_hand_v2s_little_proximal_joint">
-        <type>transmission_interface/SimpleTransmission</type>
-        <joint name="${id}_hand_v2s_little_proximal_joint">
-            <hardwareInterface>hardware_interface/EffortJointInterface</hardwareInterface>
-        </joint>
-        <actuator name="${id}_hand_v2s_little_proximal_joint_motor">
-            <hardwareInterface>hardware_interface/EffortJointInterface</hardwareInterface>
-            <mechanicalReduction>1</mechanicalReduction>
-        </actuator>
-    </transmission>
-    <transmission name="trans_${id}_hand_v2s_little_middle_joint">
-        <type>transmission_interface/SimpleTransmission</type>
-        <joint name="${id}_hand_v2s_little_middle_joint">
-            <hardwareInterface>hardware_interface/EffortJointInterface</hardwareInterface>
-        </joint>
-        <actuator name="${id}_hand_v2s_little_middle_joint_motor">
-            <hardwareInterface>hardware_interface/EffortJointInterface</hardwareInterface>
-            <mechanicalReduction>1</mechanicalReduction>
-        </actuator>
-    </transmission>
-    <transmission name="trans_${id}_hand_v2s_little_distal_joint">
-        <type>transmission_interface/SimpleTransmission</type>
-        <joint name="${id}_hand_v2s_little_distal_joint">
-            <hardwareInterface>hardware_interface/EffortJointInterface</hardwareInterface>
-        </joint>
-        <actuator name="${id}_hand_v2s_little_distal_joint_motor">
-            <hardwareInterface>hardware_interface/EffortJointInterface</hardwareInterface>
-            <mechanicalReduction>1</mechanicalReduction>
-        </actuator>
-    </transmission>
-    <transmission name="trans_${id}_hand_v2s_thumb_knuckle_joint">
-        <type>transmission_interface/SimpleTransmission</type>
-        <joint name="${id}_hand_v2s_thumb_knuckle_joint">
-            <hardwareInterface>hardware_interface/EffortJointInterface</hardwareInterface>
-        </joint>
-        <actuator name="${id}_hand_v2s_thumb_knuckle_joint_motor">
-            <hardwareInterface>hardware_interface/EffortJointInterface</hardwareInterface>
-            <mechanicalReduction>1</mechanicalReduction>
-        </actuator>
-    </transmission>
-    <transmission name="trans_${id}_hand_v2s_thumb_proximal_joint">
-        <type>transmission_interface/SimpleTransmission</type>
-        <joint name="${id}_hand_v2s_thumb_proximal_joint">
-            <hardwareInterface>hardware_interface/EffortJointInterface</hardwareInterface>
-        </joint>
-        <actuator name="${id}_hand_v2s_thumb_proximal_joint_motor">
-            <hardwareInterface>hardware_interface/EffortJointInterface</hardwareInterface>
-            <mechanicalReduction>1</mechanicalReduction>
-        </actuator>
-    </transmission>
-    <transmission name="trans_${id}_hand_v2s_thumb_distal_joint">
-        <type>transmission_interface/SimpleTransmission</type>
-        <joint name="${id}_hand_v2s_thumb_distal_joint">
-            <hardwareInterface>hardware_interface/EffortJointInterface</hardwareInterface>
-        </joint>
-        <actuator name="${id}_hand_v2s_thumb_distal_joint_motor">
+    <!-- <transmission name="trans_${id}_hand_v1s_index_knuckle_joint">
+        <type>transmission_interface/SimpleTransmission</type>
+        <joint name="${id}_hand_v1s_index_knuckle_joint">
+            <hardwareInterface>hardware_interface/EffortJointInterface</hardwareInterface>
+        </joint>
+        <actuator name="${id}_hand_v1s_index_knuckle_joint_motor">
+            <hardwareInterface>hardware_interface/EffortJointInterface</hardwareInterface>
+            <mechanicalReduction>1</mechanicalReduction>
+        </actuator>
+    </transmission>
+    <transmission name="trans_${id}_hand_v1s_index_proximal_joint">
+        <type>transmission_interface/SimpleTransmission</type>
+        <joint name="${id}_hand_v1s_index_proximal_joint">
+            <hardwareInterface>hardware_interface/EffortJointInterface</hardwareInterface>
+        </joint>
+        <actuator name="${id}_hand_v1s_index_proximal_joint_motor">
+            <hardwareInterface>hardware_interface/EffortJointInterface</hardwareInterface>
+            <mechanicalReduction>1</mechanicalReduction>
+        </actuator>
+    </transmission>
+    <transmission name="trans_${id}_hand_v1s_index_middle_joint">
+        <type>transmission_interface/SimpleTransmission</type>
+        <joint name="${id}_hand_v1s_index_middle_joint">
+            <hardwareInterface>hardware_interface/EffortJointInterface</hardwareInterface>
+        </joint>
+        <actuator name="${id}_hand_v1s_index_middle_joint_motor">
+            <hardwareInterface>hardware_interface/EffortJointInterface</hardwareInterface>
+            <mechanicalReduction>1</mechanicalReduction>
+        </actuator>
+    </transmission>
+    <transmission name="trans_${id}_hand_v1s_index_distal_joint">
+        <type>transmission_interface/SimpleTransmission</type>
+        <joint name="${id}_hand_v1s_index_distal_joint">
+            <hardwareInterface>hardware_interface/EffortJointInterface</hardwareInterface>
+        </joint>
+        <actuator name="${id}_hand_v1s_index_distal_joint_motor">
+            <hardwareInterface>hardware_interface/EffortJointInterface</hardwareInterface>
+            <mechanicalReduction>1</mechanicalReduction>
+        </actuator>
+    </transmission>
+    <transmission name="trans_${id}_hand_v1s_middle_knuckle_joint">
+        <type>transmission_interface/SimpleTransmission</type>
+        <joint name="${id}_hand_v1s_middle_knuckle_joint">
+            <hardwareInterface>hardware_interface/EffortJointInterface</hardwareInterface>
+        </joint>
+        <actuator name="${id}_hand_v1s_middle_knuckle_joint_motor">
+            <hardwareInterface>hardware_interface/EffortJointInterface</hardwareInterface>
+            <mechanicalReduction>1</mechanicalReduction>
+        </actuator>
+    </transmission>
+    <transmission name="trans_${id}_hand_v1s_middle_proximal_joint">
+        <type>transmission_interface/SimpleTransmission</type>
+        <joint name="${id}_hand_v1s_middle_proximal_joint">
+            <hardwareInterface>hardware_interface/EffortJointInterface</hardwareInterface>
+        </joint>
+        <actuator name="${id}_hand_v1s_middle_proximal_joint_motor">
+            <hardwareInterface>hardware_interface/EffortJointInterface</hardwareInterface>
+            <mechanicalReduction>1</mechanicalReduction>
+        </actuator>
+    </transmission>
+    <transmission name="trans_${id}_hand_v1s_middle_middle_joint">
+        <type>transmission_interface/SimpleTransmission</type>
+        <joint name="${id}_hand_v1s_middle_middle_joint">
+            <hardwareInterface>hardware_interface/EffortJointInterface</hardwareInterface>
+        </joint>
+        <actuator name="${id}_hand_v1s_middle_middle_joint_motor">
+            <hardwareInterface>hardware_interface/EffortJointInterface</hardwareInterface>
+            <mechanicalReduction>1</mechanicalReduction>
+        </actuator>
+    </transmission>
+    <transmission name="trans_${id}_hand_v1s_middle_distal_joint">
+        <type>transmission_interface/SimpleTransmission</type>
+        <joint name="${id}_hand_v1s_middle_distal_joint">
+            <hardwareInterface>hardware_interface/EffortJointInterface</hardwareInterface>
+        </joint>
+        <actuator name="${id}_hand_v1s_middle_distal_joint_motor">
+            <hardwareInterface>hardware_interface/EffortJointInterface</hardwareInterface>
+            <mechanicalReduction>1</mechanicalReduction>
+        </actuator>
+    </transmission>
+    <transmission name="trans_${id}_hand_v1s_ring_knuckle_joint">
+        <type>transmission_interface/SimpleTransmission</type>
+        <joint name="${id}_hand_v1s_ring_knuckle_joint">
+            <hardwareInterface>hardware_interface/EffortJointInterface</hardwareInterface>
+        </joint>
+        <actuator name="${id}_hand_v1s_ring_knuckle_joint_motor">
+            <hardwareInterface>hardware_interface/EffortJointInterface</hardwareInterface>
+            <mechanicalReduction>1</mechanicalReduction>
+        </actuator>
+    </transmission>
+    <transmission name="trans_${id}_hand_v1s_ring_proximal_joint">
+        <type>transmission_interface/SimpleTransmission</type>
+        <joint name="${id}_hand_v1s_ring_proximal_joint">
+            <hardwareInterface>hardware_interface/EffortJointInterface</hardwareInterface>
+        </joint>
+        <actuator name="${id}_hand_v1s_ring_proximal_joint_motor">
+            <hardwareInterface>hardware_interface/EffortJointInterface</hardwareInterface>
+            <mechanicalReduction>1</mechanicalReduction>
+        </actuator>
+    </transmission>
+    <transmission name="trans_${id}_hand_v1s_ring_middle_joint">
+        <type>transmission_interface/SimpleTransmission</type>
+        <joint name="${id}_hand_v1s_ring_middle_joint">
+            <hardwareInterface>hardware_interface/EffortJointInterface</hardwareInterface>
+        </joint>
+        <actuator name="${id}_hand_v1s_ring_middle_joint_motor">
+            <hardwareInterface>hardware_interface/EffortJointInterface</hardwareInterface>
+            <mechanicalReduction>1</mechanicalReduction>
+        </actuator>
+    </transmission>
+    <transmission name="trans_${id}_hand_v1s_ring_distal_joint">
+        <type>transmission_interface/SimpleTransmission</type>
+        <joint name="${id}_hand_v1s_ring_distal_joint">
+            <hardwareInterface>hardware_interface/EffortJointInterface</hardwareInterface>
+        </joint>
+        <actuator name="${id}_hand_v1s_ring_distal_joint_motor">
+            <hardwareInterface>hardware_interface/EffortJointInterface</hardwareInterface>
+            <mechanicalReduction>1</mechanicalReduction>
+        </actuator>
+    </transmission>
+    <transmission name="trans_${id}_hand_v1s_little_knuckle_joint">
+        <type>transmission_interface/SimpleTransmission</type>
+        <joint name="${id}_hand_v1s_little_knuckle_joint">
+            <hardwareInterface>hardware_interface/EffortJointInterface</hardwareInterface>
+        </joint>
+        <actuator name="${id}_hand_v1s_little_knuckle_joint_motor">
+            <hardwareInterface>hardware_interface/EffortJointInterface</hardwareInterface>
+            <mechanicalReduction>1</mechanicalReduction>
+        </actuator>
+    </transmission>
+    <transmission name="trans_${id}_hand_v1s_little_proximal_joint">
+        <type>transmission_interface/SimpleTransmission</type>
+        <joint name="${id}_hand_v1s_little_proximal_joint">
+            <hardwareInterface>hardware_interface/EffortJointInterface</hardwareInterface>
+        </joint>
+        <actuator name="${id}_hand_v1s_little_proximal_joint_motor">
+            <hardwareInterface>hardware_interface/EffortJointInterface</hardwareInterface>
+            <mechanicalReduction>1</mechanicalReduction>
+        </actuator>
+    </transmission>
+    <transmission name="trans_${id}_hand_v1s_little_middle_joint">
+        <type>transmission_interface/SimpleTransmission</type>
+        <joint name="${id}_hand_v1s_little_middle_joint">
+            <hardwareInterface>hardware_interface/EffortJointInterface</hardwareInterface>
+        </joint>
+        <actuator name="${id}_hand_v1s_little_middle_joint_motor">
+            <hardwareInterface>hardware_interface/EffortJointInterface</hardwareInterface>
+            <mechanicalReduction>1</mechanicalReduction>
+        </actuator>
+    </transmission>
+    <transmission name="trans_${id}_hand_v1s_little_distal_joint">
+        <type>transmission_interface/SimpleTransmission</type>
+        <joint name="${id}_hand_v1s_little_distal_joint">
+            <hardwareInterface>hardware_interface/EffortJointInterface</hardwareInterface>
+        </joint>
+        <actuator name="${id}_hand_v1s_little_distal_joint_motor">
+            <hardwareInterface>hardware_interface/EffortJointInterface</hardwareInterface>
+            <mechanicalReduction>1</mechanicalReduction>
+        </actuator>
+    </transmission>
+    <transmission name="trans_${id}_hand_v1s_thumb_knuckle_joint">
+        <type>transmission_interface/SimpleTransmission</type>
+        <joint name="${id}_hand_v1s_thumb_knuckle_joint">
+            <hardwareInterface>hardware_interface/EffortJointInterface</hardwareInterface>
+        </joint>
+        <actuator name="${id}_hand_v1s_thumb_knuckle_joint_motor">
+            <hardwareInterface>hardware_interface/EffortJointInterface</hardwareInterface>
+            <mechanicalReduction>1</mechanicalReduction>
+        </actuator>
+    </transmission>
+    <transmission name="trans_${id}_hand_v1s_thumb_proximal_joint">
+        <type>transmission_interface/SimpleTransmission</type>
+        <joint name="${id}_hand_v1s_thumb_proximal_joint">
+            <hardwareInterface>hardware_interface/EffortJointInterface</hardwareInterface>
+        </joint>
+        <actuator name="${id}_hand_v1s_thumb_proximal_joint_motor">
+            <hardwareInterface>hardware_interface/EffortJointInterface</hardwareInterface>
+            <mechanicalReduction>1</mechanicalReduction>
+        </actuator>
+    </transmission>
+    <transmission name="trans_${id}_hand_v1s_thumb_distal_joint">
+        <type>transmission_interface/SimpleTransmission</type>
+        <joint name="${id}_hand_v1s_thumb_distal_joint">
+            <hardwareInterface>hardware_interface/EffortJointInterface</hardwareInterface>
+        </joint>
+        <actuator name="${id}_hand_v1s_thumb_distal_joint_motor">
             <hardwareInterface>hardware_interface/EffortJointInterface</hardwareInterface>
             <mechanicalReduction>1</mechanicalReduction>
