Commit message: no longer spawn the fragments, added movegroup for both arms at once

File: repair_urdf/urdf/frag1.urdf (robot description, URDF)
Before this commit: robot frag1, 1 links, 0 joints
Links:
- link frag1: geometry collision mesh filename=package://repair_urdf/meshes/base_meshes/frag1_small.stl scale=0.01 0.01 0.01; visual mesh filename=package://repair_urdf/meshes/base_meshes/frag1_small.stl scale=0.01 0.01 0.01

Commit message: added fragment tf service

File: repair_urdf/urdf/frag1.urdf (robot description, URDF)
Before this commit: robot frag1, 1 links, 0 joints
Links:
- link frag1: geometry collision mesh filename=package://repair_urdf/meshes/base_meshes/frag1_small.stl; visual mesh filename=package://repair_urdf/meshes/base_meshes/frag1_small.stl

File: repair_urdf/urdf/frag2.urdf (robot description, URDF)
Before this commit: robot frag2, 1 links, 0 joints
Links:
- removed link frag2
- added link fragment_base_link, mass 0.05; collision mesh filename=package://repair_urdf/meshes/base_meshes/frag2_small.stl scale=2 2 2; visual mesh filename=package://repair_urdf/meshes/base_meshes/frag2_small.stl scale=2 2 2

Commit message: [softhand] reverted the mimic joint changes to softhand

File: repair_urdf/urdf/frag1.urdf (robot description, URDF)
Before this commit: robot frag1, 1 links, 0 joints
Links:
- link frag1: geometry collision mesh filename=package://repair_urdf/meshes/base_meshes/frag1_small.stl scale=0.01 0.01 0.01; visual mesh filename=package://repair_urdf/meshes/base_meshes/frag1_small.stl scale=0.01 0.01 0.01

File: repair_urdf/urdf/frag2.urdf (robot description, URDF)
Before this commit: robot frag2, 1 links, 0 joints
Links:
- removed link fragment_base_link
- added link frag2, mass 0.05; collision mesh filename=package://repair_urdf/meshes/base_meshes/frag2_small.stl; visual mesh filename=package://repair_urdf/meshes/base_meshes/frag2_small.stl

File: repair_urdf/urdf/repair_arm.urdf.xacro (robot description, xacro)
@@ -349,15 +349,8 @@
     </inertial>
 </link>
-<gazebo reference="arm_${id}_link_7">
-    <kp value="1e4" />
-    <kd value="1e2" />
-    <mu1>0.2</mu1>
-	<mu2>0.2</mu2>
-</gazebo>
 <xacro:if value="${id == 1}">
     <xacro:softhands type="right"
         version="v1.0_simple"
         parent="arm_${id}_link_7"
-        useMimicTag="true"
         position="0 0 -0.015"
         orientation="0 0.0 ${PI}"
@@ -370,5 +363,4 @@
         version="v1.0_simple"
         parent="arm_${id}_link_7"
-        useMimicTag="true"
         position="0 -0.013900 -0.015"
         orientation="0 0 0"
