Commit message: [softhand] reverted the mimic joint changes to softhand

File: repair_urdf/urdf/repair_hand_transmission.xacro (robot description, xacro)
@@ -2,16 +2,5 @@
 <robot xmlns:xacro="http://www.ros.org/wiki/xacro">
   <xacro:macro name="repair_hand_transmission" params="id">
-    <!-- synergy joint -->
-    <transmission name="trans_${id}_hand_v1s_synergy_joint">
-        <type>transmission_interface/SimpleTransmission</type>
-        <joint name="${id}_hand_v1s_synergy_joint">
-            <hardwareInterface>hardware_interface/PositionJointInterface</hardwareInterface>
-        </joint>
-        <actuator name="${id}_hand_v1s_synergy_joint_motor">
-            <!-- <hardwareInterface>hardware_interface/PositionJointInterface</hardwareInterface> -->
-            <mechanicalReduction>1</mechanicalReduction>
-        </actuator>
-    </transmission>
-    <!-- <transmission name="trans_${id}_hand_v1s_index_knuckle_joint">
+    <transmission name="trans_${id}_hand_v1s_index_knuckle_joint">
         <type>transmission_interface/SimpleTransmission</type>
         <joint name="${id}_hand_v1s_index_knuckle_joint">
@@ -202,5 +191,5 @@
             <mechanicalReduction>1</mechanicalReduction>
         </actuator>
-    </transmission> -->
+    </transmission>
   </xacro:macro>
 </robot>

File: repair_urdf/urdf/xbot2.gazebo.xacro (robot description, xacro)
@@ -30,6 +30,6 @@
         </pid>
         <ignore_joints>
-            <xacro:ignore_softhand_jnts side="right" type="v2s"/>
-            <xacro:ignore_softhand_jnts side="left" type="v2s"/>
+            <xacro:ignore_softhand_jnts side="right" type="v1s"/>
+            <xacro:ignore_softhand_jnts side="left" type="v1s"/>
         </ignore_joints>
     </plugin>
