Commit message: Added torso controller, transmission and related moveit_config

File: repair_urdf/urdf/repair.transmission.xacro (robot description, xacro)
@@ -72,4 +72,14 @@
         </actuator>
     </transmission>
+    <transmission name="trans_j_torso_1">
+        <type>transmission_interface/SimpleTransmission</type>
+        <joint name="j_torso_1">
+            <hardwareInterface>hardware_interface/PositionJointInterface</hardwareInterface>
+        </joint>
+        <actuator name="j_torso_1_motor">
+            <hardwareInterface>hardware_interface/PositionJointInterface</hardwareInterface>
+            <mechanicalReduction>1</mechanicalReduction>
+        </actuator>
+    </transmission>
   </xacro:macro>
 </robot>
