Commit message: Add perception and arm planning pipeline

File: repair_urdf/urdf/_d435.gazebo.xacro (robot description, xacro)
@@ -130,9 +130,9 @@
         <infrared2OpticalframeName>${infrared2_optical_frame}</infrared2OpticalframeName>
         <rangeMinDepth>0.2</rangeMinDepth>
-        <rangeMaxDepth>10.0</rangeMaxDepth>
+        <rangeMaxDepth>1.0</rangeMaxDepth>
         <pointCloud>${publish_pointcloud}</pointCloud>
         <pointCloudTopicName>depth/color/points</pointCloudTopicName>
         <pointCloudCutoff>0.25</pointCloudCutoff>
-        <pointCloudCutoffMax>9.0</pointCloudCutoffMax>
+        <pointCloudCutoffMax>1.0</pointCloudCutoffMax>
       </plugin>
     </gazebo>

File: repair_urdf/urdf/repair_full.urdf.xacro (robot description, xacro)
@@ -21,5 +21,5 @@
     </xacro:repair_cage>
     <xacro:sensor_d435 parent='torso_1'>
-        <origin xyz="0.09 0 -0.305" rpy="0 0.7535 0" />
+        <origin xyz="0.09 0 -0.305" rpy="0 0.9535 0" />
     </xacro:sensor_d435>
     <xacro:repair_torso parent="sliding_guide_link">
