Commit message: add realsense camera

File: repair_urdf/urdf/repair_full.urdf.xacro (robot description, xacro)
@@ -10,4 +10,5 @@
     <xacro:include filename="$(find repair_urdf)/urdf/inertial_properties.urdf.xacro" />
     <xacro:include filename="$(find repair_urdf)/urdf/limits.urdf.xacro" />
+    <xacro:include filename="$(find repair_urdf)/urdf/_d435.urdf.xacro"/>
     <!-- Only when working with Gazebo Xbot Control -->
     <!-- DO NOT USE WITH ROS_CONTROL AND MOVEIT -->
@@ -19,4 +20,7 @@
     <xacro:repair_cage parent="world">
     </xacro:repair_cage>
+    <xacro:sensor_d435 parent='world'>
+        <origin xyz="1 1 3" rpy="0 1.57 0" />
+    </xacro:sensor_d435>
     <xacro:repair_torso parent="sliding_guide_link">
     <origin xyz="${Torso_Ox} ${Torso_Oy} ${Torso_Oz}"

Commit message: fixed camera to torso

File: repair_urdf/urdf/repair_full.urdf.xacro (robot description, xacro)
@@ -20,6 +20,6 @@
     <xacro:repair_cage parent="world">
     </xacro:repair_cage>
-    <xacro:sensor_d435 parent='world'>
-        <origin xyz="1 1 3" rpy="0 1.57 0" />
+    <xacro:sensor_d435 parent='torso_1'>
+        <origin xyz="0.09 0 -0.305" rpy="0 0.7535 0" />
     </xacro:sensor_d435>
     <xacro:repair_torso parent="sliding_guide_link">

Commit message: Change camera rotation

File: repair_urdf/urdf/repair_full.urdf.xacro (robot description, xacro)
@@ -21,5 +21,5 @@
     </xacro:repair_cage>
     <xacro:sensor_d435 parent='torso_1'>
-        <origin xyz="0.09 0 -0.305" rpy="0 0.9535 0" />
+        <origin xyz="0.09 0 -0.305" rpy="0 1.178097 0" />
     </xacro:sensor_d435>
     <xacro:repair_torso parent="sliding_guide_link">

Commit message: camera translation

File: repair_urdf/urdf/repair_full.urdf.xacro (robot description, xacro)
@@ -22,4 +22,5 @@
     <xacro:sensor_d435 parent='torso_1'>
         <origin xyz="0.09 0 -0.305" rpy="0 1.178097 0" />
+        <!-- <origin xyz="0.0183991 0.0000476009 -0.3090088" rpy="0.0009783 1.1836725 1.5731959" /> -->
     </xacro:sensor_d435>
     <xacro:repair_torso parent="sliding_guide_link">

Commit message: new camera translation

File: repair_urdf/urdf/repair_full.urdf.xacro (robot description, xacro)
@@ -21,6 +21,7 @@
     </xacro:repair_cage>
     <xacro:sensor_d435 parent='torso_1'>
-        <origin xyz="0.09 0 -0.305" rpy="0 1.178097 0" />
-        <!-- <origin xyz="0.0183991 0.0000476009 -0.3090088" rpy="0.0009783 1.1836725 1.5731959" /> -->
+        <!-- <origin xyz="0.09 0 -0.305" rpy="0 1.178097 0" />  -->
+        <!-- <origin xyz="0.0857 0.0000476009 -0.273184" rpy="0.0009783 1.1836725 0" /> -->
+        <origin xyz="0.0857 0.0000476009 -0.273184" rpy="0.0009783 1.1836725 0" />
     </xacro:sensor_d435>
     <xacro:repair_torso parent="sliding_guide_link">
