Commit message: added sphere collision geoms for arms for dawnik

File: repair_urdf/urdf/repair_arm_macro.urdf.xacro (robot description, xacro)
@@ -9,5 +9,6 @@
 <!-- use_updated_wrist: visual parameter. if true, we load the latest meshes (which are adapted to the
 results of the optimization), otherwise we go with the old ones (generated for a spherical wrist) -->
-    <xacro:macro name="repair_arm" params="id rot parent *origin">
+    <xacro:include filename="$(find repair_urdf)/urdf/repair_arm_collision.urdf.xacro" />
+    <xacro:macro name="repair_arm" params="id rot parent *origin useCollisionMesh">
         <xacro:property name="limit_index" value="0" />
         <xacro:if value="${rot == -1}">
@@ -27,9 +28,5 @@
                 <material name="dark"/>
             </visual>
-            <collision>
-                <geometry>
-                    <mesh filename="package://repair_urdf/meshes/simplified/mesh_sh-pitch.stl" scale="0.001 ${rot*0.001} 0.001"/>
-                </geometry>
-            </collision>
+            <xacro:arm_1_collision id="${id}" rot="${rot}" isMesh="${useCollisionMesh}" />
         </link>
         <link name="arm_${id}_2">
@@ -46,9 +43,5 @@
                 <material name="dark"/>
             </visual>
-            <collision>
-                <geometry>
-                    <mesh filename="package://repair_urdf/meshes/simplified/mesh_sh-roll.stl" scale="0.001 ${rot*0.001} 0.001"/>
-                </geometry>
-            </collision>
+            <xacro:arm_2_collision id="${id}" rot="${rot}" isMesh="${useCollisionMesh}" />
         </link>
         <link name="arm_${id}_3">
@@ -65,9 +58,5 @@
                 <material name="dark"/>
             </visual>
-            <collision>
-                <geometry>
-                    <mesh filename="package://repair_urdf/meshes/simplified/mesh_sh-yaw.stl" scale="0.001 ${rot*0.001} 0.001"/>
-                </geometry>
-            </collision>
+            <xacro:arm_3_collision id="${id}" rot="${rot}" isMesh="${useCollisionMesh}" />
         </link>
         <link name="arm_${id}_4">
@@ -84,9 +73,5 @@
                 <material name="dark"/>
             </visual>
-            <collision>
-                <geometry>
-                    <mesh filename="package://repair_urdf/meshes/simplified/mesh_elbow.stl" scale="0.001 ${rot*0.001} 0.001"/>
-                </geometry>
-            </collision>
+            <xacro:arm_4_collision id="${id}" rot="${rot}" isMesh="${useCollisionMesh}" />
         </link>
         <link name="arm_${id}_5">
@@ -103,9 +88,5 @@
                 <material name="dark"/>
             </visual>
-            <collision>
-                <geometry>
-                    <mesh filename="package://repair_urdf/meshes/simplified/mesh_forearm-yaw.stl" scale="0.001 ${rot*0.001} 0.001"/>
-                </geometry>
-            </collision>
+            <xacro:arm_5_collision id="${id}" rot="${rot}" isMesh="${useCollisionMesh}" />
         </link>
         <link name="arm_${id}_6">
@@ -122,9 +103,5 @@
                 <material name="dark"/>
             </visual>
-            <collision>
-                <geometry>
-                    <mesh filename="package://repair_urdf/meshes/simplified/mesh_wrist-pitch.stl" scale="0.001 ${rot*0.001} 0.001"/>
-                </geometry>
-            </collision>
+            <xacro:arm_6_collision id="${id}" rot="${rot}" isMesh="${useCollisionMesh}" />
         </link>
         <link name="arm_${id}_7">
@@ -141,9 +118,5 @@
                 <material name="dark"/>
             </visual>
-            <collision>
-                <geometry>
-                    <mesh filename="package://repair_urdf/meshes/simplified/mesh_wrist-roll.stl" scale="0.001 ${rot*0.001} 0.001"/>
-                </geometry>
-            </collision>
+            <xacro:arm_7_collision id="${id}" rot="${rot}" isMesh="${useCollisionMesh}" />
         </link>
         <link name="arm_${id}_tcp">

File: repair_urdf/urdf/repair_full.urdf.xacro (robot description, xacro)
@@ -27,9 +27,9 @@
             rpy="${Torso_roll} ${Torso_pitch} ${Torso_yaw}" />
     </xacro:repair_torso>
-    <xacro:repair_arm id="2"  rot="1"  parent="torso_1">
+    <xacro:repair_arm id="2"  rot="1"  parent="torso_1" useCollisionMesh="false">
       <origin xyz="${Shoulder_1_Ox} ${Shoulder_1_Oy} ${Shoulder_1_Oz}"
               rpy="${Shoulder_1_roll} ${Shoulder_1_pitch} ${Shoulder_1_yaw}" />
     </xacro:repair_arm>
-    <xacro:repair_arm id="1"  rot="-1"  parent="torso_1">
+    <xacro:repair_arm id="1"  rot="-1"  parent="torso_1" useCollisionMesh="false">
         <origin xyz="${Shoulder_1_Ox} ${-Shoulder_1_Oy} ${Shoulder_1_Oz}"
                 rpy="${-Shoulder_1_roll} ${Shoulder_1_pitch} ${Shoulder_1_yaw}" />
