Commit message: updated visual mesh to simplified and added hands

File: repair_urdf/urdf/repair_arm_collision.urdf.xacro (robot description, xacro)
@@ -78,4 +78,5 @@
     <xacro:unless value="${isMesh}">
       <xacro:collision_sphere origin="0 0 0.0" radius="0.05" />
+      <xacro:collision_sphere origin="${rot*0.01} 0 0.14" radius="0.11" />
     </xacro:unless>
   </xacro:macro>

File: repair_urdf/urdf/repair_arm_macro.urdf.xacro (robot description, xacro)
@@ -24,5 +24,5 @@
             <visual>
                 <geometry>
-                    <mesh filename="package://repair_urdf/meshes/mesh_sh-pitch.stl" scale="0.001 ${rot*0.001} 0.001"/>
+                    <mesh filename="package://repair_urdf/meshes/simplified/mesh_sh-pitch.stl" scale="0.001 ${rot*0.001} 0.001"/>
                 </geometry>
                 <material name="dark"/>
@@ -39,5 +39,5 @@
             <visual>
                 <geometry>
-                    <mesh filename="package://repair_urdf/meshes/mesh_sh-roll.stl" scale="0.001 ${rot*0.001} 0.001"/>
+                    <mesh filename="package://repair_urdf/meshes/simplified/mesh_sh-roll.stl" scale="0.001 ${rot*0.001} 0.001"/>
                 </geometry>
                 <material name="dark"/>
@@ -54,5 +54,5 @@
             <visual>
                 <geometry>
-                    <mesh filename="package://repair_urdf/meshes/mesh_sh-yaw.stl" scale="0.001 ${rot*0.001} 0.001"/>
+                    <mesh filename="package://repair_urdf/meshes/simplified/mesh_sh-yaw.stl" scale="0.001 ${rot*0.001} 0.001"/>
                 </geometry>
                 <material name="dark"/>
@@ -69,5 +69,5 @@
             <visual>
                 <geometry>
-                    <mesh filename="package://repair_urdf/meshes/mesh_elbow.stl" scale="0.001 ${rot*0.001} 0.001"/>
+                    <mesh filename="package://repair_urdf/meshes/simplified/mesh_elbow.stl" scale="0.001 ${rot*0.001} 0.001"/>
                 </geometry>
                 <material name="dark"/>
@@ -84,5 +84,5 @@
             <visual>
                 <geometry>
-                    <mesh filename="package://repair_urdf/meshes/mesh_forearm-yaw.stl" scale="0.001 ${rot*0.001} 0.001"/>
+                    <mesh filename="package://repair_urdf/meshes/simplified/mesh_forearm-yaw.stl" scale="0.001 ${rot*0.001} 0.001"/>
                 </geometry>
                 <material name="dark"/>
@@ -99,5 +99,5 @@
             <visual>
                 <geometry>
-                    <mesh filename="package://repair_urdf/meshes/mesh_wrist-pitch.stl" scale="0.001 ${rot*0.001} 0.001"/>
+                    <mesh filename="package://repair_urdf/meshes/simplified/mesh_wrist-pitch.stl" scale="0.001 ${rot*0.001} 0.001"/>
                 </geometry>
                 <material name="dark"/>
@@ -114,5 +114,5 @@
             <visual>
                 <geometry>
-                    <mesh filename="package://repair_urdf/meshes/mesh_wrist-roll.stl" scale="0.001 ${rot*0.001} 0.001"/>
+                    <mesh filename="package://repair_urdf/meshes/simplified/mesh_wrist-roll.stl" scale="0.001 ${rot*0.001} 0.001"/>
                 </geometry>
                 <material name="dark"/>

File: repair_urdf/urdf/repair_full.urdf.xacro (robot description, xacro)
@@ -17,4 +17,6 @@
     <xacro:include filename="$(find repair_urdf)/urdf/common.gazebo.xacro" />
     <xacro:include filename="$(find repair_urdf)/urdf/repair_hand_transmission.xacro" />
+    <!-- property for enabling meshes for collision -->
+    <xacro:property name="useCollisionMesh" value="false" />
     <link name="world"/>
     <xacro:repair_cage parent="world">
@@ -27,13 +29,13 @@
             rpy="${Torso_roll} ${Torso_pitch} ${Torso_yaw}" />
     </xacro:repair_torso>
-    <xacro:repair_arm id="2"  rot="1"  parent="torso_1" useCollisionMesh="false">
+    <xacro:repair_arm id="2"  rot="1"  parent="torso_1" useCollisionMesh="${useCollisionMesh}">
       <origin xyz="${Shoulder_1_Ox} ${Shoulder_1_Oy} ${Shoulder_1_Oz}"
               rpy="${Shoulder_1_roll} ${Shoulder_1_pitch} ${Shoulder_1_yaw}" />
     </xacro:repair_arm>
-    <xacro:repair_arm id="1"  rot="-1"  parent="torso_1" useCollisionMesh="false">
+    <xacro:repair_arm id="1"  rot="-1"  parent="torso_1" useCollisionMesh="${useCollisionMesh}">
         <origin xyz="${Shoulder_1_Ox} ${-Shoulder_1_Oy} ${Shoulder_1_Oz}"
                 rpy="${-Shoulder_1_roll} ${Shoulder_1_pitch} ${Shoulder_1_yaw}" />
       </xacro:repair_arm>
-    <!-- <xacro:softhands type="left"
+    <xacro:softhands type="left"
         version="v1.0_simple"
         parent="arm_1_7"
@@ -42,5 +44,6 @@
         translation="0"
         operation_mode="0"
-        fixed_hands="false">
+        fixed_hands="false"
+        useCollisionMesh="${useCollisionMesh}">
     </xacro:softhands>
     <xacro:softhands type="right"
@@ -51,10 +54,11 @@
         translation="0"
         operation_mode="0"
-        fixed_hands="false">
-    </xacro:softhands> -->
-    <!-- <gazebo reference="table_top_link">
+        fixed_hands="false"
+        useCollisionMesh="${useCollisionMesh}">
+    </xacro:softhands>
+    <gazebo reference="table_top_link">
         <selfCollide> 1 </selfCollide>
-    </gazebo> -->
-    <!-- <xacro:repair_hand_transmission id="left" />
-    <xacro:repair_hand_transmission id="right" /> -->
+    </gazebo>
+    <xacro:repair_hand_transmission id="left" />
+    <xacro:repair_hand_transmission id="right" />
 </robot>
