Commit message: edited limits, free_motion and box_bimanual scripts

File: repair_urdf/urdf/limits.urdf.xacro (robot description, xacro)
@@ -20,6 +20,6 @@
     <xacro:property name="j_arm_6_upper" value="${[2.1, 2.8]}"/>
     <xacro:property name="j_arm_7_upper" value="${[2.8, 2.8]}"/>
-    <xacro:property name="j_prismatic_velocity" value="${[3]}"/>
-    <xacro:property name="j_torso_velocity" value="${[3.86]}"/>
+    <xacro:property name="j_prismatic_velocity" value="${[2.]}"/>
+    <xacro:property name="j_torso_velocity" value="${[2.]}"/>
     <xacro:property name="j_arm_1_velocity" value="${[3.86]}"/>
     <xacro:property name="j_arm_2_velocity" value="${[3.86]}"/>

File: repair_urdf/urdf/repair_full.urdf (robot description, URDF)
Before this commit: robot repair_full, 116 links, 115 joints
Joints:
- joint j_torso_1: limit lower=-2.6 upper=2.6 effort=147.0 velocity=3.86 -> lower=-2.6 upper=2.6 effort=147.0 velocity=2.0
- joint j_torso_base: limit lower=-0.8 upper=0.8 effort=147 velocity=3 -> lower=-0.8 upper=0.8 effort=147 velocity=2.0
