Commit message: working configuration with small and wide hands working tree

File: repair_urdf/urdf/kinematics_properties.urdf.xacro (robot description, xacro)
@@ -17,7 +17,7 @@
     <xacro:property name="Torso_Oy" value=" 0.0 "/>
     <xacro:property name="Torso_Oz" value=" 0.0 "/>
-    <xacro:property name="Torso_roll" value=" ${PI/2} "/>
+    <xacro:property name="Torso_roll" value=" 0.0 "/>
     <xacro:property name="Torso_pitch" value=" 0.0 "/>
-    <xacro:property name="Torso_yaw" value=" ${PI/2}"/>
+    <xacro:property name="Torso_yaw" value=" 0.0"/>
     <!-- Origin -->
     <xacro:property name="Shoulder_1_Ox" value=" 0.0 "/>  <!-- 0.0  -->

File: repair_urdf/urdf/repair_full.urdf (robot description, URDF)
Before this commit: robot repair_full, 120 links, 119 joints
Joints:
- joint j_torso_base: origin xyz=0.0 0.0 0.0 rpy=1.570796326795 0.0 1.570796326795 -> xyz=0.0 0.0 0.0 rpy=0.0 0.0 0.0
