Commit message: bimanual with both small hands

File: repair_urdf/urdf/kinematics_properties.urdf.xacro (robot description, xacro)
@@ -17,7 +17,7 @@
     <xacro:property name="Torso_Oy" value=" 0.0 "/>
     <xacro:property name="Torso_Oz" value=" 0.0 "/>
-    <xacro:property name="Torso_roll" value=" 0.0 "/>
+    <xacro:property name="Torso_roll" value=" ${PI/2} "/>
     <xacro:property name="Torso_pitch" value=" 0.0 "/>
-    <xacro:property name="Torso_yaw" value=" 0.0"/>
+    <xacro:property name="Torso_yaw" value=" ${PI/2}"/>
     <!-- Origin -->
     <xacro:property name="Shoulder_1_Ox" value=" 0.0 "/>  <!-- 0.0  -->

File: repair_urdf/urdf/limits.urdf.xacro (robot description, xacro)
@@ -20,5 +20,5 @@
     <xacro:property name="j_arm_6_upper" value="${[2.1, 2.8]}"/>
     <xacro:property name="j_arm_7_upper" value="${[2.8, 2.8]}"/>
-    <xacro:property name="j_prismatic_velocity" value="${[5]}"/>
+    <xacro:property name="j_prismatic_velocity" value="${[3]}"/>
     <xacro:property name="j_torso_velocity" value="${[3.86]}"/>
     <xacro:property name="j_arm_1_velocity" value="${[3.86]}"/>

File: repair_urdf/urdf/repair_full.urdf (robot description, URDF)
Before this commit: robot repair_full, 120 links, 119 joints
Links:
- removed link left_hand_v1_wide_grasp_link
- removed link left_hand_v1_wide_index_distal_link
- removed link left_hand_v1_wide_index_distal_virtual_link
- removed link left_hand_v1_wide_index_knuckle_link
- removed link left_hand_v1_wide_index_middle_link
- removed link left_hand_v1_wide_index_middle_virtual_link
- removed link left_hand_v1_wide_index_proximal_link
- removed link left_hand_v1_wide_index_proximal_virtual_link
- removed link left_hand_v1_wide_little_distal_link
- removed link left_hand_v1_wide_little_distal_virtual_link
- removed link left_hand_v1_wide_little_knuckle_link
- removed link left_hand_v1_wide_little_middle_link
- removed link left_hand_v1_wide_little_middle_virtual_link
- removed link left_hand_v1_wide_little_proximal_link
- removed link left_hand_v1_wide_little_proximal_virtual_link
- removed link left_hand_v1_wide_middle_distal_link
- removed link left_hand_v1_wide_middle_distal_virtual_link
- removed link left_hand_v1_wide_middle_knuckle_link
- removed link left_hand_v1_wide_middle_middle_link
- removed link left_hand_v1_wide_middle_middle_virtual_link
- removed link left_hand_v1_wide_middle_proximal_link
- removed link left_hand_v1_wide_middle_proximal_virtual_link
- removed link left_hand_v1_wide_palm_central_link
- removed link left_hand_v1_wide_palm_central_little_link
- removed link left_hand_v1_wide_palm_central_thumb_link
- removed link left_hand_v1_wide_palm_little_link
- removed link left_hand_v1_wide_palm_thumb_link
- removed link left_hand_v1_wide_palm_thumb_support_link
- removed link left_hand_v1_wide_ring_distal_link
- removed link left_hand_v1_wide_ring_distal_virtual_link
- removed link left_hand_v1_wide_ring_knuckle_link
- removed link left_hand_v1_wide_ring_middle_link
- removed link left_hand_v1_wide_ring_middle_virtual_link
- removed link left_hand_v1_wide_ring_proximal_link
- removed link left_hand_v1_wide_ring_proximal_virtual_link
- removed link left_hand_v1_wide_thumb_distal_link
- removed link left_hand_v1_wide_thumb_distal_virtual_link
- removed link left_hand_v1_wide_thumb_knuckle_link
- removed link left_hand_v1_wide_thumb_proximal_link
- removed link left_hand_v1_wide_thumb_proximal_virtual_link
- added link left_hand_v1_2_research_grasp_link
- added link left_hand_v1_2_research_index_distal_link, mass 0.009; collision mesh filename=package://softhands_description/meshes/v1_2_research/left/p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 scale=0.001 0.001 0.001; visual mesh filename=package://softhands_description/meshes/v1_2_research/left/p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 scale=0.001 0.001 0.001
- added link left_hand_v1_2_research_index_distal_virtual_link, mass 0.009
- added link left_hand_v1_2_research_index_knuckle_link, mass 0.0095; collision mesh filename=package://softhands_description/meshes/v1_2_research/left/p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 scale=0.001 0.001 0.001; visual mesh filename=package://softhands_description/meshes/v1_2_research/left/p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 scale=0.001 0.001 0.001
- added link left_hand_v1_2_research_index_middle_link, mass 0.0063; collision mesh filename=package://softhands_description/meshes/v1_2_research/left/p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 scale=0.001 0.001 0.001; visual mesh filename=package://softhands_description/meshes/v1_2_research/left/p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 scale=0.001 0.001 0.001
- added link left_hand_v1_2_research_index_middle_virtual_link, mass 0.0063
- added link left_hand_v1_2_research_index_proximal_link, mass 0.009; collision mesh filename=package://softhands_description/meshes/v1_2_research/left/p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 scale=0.001 0.001 0.001; visual mesh filename=package://softhands_description/meshes/v1_2_research/left/p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 scale=0.001 0.001 0.001
- added link left_hand_v1_2_research_index_proximal_virtual_link, mass 0.009
- added link left_hand_v1_2_research_iso_link, mass 0.205; collision mesh filename=package://softhands_description/meshes/v1_2_research/left/f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 scale=0.001 0.001 0.001; visual mesh filename=package://softhands_description/meshes/v1_2_research/left/f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 scale=0.001 0.001 0.001
- added link left_hand_v1_2_research_little_distal_link, mass 0.009; collision mesh filename=package://softhands_description/meshes/v1_2_research/left/p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 scale=0.001 0.001 0.001; visual mesh filename=package://softhands_description/meshes/v1_2_research/left/p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 scale=0.001 0.001 0.001
- added link left_hand_v1_2_research_little_distal_virtual_link, mass 0.009
- added link left_hand_v1_2_research_little_knuckle_link, mass 0.0095; collision mesh filename=package://softhands_description/meshes/v1_2_research/left/p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 scale=0.001 0.001 0.001; visual mesh filename=package://softhands_description/meshes/v1_2_research/left/p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 scale=0.001 0.001 0.001
- added link left_hand_v1_2_research_little_middle_link, mass 0.0063; collision mesh filename=package://softhands_description/meshes/v1_2_research/left/p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 scale=0.001 0.001 0.001; visual mesh filename=package://softhands_description/meshes/v1_2_research/left/p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 scale=0.001 0.001 0.001
- added link left_hand_v1_2_research_little_middle_virtual_link, mass 0.0063
- added link left_hand_v1_2_research_little_proximal_link, mass 0.009; collision mesh filename=package://softhands_description/meshes/v1_2_research/left/p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 scale=0.001 0.001 0.001; visual mesh filename=package://softhands_description/meshes/v1_2_research/left/p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 scale=0.001 0.001 0.001
- added link left_hand_v1_2_research_little_proximal_virtual_link, mass 0.009
- added link left_hand_v1_2_research_middle_distal_link, mass 0.009; collision mesh filename=package://softhands_description/meshes/v1_2_research/left/p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 scale=0.001 0.001 0.001; visual mesh filename=package://softhands_description/meshes/v1_2_research/left/p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 scale=0.001 0.001 0.001
- added link left_hand_v1_2_research_middle_distal_virtual_link, mass 0.009
- added link left_hand_v1_2_research_middle_knuckle_link, mass 0.0095; collision mesh filename=package://softhands_description/meshes/v1_2_research/left/p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 scale=0.001 0.001 0.001; visual mesh filename=package://softhands_description/meshes/v1_2_research/left/p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 scale=0.001 0.001 0.001
- added link left_hand_v1_2_research_middle_middle_link, mass 0.0063; collision mesh filename=package://softhands_description/meshes/v1_2_research/left/p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 scale=0.001 0.001 0.001; visual mesh filename=package://softhands_description/meshes/v1_2_research/left/p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 scale=0.001 0.001 0.001
- added link left_hand_v1_2_research_middle_middle_virtual_link, mass 0.0063
- added link left_hand_v1_2_research_middle_proximal_link, mass 0.009; collision mesh filename=package://softhands_description/meshes/v1_2_research/left/p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 scale=0.001 0.001 0.001; visual mesh filename=package://softhands_description/meshes/v1_2_research/left/p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 scale=0.001 0.001 0.001
- added link left_hand_v1_2_research_middle_proximal_virtual_link, mass 0.009
- added link left_hand_v1_2_research_palm_link, mass 0.45; collision mesh filename=package://softhands_description/meshes/v1_2_research/left/p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 scale=0.001 0.001 0.001; visual mesh filename=package://softhands_description/meshes/v1_2_research/left/p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 scale=0.001 0.001 0.001
- added link left_hand_v1_2_research_ring_distal_link, mass 0.009; collision mesh filename=package://softhands_description/meshes/v1_2_research/left/p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 scale=0.001 0.001 0.001; visual mesh filename=package://softhands_description/meshes/v1_2_research/left/p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 scale=0.001 0.001 0.001
- added link left_hand_v1_2_research_ring_distal_virtual_link, mass 0.009
- added link left_hand_v1_2_research_ring_knuckle_link, mass 0.0095; collision mesh filename=package://softhands_description/meshes/v1_2_research/left/p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 scale=0.001 0.001 0.001; visual mesh filename=package://softhands_description/meshes/v1_2_research/left/p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 scale=0.001 0.001 0.001
- added link left_hand_v1_2_research_ring_middle_link, mass 0.0063; collision mesh filename=package://softhands_description/meshes/v1_2_research/left/p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 scale=0.001 0.001 0.001; visual mesh filename=package://softhands_description/meshes/v1_2_research/left/p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 scale=0.001 0.001 0.001
- added link left_hand_v1_2_research_ring_middle_virtual_link, mass 0.0063
- added link left_hand_v1_2_research_ring_proximal_link, mass 0.009; collision mesh filename=package://softhands_description/meshes/v1_2_research/left/p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 scale=0.001 0.001 0.001; visual mesh filename=package://softhands_description/meshes/v1_2_research/left/p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 scale=0.001 0.001 0.001
- added link left_hand_v1_2_research_ring_proximal_virtual_link, mass 0.009
- added link left_hand_v1_2_research_thumb_distal_link, mass 0.009; collision mesh filename=package://softhands_description/meshes/v1_2_research/left/p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 scale=0.001 0.001 0.001; visual mesh filename=package://softhands_description/meshes/v1_2_research/left/p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 scale=0.001 0.001 0.001
- added link left_hand_v1_2_research_thumb_distal_virtual_link, mass 0.009
- added link left_hand_v1_2_research_thumb_knuckle_link, mass 0.01; collision mesh filename=package://softhands_description/meshes/v1_2_research/left/p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 scale=0.001 0.001 0.001; visual mesh filename=package://softhands_description/meshes/v1_2_research/left/p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 scale=0.001 0.001 0.001
- added link left_hand_v1_2_research_thumb_proximal_link, mass 0.0063; collision mesh filename=package://softhands_description/meshes/v1_2_research/left/p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 scale=0.001 0.001 0.001; visual mesh filename=package://softhands_description/meshes/v1_2_research/left/p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 scale=0.001 0.001 0.001
- added link left_hand_v1_2_research_thumb_proximal_virtual_link, mass 0.0063
Joints:
- removed joint left_hand_v1_wide_grasp_joint
- removed joint left_hand_v1_wide_index_distal_joint
- removed joint left_hand_v1_wide_index_distal_virtual_joint
- removed joint left_hand_v1_wide_index_knuckle_joint
- removed joint left_hand_v1_wide_index_middle_joint
- removed joint left_hand_v1_wide_index_middle_virtual_joint
- removed joint left_hand_v1_wide_index_proximal_joint
- removed joint left_hand_v1_wide_index_proximal_virtual_joint
- removed joint left_hand_v1_wide_little_distal_joint
- removed joint left_hand_v1_wide_little_distal_virtual_joint
- removed joint left_hand_v1_wide_little_knuckle_joint
- removed joint left_hand_v1_wide_little_middle_joint
- removed joint left_hand_v1_wide_little_middle_virtual_joint
- removed joint left_hand_v1_wide_little_proximal_joint
- removed joint left_hand_v1_wide_little_proximal_virtual_joint
- removed joint left_hand_v1_wide_middle_distal_joint
- removed joint left_hand_v1_wide_middle_distal_virtual_joint
- removed joint left_hand_v1_wide_middle_knuckle_joint
- removed joint left_hand_v1_wide_middle_middle_joint
- removed joint left_hand_v1_wide_middle_middle_virtual_joint
- removed joint left_hand_v1_wide_middle_proximal_joint
- removed joint left_hand_v1_wide_middle_proximal_virtual_joint
- removed joint left_hand_v1_wide_palm_central_joint
- removed joint left_hand_v1_wide_palm_central_little_joint
- removed joint left_hand_v1_wide_palm_central_little_virtual_joint
- removed joint left_hand_v1_wide_palm_central_thumb_joint
- removed joint left_hand_v1_wide_palm_central_thumb_virtual_joint
- removed joint left_hand_v1_wide_palm_thumb_support_joint
- removed joint left_hand_v1_wide_ring_distal_joint
- removed joint left_hand_v1_wide_ring_distal_virtual_joint
- removed joint left_hand_v1_wide_ring_knuckle_joint
- removed joint left_hand_v1_wide_ring_middle_joint
- removed joint left_hand_v1_wide_ring_middle_virtual_joint
- removed joint left_hand_v1_wide_ring_proximal_joint
- removed joint left_hand_v1_wide_ring_proximal_virtual_joint
- removed joint left_hand_v1_wide_thumb_distal_joint
- removed joint left_hand_v1_wide_thumb_distal_virtual_joint
- removed joint left_hand_v1_wide_thumb_knuckle_joint
- removed joint left_hand_v1_wide_thumb_proximal_joint
- removed joint left_hand_v1_wide_thumb_proximal_virtual_joint
- added joint left_hand_v1_2_research_grasp_joint: type fixed, parent left_hand_v1_2_research_iso_link, child left_hand_v1_2_research_grasp_link, origin xyz=0.06 0.03 0.16 rpy=0 0 1.57
- added joint left_hand_v1_2_research_index_distal_joint: type fixed, parent left_hand_v1_2_research_index_distal_virtual_link, child left_hand_v1_2_research_index_distal_link, origin xyz=0.013 0 0 rpy=0 0 0, axis 0 0 -1, limit lower=0.0 upper=0.785398 effort=30 velocity=10.0
- added joint left_hand_v1_2_research_index_distal_virtual_joint: type fixed, parent left_hand_v1_2_research_index_middle_link, child left_hand_v1_2_research_index_distal_virtual_link, origin xyz=0.009 0 0 rpy=0 0 0, axis 0 0 -1, limit lower=0.0 upper=0.785398 effort=30 velocity=10.0
- added joint left_hand_v1_2_research_index_knuckle_joint: type fixed, parent left_hand_v1_2_research_palm_link, child left_hand_v1_2_research_index_knuckle_link, origin xyz=-0.02 -0.007 -0.014 rpy=0 3.14 -1.57, axis 0 0 -1, limit lower=-0.524 upper=0.524 effort=30 velocity=10.0
- added joint left_hand_v1_2_research_index_middle_joint: type fixed, parent left_hand_v1_2_research_index_middle_virtual_link, child left_hand_v1_2_research_index_middle_link, origin xyz=0.017 0 0 rpy=0 0 0, axis 0 0 -1, limit lower=0.0 upper=0.785398 effort=30 velocity=10.0
- added joint left_hand_v1_2_research_index_middle_virtual_joint: type fixed, parent left_hand_v1_2_research_index_proximal_link, child left_hand_v1_2_research_index_middle_virtual_link, origin xyz=0.013 0 0  rpy=0.0 0.0 0.0, axis 0 0 -1, limit lower=0.0 upper=0.785398 effort=30 velocity=10.0
- added joint left_hand_v1_2_research_index_proximal_joint: type fixed, parent left_hand_v1_2_research_index_proximal_virtual_link, child left_hand_v1_2_research_index_proximal_link, origin xyz=0.013 0 0 rpy=0.0 0 0, axis 0 0 -1, limit lower=0.0 upper=0.785398 effort=30 velocity=10.0
- added joint left_hand_v1_2_research_index_proximal_virtual_joint: type fixed, parent left_hand_v1_2_research_index_knuckle_link, child left_hand_v1_2_research_index_proximal_virtual_link, origin xyz=0.009 0 0 rpy=1.57 0 0, axis 0 0 -1, limit lower=0.0 upper=0.785398 effort=30 velocity=10.0
- added joint left_hand_v1_2_research_iso_joint: type fixed, parent arm_1_7, child left_hand_v1_2_research_iso_link, origin xyz=0 -0. 0.00 rpy=0 0 0
- added joint left_hand_v1_2_research_little_distal_joint: type fixed, parent left_hand_v1_2_research_little_distal_virtual_link, child left_hand_v1_2_research_little_distal_link, origin xyz=0.013 0 0 rpy=0 0 0, axis 0 0 -1, limit lower=0.0 upper=0.785398 effort=30 velocity=10.0
- added joint left_hand_v1_2_research_little_distal_virtual_joint: type fixed, parent left_hand_v1_2_research_little_middle_link, child left_hand_v1_2_research_little_distal_virtual_link, origin xyz=0.009 0 0 rpy=0 0 0, axis 0 0 -1, limit lower=0.0 upper=0.785398 effort=30 velocity=10.0
- added joint left_hand_v1_2_research_little_knuckle_joint: type fixed, parent left_hand_v1_2_research_palm_link, child left_hand_v1_2_research_little_knuckle_link, origin xyz=0.04 -0.012 -0.014 rpy=0 3.14 -1.57, axis 0 0 -1, limit lower=-0.524 upper=0.524 effort=30 velocity=10.0
- added joint left_hand_v1_2_research_little_middle_joint: type fixed, parent left_hand_v1_2_research_little_middle_virtual_link, child left_hand_v1_2_research_little_middle_link, origin xyz=0.017 0 0 rpy=0 0 0, axis 0 0 -1, limit lower=0.0 upper=0.785398 effort=30 velocity=10.0
- added joint left_hand_v1_2_research_little_middle_virtual_joint: type fixed, parent left_hand_v1_2_research_little_proximal_link, child left_hand_v1_2_research_little_middle_virtual_link, origin xyz=0.013 0 0  rpy=0.0 0.0 0.0, axis 0 0 -1, limit lower=0.0 upper=0.785398 effort=30 velocity=10.0
- added joint left_hand_v1_2_research_little_proximal_joint: type fixed, parent left_hand_v1_2_research_little_proximal_virtual_link, child left_hand_v1_2_research_little_proximal_link, origin xyz=0.013 0 0 rpy=0.0 0 0, axis 0 0 -1, limit lower=0.0 upper=0.785398 effort=30 velocity=10.0
- added joint left_hand_v1_2_research_little_proximal_virtual_joint: type fixed, parent left_hand_v1_2_research_little_knuckle_link, child left_hand_v1_2_research_little_proximal_virtual_link, origin xyz=0.009 0 0 rpy=1.57 0 0, axis 0 0 -1, limit lower=0.0 upper=0.785398 effort=30 velocity=10.0
- added joint left_hand_v1_2_research_middle_distal_joint: type fixed, parent left_hand_v1_2_research_middle_distal_virtual_link, child left_hand_v1_2_research_middle_distal_link, origin xyz=0.013 0 0 rpy=0 0 0, axis 0 0 -1, limit lower=0.0 upper=0.785398 effort=30 velocity=10.0
- added joint left_hand_v1_2_research_middle_distal_virtual_joint: type fixed, parent left_hand_v1_2_research_middle_middle_link, child left_hand_v1_2_research_middle_distal_virtual_link, origin xyz=0.009 0 0 rpy=0 0 0, axis 0 0 -1, limit lower=0.0 upper=0.785398 effort=30 velocity=10.0
- added joint left_hand_v1_2_research_middle_knuckle_joint: type fixed, parent left_hand_v1_2_research_palm_link, child left_hand_v1_2_research_middle_knuckle_link, origin xyz=0 0 -0.014 rpy=0 3.14 -1.57, axis 0 0 -1, limit lower=-0.524 upper=0.524 effort=30 velocity=10.0
- added joint left_hand_v1_2_research_middle_middle_joint: type fixed, parent left_hand_v1_2_research_middle_middle_virtual_link, child left_hand_v1_2_research_middle_middle_link, origin xyz=0.017 0 0 rpy=0 0 0, axis 0 0 -1, limit lower=0.0 upper=0.785398 effort=30 velocity=10.0
- added joint left_hand_v1_2_research_middle_middle_virtual_joint: type fixed, parent left_hand_v1_2_research_middle_proximal_link, child left_hand_v1_2_research_middle_middle_virtual_link, origin xyz=0.013 0 0  rpy=0.0 0.0 0.0, axis 0 0 -1, limit lower=0.0 upper=0.785398 effort=30 velocity=10.0
- added joint left_hand_v1_2_research_middle_proximal_joint: type fixed, parent left_hand_v1_2_research_middle_proximal_virtual_link, child left_hand_v1_2_research_middle_proximal_link, origin xyz=0.013 0 0 rpy=0.0 0 0, axis 0 0 -1, limit lower=0.0 upper=0.785398 effort=30 velocity=10.0
- added joint left_hand_v1_2_research_middle_proximal_virtual_joint: type fixed, parent left_hand_v1_2_research_middle_knuckle_link, child left_hand_v1_2_research_middle_proximal_virtual_link, origin xyz=0.009 0 0 rpy=1.57 0 0, axis 0 0 -1, limit lower=0.0 upper=0.785398 effort=30 velocity=10.0
- added joint left_hand_v1_2_research_palm_joint: type fixed, parent left_hand_v1_2_research_iso_link, child left_hand_v1_2_research_palm_link, origin xyz=0.0045 0.0145 0.144 rpy=1.57 0  3.14
- added joint left_hand_v1_2_research_ring_distal_joint: type fixed, parent left_hand_v1_2_research_ring_distal_virtual_link, child left_hand_v1_2_research_ring_distal_link, origin xyz=0.013 0 0 rpy=0 0 0, axis 0 0 -1, limit lower=0.0 upper=0.785398 effort=30 velocity=10.0
- added joint left_hand_v1_2_research_ring_distal_virtual_joint: type fixed, parent left_hand_v1_2_research_ring_middle_link, child left_hand_v1_2_research_ring_distal_virtual_link, origin xyz=0.009 0 0 rpy=0 0 0, axis 0 0 -1, limit lower=0.0 upper=0.785398 effort=30 velocity=10.0
- added joint left_hand_v1_2_research_ring_knuckle_joint: type fixed, parent left_hand_v1_2_research_palm_link, child left_hand_v1_2_research_ring_knuckle_link, origin xyz=0.02 -0.007 -0.014 rpy=0 3.14 -1.57, axis 0 0 -1, limit lower=-0.524 upper=0.524 effort=30 velocity=10.0
- added joint left_hand_v1_2_research_ring_middle_joint: type fixed, parent left_hand_v1_2_research_ring_middle_virtual_link, child left_hand_v1_2_research_ring_middle_link, origin xyz=0.017 0 0 rpy=0 0 0, axis 0 0 -1, limit lower=0.0 upper=0.785398 effort=30 velocity=10.0
- added joint left_hand_v1_2_research_ring_middle_virtual_joint: type fixed, parent left_hand_v1_2_research_ring_proximal_link, child left_hand_v1_2_research_ring_middle_virtual_link, origin xyz=0.013 0 0  rpy=0.0 0.0 0.0, axis 0 0 -1, limit lower=0.0 upper=0.785398 effort=30 velocity=10.0
- added joint left_hand_v1_2_research_ring_proximal_joint: type fixed, parent left_hand_v1_2_research_ring_proximal_virtual_link, child left_hand_v1_2_research_ring_proximal_link, origin xyz=0.013 0 0 rpy=0.0 0 0, axis 0 0 -1, limit lower=0.0 upper=0.785398 effort=30 velocity=10.0
- added joint left_hand_v1_2_research_ring_proximal_virtual_joint: type fixed, parent left_hand_v1_2_research_ring_knuckle_link, child left_hand_v1_2_research_ring_proximal_virtual_link, origin xyz=0.009 0 0 rpy=1.57 0 0, axis 0 0 -1, limit lower=0.0 upper=0.785398 effort=30 velocity=10.0
- added joint left_hand_v1_2_research_thumb_distal_joint: type fixed, parent left_hand_v1_2_research_thumb_distal_virtual_link, child left_hand_v1_2_research_thumb_distal_link, origin xyz=0.013 0 0 rpy=0 0 0, axis 0 0 -1, limit lower=0.0 upper=0.785398 effort=30 velocity=10.0
- added joint left_hand_v1_2_research_thumb_distal_virtual_joint: type fixed, parent left_hand_v1_2_research_thumb_proximal_link, child left_hand_v1_2_research_thumb_distal_virtual_link, origin xyz=0.009 0 0 rpy=0 0 0, axis 0 0 -1, limit lower=0.0 upper=0.785398 effort=30 velocity=10.0
- added joint left_hand_v1_2_research_thumb_knuckle_joint: type fixed, parent left_hand_v1_2_research_palm_link, child left_hand_v1_2_research_thumb_knuckle_link, origin xyz=-0.044 -0.0465 0.002 rpy=-1.57 3.14 0.0, axis 0 0 1, limit lower=0.0 upper=1.57 effort=30 velocity=10.0
- added joint left_hand_v1_2_research_thumb_proximal_joint: type fixed, parent left_hand_v1_2_research_thumb_proximal_virtual_link, child left_hand_v1_2_research_thumb_proximal_link, origin xyz=0.013 0 0 rpy=0 0 0, axis 0 0 -1, limit lower=0.0 upper=0.785398 effort=30 velocity=10.0
- added joint left_hand_v1_2_research_thumb_proximal_virtual_joint: type fixed, parent left_hand_v1_2_research_thumb_knuckle_link, child left_hand_v1_2_research_thumb_proximal_virtual_link, origin xyz=0.0255 0.0038 -0.00012 rpy=-2 0.0 0.0, axis 0 0 -1, limit lower=0.0 upper=0.785398 effort=30 velocity=10.0
- joint j_torso_base: limit lower=-0.8 upper=0.8 effort=147 velocity=5 -> lower=-0.8 upper=0.8 effort=147 velocity=3
