Commit message: bimanual with both small hands

File: repair_urdf/urdf/repair_full.urdf.xacro (robot description, xacro)
@@ -37,5 +37,5 @@
     <!--QUIRINO/GIANNIROS: here change the version for v1_2_research (small hand) or v1_wide (wide hand)-->
     <xacro:softhands
-        version="mixed_hands"
+        version="v1_2_research"
         position="0 0 0"
         orientation="${PI}"

File: repair_urdf/urdf/repair_torso_macro.urdf.xacro (robot description, xacro)
@@ -23,5 +23,6 @@
         </link>
         <joint name="j_torso_base" type="prismatic">
-            <xacro:insert_block name="origin" />
+            <!-- <xacro:insert_block name="origin" /> -->
+            <origin rpy="0.0 0.0 0.0" xyz="0.0 0.0 0.0"/>
             <parent link="${parent}" />
             <child link="dummy_prismatic_link"/>

Commit message: partiallz working state tuesday

File: repair_urdf/urdf/kinematics_properties.urdf.xacro (robot description, xacro)
@@ -67,5 +67,5 @@
     <xacro:property name="Wrist_2_Oz" value=" 0.050 "/>
     <xacro:property name="Wrist_2_roll" value=" ${-PI/2} "/>
-    <xacro:property name="Wrist_2_pitch" value=" 0.3316123 "/>
+    <xacro:property name="Wrist_2_pitch" value=" 0.0"/>
     <xacro:property name="Wrist_2_yaw" value=" 0.0 "/>
     <!-- END-EFFECTORS-->

File: repair_urdf/urdf/repair_full.urdf (robot description, URDF)
Before this commit: robot repair_full, 128 links, 127 joints
Joints:
- joint j_arm_1_7: origin xyz=0.0 -0.062877 0.05 rpy=1.570796326795 0.3316123 0.0 -> xyz=0.0 -0.062877 0.05 rpy=1.570796326795 0.03316123 0.0
- joint j_arm_2_7: origin xyz=0.0 0.062877 0.05 rpy=-1.570796326795 0.3316123 0.0 -> xyz=0.0 0.062877 0.05 rpy=-1.570796326795 0.03316123 0.0

File: repair_urdf/urdf/repair_torso_macro.urdf.xacro (robot description, xacro)
@@ -2,11 +2,11 @@
 <robot xmlns:xacro="http://ros.org/wiki/xacro">
     <xacro:macro name="repair_torso" params="parent *origin">
-        <joint name="j_sliding_guide" type="fixed">
+        <!-- <joint name="j_sliding_guide" type="fixed">
             <origin xyz="0 0 0" rpy="0 0 0" />
             <parent link="${parent}" />
             <child link="dummy_prismatic_link"/>
-            <!-- <axis xyz="0 0 -1"/> -->
-            <!-- <limit lower="${j_prismatic_lower[0]/2}" upper= "${j_prismatic_upper[0]/2}" effort="${j_prismatic_torque[0]}" velocity="${j_prismatic_velocity[0]}"/> -->
-        </joint>
+            <axis xyz="0 0 -1"/>
+            <limit lower="${j_prismatic_lower[0]/2}" upper= "${j_prismatic_upper[0]/2}" effort="${j_prismatic_torque[0]}" velocity="${j_prismatic_velocity[0]}"/>
+        </joint>-->
         <link name="dummy_prismatic_link"/>
         <link name="torso_1">
@@ -29,19 +29,12 @@
             </collision>
         </link>
-        <!-- <joint name="j_torso_base" type="fixed">
-            <xacro:insert_block name="origin" />
-            <parent link="${parent}" />
-            <child link="dummy_prismatic_link"/>
-            <axis xyz="0 0 1"/>
-            <limit lower="${j_prismatic_lower[0]/2}" upper= "${j_prismatic_upper[0]/2}" effort="${j_prismatic_torque[0]}" velocity="${j_prismatic_velocity[0]}"/>
-        </joint> -->
-        <!-- <joint name="j_torso_base" type="fixed">
-         <xacro:insert_block name="origin" />
+        <joint name="j_torso_base" type="fixed">
+        <!-- <xacro:insert_block name="origin" /> -->
         <origin rpy="0.0 0.0 0.0" xyz="0.0 0.0 0.0"/>
         <parent link="sliding_guide_link"/>
                 <child link="dummy_prismatic_link"/>
                 <axis xyz="0 0 1"/>
-        <limit effort="147" lower="-0.8" upper="0.8" velocity="2.2"/>
-            </joint> -->
+        <limit lower="${j_prismatic_lower[0]/2}" upper= "${j_prismatic_upper[0]/2}" effort="${j_prismatic_torque[0]}" velocity="${j_prismatic_velocity[0]}"/>
+            </joint>
         <!-- torso -->
         <joint name="j_torso_1" type="revolute">

Commit message: first working demo and new recognition script

File: repair_urdf/urdf/kinematics_properties.urdf.xacro (robot description, xacro)
@@ -15,5 +15,5 @@
     <xacro:property name="Cage_sliding_guide_width" value="0.4"/>
     <xacro:property name="Torso_Ox" value=" 0.0 "/>
-    <xacro:property name="Torso_Oy" value=" 0.0 "/>
+    <xacro:property name="Torso_Oy" value=" 0.07 "/>
     <xacro:property name="Torso_Oz" value=" 0.0 "/>
     <xacro:property name="Torso_roll" value=" ${PI/2} "/>

File: repair_urdf/urdf/repair_full.urdf (robot description, URDF)
Before this commit: robot repair_full, 128 links, 127 joints
Joints:
- added joint j_torso_base: type fixed, parent sliding_guide_link, child dummy_prismatic_link, origin xyz=0.0 0.0 0.07 rpy=0.0 0.0 0.0, axis 0 0 1, limit lower=-0.8 upper=0.8 effort=147 velocity=0.35

File: repair_urdf/urdf/repair_torso_macro.urdf.xacro (robot description, xacro)
@@ -31,10 +31,10 @@
         <joint name="j_torso_base" type="fixed">
         <!-- <xacro:insert_block name="origin" /> -->
-        <origin rpy="0.0 0.0 0.0" xyz="0.0 0.0 0.0"/>
+        <origin rpy="0.0 0.0 0.0" xyz="0.0 0.0 0.07"/>
         <parent link="sliding_guide_link"/>
                 <child link="dummy_prismatic_link"/>
                 <axis xyz="0 0 1"/>
-        <limit lower="${j_prismatic_lower[0]/2}" upper= "${j_prismatic_upper[0]/2}" effort="${j_prismatic_torque[0]}" velocity="${j_prismatic_velocity[0]}"/>
-            </joint>
+        <limit effort="147" lower="-0.8" upper="0.8" velocity="0.35"/>
+        </joint>
         <!-- torso -->
         <joint name="j_torso_1" type="revolute">
