Commit message: modifications for new moveit library

File: repair_urdf/urdf/repair_torso_macro.urdf.xacro (robot description, xacro)
@@ -36,14 +36,20 @@
             <limit lower="${j_prismatic_lower[0]/2}" upper= "${j_prismatic_upper[0]/2}" effort="${j_prismatic_torque[0]}" velocity="${j_prismatic_velocity[0]}"/>
         </joint> -->
+        <joint name="j_torso_base" type="prismatic">
+        <!-- <xacro:insert_block name="origin" /> -->
+        <origin rpy="0.0 0.0 0.0" xyz="0.0 0.0 0.0"/>
+        <parent link="sliding_guide_link"/>
+                <child link="dummy_prismatic_link"/>
+                <axis xyz="0 0 1"/>
+        <limit effort="147" lower="-0.8" upper="0.8" velocity="2.2"/>
+            </joint>
         <!-- torso -->
-        <joint name="j_torso_1" type="fixed">
-            <parent link="dummy_prismatic_link" />
-            <child link="torso_1" />
-            <!-- <axis xyz="0 0 1" /> -->
-            <xacro:insert_block name="origin" />
-            <!-- <limit lower="${j_torso_lower[0]}" upper="${j_torso_upper[0]}"
-            effort="${j_torso_torque[0]}" velocity="${j_torso_velocity[0]}" /> -->
+        <joint name="j_torso_1" type="revolute">
+            <parent link="dummy_prismatic_link"/>
+            <child link="torso_1"/>
+            <axis xyz="0 0 1"/>
+            <origin rpy="1.570796326795 0.0 1.570796326795" xyz="0.0 0.0 0.0"/>
+            <limit effort="147.0" lower="-2.6" upper="2.6" velocity="2.0"/>
         </joint>
-        <!-- torso  -->
     </xacro:macro>
 </robot>

Commit message: working state after integration week 4

File: repair_urdf/urdf/repair_torso_macro.urdf.xacro (robot description, xacro)
@@ -36,6 +36,6 @@
             <limit lower="${j_prismatic_lower[0]/2}" upper= "${j_prismatic_upper[0]/2}" effort="${j_prismatic_torque[0]}" velocity="${j_prismatic_velocity[0]}"/>
         </joint> -->
-        <joint name="j_torso_base" type="prismatic">
-        <!-- <xacro:insert_block name="origin" /> -->
+        <!-- <joint name="j_torso_base" type="fixed">
+         <xacro:insert_block name="origin" />
         <origin rpy="0.0 0.0 0.0" xyz="0.0 0.0 0.0"/>
         <parent link="sliding_guide_link"/>
@@ -43,5 +43,5 @@
                 <axis xyz="0 0 1"/>
         <limit effort="147" lower="-0.8" upper="0.8" velocity="2.2"/>
-            </joint>
+            </joint> -->
         <!-- torso -->
         <joint name="j_torso_1" type="revolute">

Commit message: reinitialize pick and place class after ever try. fixed problem. still offset needs to be set without small pre movement

File: repair_urdf/urdf/repair_torso_macro.urdf.xacro (robot description, xacro)
@@ -29,5 +29,5 @@
             </collision>
         </link>
-        <joint name="j_torso_base" type="fixed">
+        <joint name="j_torso_base" type="prismatic">
         <!-- <xacro:insert_block name="origin" /> -->
         <origin rpy="0.0 0.0 0.0" xyz="0.0 0.0 0.07"/>
