Commit message: working loop state fridaz 5.04.2025

File: repair_urdf/urdf/repair_cage_macro.urdf.xacro (robot description, xacro)
@@ -2,4 +2,23 @@
 <robot xmlns:xacro="http://ros.org/wiki/xacro">
   <xacro:macro name="repair_cage" params="parent">
+  <link name="sand_bed_b1_link">
+    <visual>
+      <origin xyz="${Table_x} ${Table_y} ${Table_z+table_height+table_top_thickness/2}" />
+      <geometry>
+        <box size="2.0 0.035  0.035" />
+      </geometry>
+      <material name="wood" />
+    </visual>
+    <collision>
+      <origin xyz="${Table_x} ${Table_y} ${Table_z+table_height+table_top_thickness/2}" />
+      <geometry>
+        <box size="2.0 0.035  0.035" />
+      </geometry>
+    </collision>
+  </link>
+  <joint name="sand_bed_b1_joint" type="fixed" >
+    <parent link="table_top_link" />
+    <child link="sand_bed_b1_link" />
+  </joint>
   <link name="table_top_link">
     <visual>

File: repair_urdf/urdf/repair_full.urdf (robot description, URDF)
Before this commit: robot repair_full, 128 links, 128 joints
Joints:
- joint j_torso_1: limit (none) -> lower=-2.6 upper=2.6 effort=147.0 velocity=2.0

File: repair_urdf/urdf/repair_torso_macro.urdf.xacro (robot description, xacro)
@@ -35,5 +35,5 @@
                 <child link="dummy_prismatic_link"/>
                 <axis xyz="0 0 1"/>
-        <limit effort="147" lower="-0.8" upper="0.8" velocity="0.35"/>
+        <limit effort="147" lower="-0.8" upper="0.8" velocity="0.25"/>
         </joint>
         <!-- torso -->
