Commit message: adding some files to launch real frescos, adding repository for sdf files later

File: repair_urdf/urdf/RPf_00097.urdf (robot description, URDF)
Before this commit: robot frag2, 1 links, 0 joints
Links:
- removed link fragment_base_link
- added link RPf_00204_link, mass 0.5; collision mesh filename=package://repair_urdf/sdf/RPf_00097/RPf_00097.stl scale=0.001 0.001 0.001; visual mesh filename=package://repair_urdf/sdf/RPf_00097/RPf_00097.dae scale=0.001 0.001 0.001

File: repair_urdf/urdf/RPf_00204.urdf (robot description, URDF)
Before this commit: robot frag2, 1 links, 0 joints
Links:
- removed link fragment_base_link
- added link RPf_00204_link, mass 0.5; collision mesh filename=package://repair_urdf/sdf/test_frag/meshes/RPf_00204.stl scale=0.001 0.001 0.001; visual mesh filename=package://repair_urdf/sdf/test_frag/meshes/RPf_00204.dae scale=0.001 0.001 0.001

File: repair_urdf/urdf/RPf_00205.urdf (robot description, URDF)
Before this commit: robot frag2, 1 links, 0 joints
Links:
- removed link fragment_base_link
- added link RPf_00204_link, mass 0.5; collision mesh filename=package://repair_urdf/sdf/RPf_00205/RPf_00205.stl scale=0.001 0.001 0.001; visual mesh filename=package://repair_urdf/sdf/RPf_00205/RPf_00205.dae scale=0.001 0.001 0.001
