Commit message: gazebo depth cam to 1920x1080

File: repair_urdf/urdf/_l515.gazebo.xacro (robot description, xacro)
@@ -6,5 +6,6 @@
 -->
 <robot xmlns:xacro="http://ros.org/wiki/xacro">
-  <xacro:macro name="gazebo_l515" params="camera_name reference_link topics_ns depth_optical_frame color_optical_frame infrared_optical_frame publish_pointcloud:=true" >
+  <xacro:macro name="gazebo_l515"
+    params="camera_name reference_link topics_ns depth_optical_frame color_optical_frame infrared_optical_frame publish_pointcloud:=true" >
     <!-- Load parameters to model's main link-->
     <xacro:property name="deg_to_rad" value="0.01745329251994329577" />
@@ -71,6 +72,10 @@
           <horizontal_fov>${70*deg_to_rad}</horizontal_fov>
           <image>
-            <width>1024</width>
-            <height>768</height>
+            <!-- <width>1024</width>
+            <height>768</height> -->
+            <width>1920</width>
+            <height>1080</height>
+            <!-- <width>640</width>
+            <height>480</height> -->
           </image>
           <clip>
