Commit message: Gazebo adjustments, explicitly models and launch function for multi launch

File: repair_urdf/urdf/RPf_00205.urdf (robot description, URDF)
Before this commit: robot RPf_00204, 1 links, 0 joints
Links:
- removed link RPf_00204_link
- added link RPf_00205_link, mass 0.5; collision mesh filename=package://repair_urdf/sdf/RPf_00205/RPf_00205.stl scale=0.001 0.001 0.001; visual mesh filename=package://repair_urdf/sdf/RPf_00205/RPf_00205.dae scale=0.001 0.001 0.001
