Commit message: almost working demo, still problem with fragment dynamics and gazebo simulation time

File: repair_urdf/urdf/repair_full.urdf (robot description, URDF)
Before this commit: robot repair_full, 79 links, 78 joints
Links:
- removed link left_hand_v1s_index_distal_link
- removed link left_hand_v1s_index_knuckle_link
- removed link left_hand_v1s_index_middle_link
- removed link left_hand_v1s_index_proximal_link
- removed link left_hand_v1s_little_distal_link
- removed link left_hand_v1s_little_knuckle_link
- removed link left_hand_v1s_little_middle_link
- removed link left_hand_v1s_little_proximal_link
- removed link left_hand_v1s_middle_distal_link
- removed link left_hand_v1s_middle_knuckle_link
- removed link left_hand_v1s_middle_middle_link
- removed link left_hand_v1s_middle_proximal_link
- removed link left_hand_v1s_palm_base
- removed link left_hand_v1s_palm_link
- removed link left_hand_v1s_ring_distal_link
- removed link left_hand_v1s_ring_knuckle_link
- removed link left_hand_v1s_ring_middle_link
- removed link left_hand_v1s_ring_proximal_link
- removed link left_hand_v1s_thumb_distal_link
- removed link left_hand_v1s_thumb_knuckle_link
- removed link left_hand_v1s_thumb_proximal_link
- removed link right_hand_v1s_index_distal_link
- removed link right_hand_v1s_index_knuckle_link
- removed link right_hand_v1s_index_middle_link
- removed link right_hand_v1s_index_proximal_link
- removed link right_hand_v1s_little_distal_link
- removed link right_hand_v1s_little_knuckle_link
- removed link right_hand_v1s_little_middle_link
- removed link right_hand_v1s_little_proximal_link
- removed link right_hand_v1s_middle_distal_link
- removed link right_hand_v1s_middle_knuckle_link
- removed link right_hand_v1s_middle_middle_link
- removed link right_hand_v1s_middle_proximal_link
- removed link right_hand_v1s_palm_base
- removed link right_hand_v1s_palm_link
- removed link right_hand_v1s_ring_distal_link
- removed link right_hand_v1s_ring_knuckle_link
- removed link right_hand_v1s_ring_middle_link
- removed link right_hand_v1s_ring_proximal_link
- removed link right_hand_v1s_thumb_distal_link
- removed link right_hand_v1s_thumb_knuckle_link
- removed link right_hand_v1s_thumb_proximal_link
- added link left_hand_v2s_grasp_link, mass 0.1
- added link left_hand_v2s_index_distal_link, mass 0.005; collision mesh filename=package://softhands_description/meshes/softhands/v2.0/right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 scale=0.001 0.001 0.001; visual mesh filename=package://softhands_description/meshes/softhands/v2.0/right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 scale=0.001 0.001 0.001
- added link left_hand_v2s_index_knuckle_link, mass 0.009; collision mesh filename=package://softhands_description/meshes/softhands/v2.0/left/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 scale=0.001 0.001 0.001; visual mesh filename=package://softhands_description/meshes/softhands/v2.0/left/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 scale=0.001 0.001 0.001
- added link left_hand_v2s_index_middle_link, mass 0.005; collision mesh filename=package://softhands_description/meshes/softhands/v2.0/right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 scale=0.001 0.001 0.001; visual mesh filename=package://softhands_description/meshes/softhands/v2.0/right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 scale=0.001 0.001 0.001
- added link left_hand_v2s_index_proximal_link, mass 0.005; collision mesh filename=package://softhands_description/meshes/softhands/v2.0/right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 scale=0.001 0.001 0.001; visual mesh filename=package://softhands_description/meshes/softhands/v2.0/right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 scale=0.001 0.001 0.001
- added link left_hand_v2s_little_distal_link, mass 0.005; collision mesh filename=package://softhands_description/meshes/softhands/v2.0/right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 scale=0.001 0.001 0.001; visual mesh filename=package://softhands_description/meshes/softhands/v2.0/right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 scale=0.001 0.001 0.001
- added link left_hand_v2s_little_knuckle_link, mass 0.009; collision mesh filename=package://softhands_description/meshes/softhands/v2.0/left/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 scale=0.001 0.001 0.001; visual mesh filename=package://softhands_description/meshes/softhands/v2.0/left/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 scale=0.001 0.001 0.001
- added link left_hand_v2s_little_middle_link, mass 0.005; collision mesh filename=package://softhands_description/meshes/softhands/v2.0/right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 scale=0.001 0.001 0.001; visual mesh filename=package://softhands_description/meshes/softhands/v2.0/right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 scale=0.001 0.001 0.001
- added link left_hand_v2s_little_proximal_link, mass 0.005; collision mesh filename=package://softhands_description/meshes/softhands/v2.0/right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 scale=0.001 0.001 0.001; visual mesh filename=package://softhands_description/meshes/softhands/v2.0/right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 scale=0.001 0.001 0.001
- added link left_hand_v2s_middle_distal_link, mass 0.005; collision mesh filename=package://softhands_description/meshes/softhands/v2.0/right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 scale=0.001 0.001 0.001; visual mesh filename=package://softhands_description/meshes/softhands/v2.0/right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 scale=0.001 0.001 0.001
- added link left_hand_v2s_middle_knuckle_link, mass 0.009; collision mesh filename=package://softhands_description/meshes/softhands/v2.0/left/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 scale=0.001 0.001 0.001; visual mesh filename=package://softhands_description/meshes/softhands/v2.0/left/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 scale=0.001 0.001 0.001
- added link left_hand_v2s_middle_middle_link, mass 0.005; collision mesh filename=package://softhands_description/meshes/softhands/v2.0/right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 scale=0.001 0.001 0.001; visual mesh filename=package://softhands_description/meshes/softhands/v2.0/right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 scale=0.001 0.001 0.001
- added link left_hand_v2s_middle_proximal_link, mass 0.005; collision mesh filename=package://softhands_description/meshes/softhands/v2.0/right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 scale=0.001 0.001 0.001; visual mesh filename=package://softhands_description/meshes/softhands/v2.0/right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 scale=0.001 0.001 0.001
- added link left_hand_v2s_palm_base
- added link left_hand_v2s_palm_link, mass 0.266; collision mesh filename=package://softhands_description/meshes/softhands/v2.0/left/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 scale=0.001 0.001 0.001; visual mesh filename=package://softhands_description/meshes/softhands/v2.0/left/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 scale=0.001 0.001 0.001
- added link left_hand_v2s_ring_distal_link, mass 0.005; collision mesh filename=package://softhands_description/meshes/softhands/v2.0/right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 scale=0.001 0.001 0.001; visual mesh filename=package://softhands_description/meshes/softhands/v2.0/right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 scale=0.001 0.001 0.001
- added link left_hand_v2s_ring_knuckle_link, mass 0.009; collision mesh filename=package://softhands_description/meshes/softhands/v2.0/left/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 scale=0.001 0.001 0.001; visual mesh filename=package://softhands_description/meshes/softhands/v2.0/left/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 scale=0.001 0.001 0.001
- added link left_hand_v2s_ring_middle_link, mass 0.005; collision mesh filename=package://softhands_description/meshes/softhands/v2.0/right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 scale=0.001 0.001 0.001; visual mesh filename=package://softhands_description/meshes/softhands/v2.0/right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 scale=0.001 0.001 0.001
- added link left_hand_v2s_ring_proximal_link, mass 0.005; collision mesh filename=package://softhands_description/meshes/softhands/v2.0/right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 scale=0.001 0.001 0.001; visual mesh filename=package://softhands_description/meshes/softhands/v2.0/right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 scale=0.001 0.001 0.001
- added link left_hand_v2s_synergy_link, mass 0.1
- added link left_hand_v2s_thumb_distal_link, mass 0.05; collision mesh filename=package://softhands_description/meshes/softhands/v2.0/right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 scale=0.001 0.001 0.001; visual mesh filename=package://softhands_description/meshes/softhands/v2.0/right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 scale=0.001 0.001 0.001
- added link left_hand_v2s_thumb_knuckle_link, mass 0.009; collision mesh filename=package://softhands_description/meshes/softhands/v2.0/left/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 scale=0.001 0.001 0.001; visual mesh filename=package://softhands_description/meshes/softhands/v2.0/left/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 scale=0.001 0.001 0.001
- added link left_hand_v2s_thumb_proximal_link, mass 0.05; collision mesh filename=package://softhands_description/meshes/softhands/v2.0/right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 scale=0.001 0.001 0.001; visual mesh filename=package://softhands_description/meshes/softhands/v2.0/right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 scale=0.001 0.001 0.001
- added link right_hand_v2s_grasp_link, mass 0.1
- added link right_hand_v2s_index_distal_link, mass 0.005; collision mesh filename=package://softhands_description/meshes/softhands/v2.0/right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 scale=0.001 0.001 0.001; visual mesh filename=package://softhands_description/meshes/softhands/v2.0/right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 scale=0.001 0.001 0.001
- added link right_hand_v2s_index_knuckle_link, mass 0.009; collision mesh filename=package://softhands_description/meshes/softhands/v2.0/right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 scale=0.001 0.001 0.001; visual mesh filename=package://softhands_description/meshes/softhands/v2.0/right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 scale=0.001 0.001 0.001
- added link right_hand_v2s_index_middle_link, mass 0.005; collision mesh filename=package://softhands_description/meshes/softhands/v2.0/right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 scale=0.001 0.001 0.001; visual mesh filename=package://softhands_description/meshes/softhands/v2.0/right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 scale=0.001 0.001 0.001
- added link right_hand_v2s_index_proximal_link, mass 0.005; collision mesh filename=package://softhands_description/meshes/softhands/v2.0/right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 scale=0.001 0.001 0.001; visual mesh filename=package://softhands_description/meshes/softhands/v2.0/right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 scale=0.001 0.001 0.001
- added link right_hand_v2s_little_distal_link, mass 0.005; collision mesh filename=package://softhands_description/meshes/softhands/v2.0/right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 scale=0.001 0.001 0.001; visual mesh filename=package://softhands_description/meshes/softhands/v2.0/right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 scale=0.001 0.001 0.001
- added link right_hand_v2s_little_knuckle_link, mass 0.009; collision mesh filename=package://softhands_description/meshes/softhands/v2.0/right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 scale=0.001 0.001 0.001; visual mesh filename=package://softhands_description/meshes/softhands/v2.0/right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 scale=0.001 0.001 0.001
- added link right_hand_v2s_little_middle_link, mass 0.005; collision mesh filename=package://softhands_description/meshes/softhands/v2.0/right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 scale=0.001 0.001 0.001; visual mesh filename=package://softhands_description/meshes/softhands/v2.0/right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 scale=0.001 0.001 0.001
- added link right_hand_v2s_little_proximal_link, mass 0.005; collision mesh filename=package://softhands_description/meshes/softhands/v2.0/right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 scale=0.001 0.001 0.001; visual mesh filename=package://softhands_description/meshes/softhands/v2.0/right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 scale=0.001 0.001 0.001
- added link right_hand_v2s_middle_distal_link, mass 0.005; collision mesh filename=package://softhands_description/meshes/softhands/v2.0/right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 scale=0.001 0.001 0.001; visual mesh filename=package://softhands_description/meshes/softhands/v2.0/right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 scale=0.001 0.001 0.001
- added link right_hand_v2s_middle_knuckle_link, mass 0.009; collision mesh filename=package://softhands_description/meshes/softhands/v2.0/right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 scale=0.001 0.001 0.001; visual mesh filename=package://softhands_description/meshes/softhands/v2.0/right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 scale=0.001 0.001 0.001
- added link right_hand_v2s_middle_middle_link, mass 0.005; collision mesh filename=package://softhands_description/meshes/softhands/v2.0/right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 scale=0.001 0.001 0.001; visual mesh filename=package://softhands_description/meshes/softhands/v2.0/right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 scale=0.001 0.001 0.001
- added link right_hand_v2s_middle_proximal_link, mass 0.005; collision mesh filename=package://softhands_description/meshes/softhands/v2.0/right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 scale=0.001 0.001 0.001; visual mesh filename=package://softhands_description/meshes/softhands/v2.0/right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 scale=0.001 0.001 0.001
- added link right_hand_v2s_palm_base
- added link right_hand_v2s_palm_link, mass 0.266; collision mesh filename=package://softhands_description/meshes/softhands/v2.0/right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 scale=0.001 0.001 0.001; visual mesh filename=package://softhands_description/meshes/softhands/v2.0/right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 scale=0.001 0.001 0.001
- added link right_hand_v2s_ring_distal_link, mass 0.005; collision mesh filename=package://softhands_description/meshes/softhands/v2.0/right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 scale=0.001 0.001 0.001; visual mesh filename=package://softhands_description/meshes/softhands/v2.0/right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 scale=0.001 0.001 0.001
- added link right_hand_v2s_ring_knuckle_link, mass 0.009; collision mesh filename=package://softhands_description/meshes/softhands/v2.0/right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 scale=0.001 0.001 0.001; visual mesh filename=package://softhands_description/meshes/softhands/v2.0/right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 scale=0.001 0.001 0.001
- added link right_hand_v2s_ring_middle_link, mass 0.005; collision mesh filename=package://softhands_description/meshes/softhands/v2.0/right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 scale=0.001 0.001 0.001; visual mesh filename=package://softhands_description/meshes/softhands/v2.0/right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 scale=0.001 0.001 0.001
- added link right_hand_v2s_ring_proximal_link, mass 0.005; collision mesh filename=package://softhands_description/meshes/softhands/v2.0/right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 scale=0.001 0.001 0.001; visual mesh filename=package://softhands_description/meshes/softhands/v2.0/right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 scale=0.001 0.001 0.001
- added link right_hand_v2s_synergy_link, mass 0.1
- added link right_hand_v2s_thumb_distal_link, mass 0.05; collision mesh filename=package://softhands_description/meshes/softhands/v2.0/right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 scale=0.001 0.001 0.001; visual mesh filename=package://softhands_description/meshes/softhands/v2.0/right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 scale=0.001 0.001 0.001
- added link right_hand_v2s_thumb_knuckle_link, mass 0.009; collision mesh filename=package://softhands_description/meshes/softhands/v2.0/right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 scale=0.001 0.001 0.001; visual mesh filename=package://softhands_description/meshes/softhands/v2.0/right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 scale=0.001 0.001 0.001
- added link right_hand_v2s_thumb_proximal_link, mass 0.05; collision mesh filename=package://softhands_description/meshes/softhands/v2.0/right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 scale=0.001 0.001 0.001; visual mesh filename=package://softhands_description/meshes/softhands/v2.0/right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 scale=0.001 0.001 0.001
Joints:
- removed joint left_hand_base_joint
- removed joint left_hand_v1s_index_distal_joint
- removed joint left_hand_v1s_index_knuckle_joint
- removed joint left_hand_v1s_index_middle_joint
- removed joint left_hand_v1s_index_proximal_joint
- removed joint left_hand_v1s_little_distal_joint
- removed joint left_hand_v1s_little_knuckle_joint
- removed joint left_hand_v1s_little_middle_joint
- removed joint left_hand_v1s_little_proximal_joint
- removed joint left_hand_v1s_middle_distal_joint
- removed joint left_hand_v1s_middle_knuckle_joint
- removed joint left_hand_v1s_middle_middle_joint
- removed joint left_hand_v1s_middle_proximal_joint
- removed joint left_hand_v1s_palm_joint
- removed joint left_hand_v1s_ring_distal_joint
- removed joint left_hand_v1s_ring_knuckle_joint
- removed joint left_hand_v1s_ring_middle_joint
- removed joint left_hand_v1s_ring_proximal_joint
- removed joint left_hand_v1s_thumb_distal_joint
- removed joint left_hand_v1s_thumb_knuckle_joint
- removed joint left_hand_v1s_thumb_proximal_joint
- removed joint right_hand_base_joint
- removed joint right_hand_v1s_index_distal_joint
- removed joint right_hand_v1s_index_knuckle_joint
- removed joint right_hand_v1s_index_middle_joint
- removed joint right_hand_v1s_index_proximal_joint
- removed joint right_hand_v1s_little_distal_joint
- removed joint right_hand_v1s_little_knuckle_joint
- removed joint right_hand_v1s_little_middle_joint
- removed joint right_hand_v1s_little_proximal_joint
- removed joint right_hand_v1s_middle_distal_joint
- removed joint right_hand_v1s_middle_knuckle_joint
- removed joint right_hand_v1s_middle_middle_joint
- removed joint right_hand_v1s_middle_proximal_joint
- removed joint right_hand_v1s_palm_joint
- removed joint right_hand_v1s_ring_distal_joint
- removed joint right_hand_v1s_ring_knuckle_joint
- removed joint right_hand_v1s_ring_middle_joint
- removed joint right_hand_v1s_ring_proximal_joint
- removed joint right_hand_v1s_thumb_distal_joint
- removed joint right_hand_v1s_thumb_knuckle_joint
- removed joint right_hand_v1s_thumb_proximal_joint
- added joint left_hand_v2s_base_joint: type fixed, parent arm_2_link_7, child left_hand_v2s_palm_base, origin xyz=0 -0.013900 -0.015 rpy=0 0 0
- added joint left_hand_v2s_grasp_joint: type fixed, parent left_hand_v2s_palm_base, child left_hand_v2s_grasp_link, origin xyz=0 0 0.07 rpy=0 0 0
- added joint left_hand_v2s_index_distal_joint: type revolute, parent left_hand_v2s_index_middle_link, child left_hand_v2s_index_distal_link, origin xyz=0.022 0 0 rpy=0 0 0, axis 0 0 1, limit lower=-0.785398 upper=1.57 effort=30 velocity=1.0, mimic joint=left_hand_v2s_synergy_joint multiplier=0.7853981633974483
- added joint left_hand_v2s_index_knuckle_joint: type revolute, parent left_hand_v2s_palm_link, child left_hand_v2s_index_knuckle_link, origin xyz=0.099 0.0255 0.00766056 rpy=0 0 0.1745327, axis 0 0 1, limit lower=-0.1 upper=0.1 effort=30 velocity=1.0, mimic joint=left_hand_v2s_synergy_joint multiplier=-0.2
- added joint left_hand_v2s_index_middle_joint: type revolute, parent left_hand_v2s_index_proximal_link, child left_hand_v2s_index_middle_link, origin xyz=0.022 0 0 rpy=0 0 0, axis 0 0 1, limit lower=-0.785398 upper=1.57 effort=30 velocity=1.0, mimic joint=left_hand_v2s_synergy_joint multiplier=0.7853981633974483
- added joint left_hand_v2s_index_proximal_joint: type revolute, parent left_hand_v2s_index_knuckle_link, child left_hand_v2s_index_proximal_link, origin xyz=0.0211 0.0023 0 rpy=1.5707963 0 0, axis 0 0 1, limit lower=-0.785398 upper=1.57 effort=30 velocity=1.0, mimic joint=left_hand_v2s_synergy_joint multiplier=0.7853981633974483
- added joint left_hand_v2s_little_distal_joint: type revolute, parent left_hand_v2s_little_middle_link, child left_hand_v2s_little_distal_link, origin xyz=0.022 0 0 rpy=0 0 0, axis 0 0 1, limit lower=-0.785398 upper=1.57 effort=30 velocity=1.0, mimic joint=left_hand_v2s_synergy_joint multiplier=0.7853981633974483
- added joint left_hand_v2s_little_knuckle_joint: type revolute, parent left_hand_v2s_palm_link, child left_hand_v2s_little_knuckle_link, origin xyz=0.094 -0.0257 0.00766056 rpy=0 0 -0.2617993, axis 0 0 1, limit lower=-0.1 upper=0.1 effort=30 velocity=1.0, mimic joint=left_hand_v2s_synergy_joint multiplier=0.4
- added joint left_hand_v2s_little_middle_joint: type revolute, parent left_hand_v2s_little_proximal_link, child left_hand_v2s_little_middle_link, origin xyz=0.022 0 0 rpy=0 0 0, axis 0 0 1, limit lower=-0.785398 upper=1.57 effort=30 velocity=1.0, mimic joint=left_hand_v2s_synergy_joint multiplier=0.7853981633974483
- added joint left_hand_v2s_little_proximal_joint: type revolute, parent left_hand_v2s_little_knuckle_link, child left_hand_v2s_little_proximal_link, origin xyz=0.0211 -0.0023 0 rpy=1.5707963 0 0, axis 0 0 1, limit lower=-0.785398 upper=1.57 effort=30 velocity=1.0, mimic joint=left_hand_v2s_synergy_joint multiplier=0.7853981633974483
- added joint left_hand_v2s_middle_distal_joint: type revolute, parent left_hand_v2s_middle_middle_link, child left_hand_v2s_middle_distal_link, origin xyz=0.022 0 0 rpy=0 0 0, axis 0 0 1, limit lower=-0.785398 upper=1.57 effort=30 velocity=1.0, mimic joint=left_hand_v2s_synergy_joint multiplier=0.7853981633974483
- added joint left_hand_v2s_middle_knuckle_joint: type revolute, parent left_hand_v2s_palm_link, child left_hand_v2s_middle_knuckle_link, origin xyz=0.104 0.0075 0.00766056 rpy=0.0 0.0 0.0, axis 0 0 1, limit lower=-0.1 upper=0.1 effort=30 velocity=1.0, mimic joint=left_hand_v2s_synergy_joint multiplier=0.0
- added joint left_hand_v2s_middle_middle_joint: type revolute, parent left_hand_v2s_middle_proximal_link, child left_hand_v2s_middle_middle_link, origin xyz=0.022 0 0 rpy=0 0 0, axis 0 0 1, limit lower=-0.785398 upper=1.57 effort=30 velocity=1.0, mimic joint=left_hand_v2s_synergy_joint multiplier=0.7853981633974483
- added joint left_hand_v2s_middle_proximal_joint: type revolute, parent left_hand_v2s_middle_knuckle_link, child left_hand_v2s_middle_proximal_link, origin xyz=0.0211 0.0 0 rpy=1.5707963 0 0, axis 0 0 1, limit lower=-0.785398 upper=1.57 effort=30 velocity=1.0, mimic joint=left_hand_v2s_synergy_joint multiplier=0.7853981633974483
- added joint left_hand_v2s_palm_joint: type fixed, parent left_hand_v2s_palm_base, child left_hand_v2s_palm_link, origin xyz=0 0 0.00 rpy=0 -1.57 3.14159
- added joint left_hand_v2s_ring_distal_joint: type revolute, parent left_hand_v2s_ring_middle_link, child left_hand_v2s_ring_distal_link, origin xyz=0.022 0 0 rpy=0 0 0, axis 0 0 1, limit lower=-0.785398 upper=1.57 effort=30 velocity=1.0, mimic joint=left_hand_v2s_synergy_joint multiplier=0.7853981633974483
- added joint left_hand_v2s_ring_knuckle_joint: type revolute, parent left_hand_v2s_palm_link, child left_hand_v2s_ring_knuckle_link, origin xyz=0.099 -0.0105 0.00766056 rpy=0 0 -0.0872667 , axis 0 0 1, limit lower=-0.1 upper=0.1 effort=30 velocity=1.0, mimic joint=left_hand_v2s_synergy_joint multiplier=0.2
- added joint left_hand_v2s_ring_middle_joint: type revolute, parent left_hand_v2s_ring_proximal_link, child left_hand_v2s_ring_middle_link, origin xyz=0.022 0 0 rpy=0 0 0, axis 0 0 1, limit lower=-0.785398 upper=1.57 effort=30 velocity=1.0, mimic joint=left_hand_v2s_synergy_joint multiplier=0.7853981633974483
- added joint left_hand_v2s_ring_proximal_joint: type revolute, parent left_hand_v2s_ring_knuckle_link, child left_hand_v2s_ring_proximal_link, origin xyz=0.0211 -0.0023 0 rpy=1.5707963 0 0, axis 0 0 1, limit lower=-0.785398 upper=1.57 effort=30 velocity=1.0, mimic joint=left_hand_v2s_synergy_joint multiplier=0.7853981633974483
- added joint left_hand_v2s_synergy_joint: type revolute, parent left_hand_v2s_palm_link, child left_hand_v2s_synergy_link, axis 0 0 1, limit lower=0.0 upper=1.0 effort=100 velocity=100000
- added joint left_hand_v2s_thumb_distal_joint: type revolute, parent left_hand_v2s_thumb_proximal_link, child left_hand_v2s_thumb_distal_link, origin xyz=0.022 0 0 rpy=0 0 0.3, axis 0 0 1, limit lower=-0.785398 upper=1.57 effort=30 velocity=1.0, mimic joint=left_hand_v2s_synergy_joint multiplier=0.7853981633974483
- added joint left_hand_v2s_thumb_knuckle_joint: type revolute, parent left_hand_v2s_palm_link, child left_hand_v2s_thumb_knuckle_link, origin xyz=0.06643 0.0437097 0.0210 rpy=1.5707963 0 1.0471971, axis 0 0 1, limit lower=0 upper=1.57 effort=30 velocity=1.0, mimic joint=left_hand_v2s_synergy_joint multiplier=2.0420352248333655
- added joint left_hand_v2s_thumb_proximal_joint: type revolute, parent left_hand_v2s_thumb_knuckle_link, child left_hand_v2s_thumb_proximal_link, origin xyz=0.0235 0.00343074 0.00392231  rpy=1.4819366 -0.3 0, axis 0 0 1, limit lower=-0.785398 upper=1.57 effort=30 velocity=1.0, mimic joint=left_hand_v2s_synergy_joint multiplier=1.0210176124166828
- added joint right_hand_v2s_base_joint: type fixed, parent arm_1_link_7, child right_hand_v2s_palm_base, origin xyz=0 0 -0.015 rpy=0 0.0 3.14159265359
- added joint right_hand_v2s_grasp_joint: type fixed, parent right_hand_v2s_palm_base, child right_hand_v2s_grasp_link, origin xyz=0 0 0.07 rpy=0 0 0
- added joint right_hand_v2s_index_distal_joint: type revolute, parent right_hand_v2s_index_middle_link, child right_hand_v2s_index_distal_link, origin xyz=0.022 0 0 rpy=0 0 0, axis 0 0 1, limit lower=-0.785398 upper=1.57 effort=30 velocity=1.0, mimic joint=right_hand_v2s_synergy_joint multiplier=0.7853981633974483
- added joint right_hand_v2s_index_knuckle_joint: type revolute, parent right_hand_v2s_palm_link, child right_hand_v2s_index_knuckle_link, origin xyz=0.099 -0.0255 0.00766056 rpy=0 0 -0.1745327, axis 0 0 1, limit lower=-0.1 upper=0.1 effort=30 velocity=1.0, mimic joint=right_hand_v2s_synergy_joint multiplier=-0.2
- added joint right_hand_v2s_index_middle_joint: type revolute, parent right_hand_v2s_index_proximal_link, child right_hand_v2s_index_middle_link, origin xyz=0.022 0 0 rpy=0 0 0, axis 0 0 1, limit lower=-0.785398 upper=1.57 effort=30 velocity=1.0, mimic joint=right_hand_v2s_synergy_joint multiplier=0.7853981633974483
- added joint right_hand_v2s_index_proximal_joint: type revolute, parent right_hand_v2s_index_knuckle_link, child right_hand_v2s_index_proximal_link, origin xyz=0.0211 0.0023 0 rpy=1.5707963 0 0, axis 0 0 1, limit lower=-0.785398 upper=1.57 effort=30 velocity=1.0, mimic joint=right_hand_v2s_synergy_joint multiplier=0.7853981633974483
- added joint right_hand_v2s_little_distal_joint: type revolute, parent right_hand_v2s_little_middle_link, child right_hand_v2s_little_distal_link, origin xyz=0.022 0 0 rpy=0 0 0, axis 0 0 1, limit lower=-0.785398 upper=1.57 effort=30 velocity=1.0, mimic joint=right_hand_v2s_synergy_joint multiplier=0.7853981633974483
- added joint right_hand_v2s_little_knuckle_joint: type revolute, parent right_hand_v2s_palm_link, child right_hand_v2s_little_knuckle_link, origin xyz=0.094 0.0257 0.00766056 rpy=0 0 0.2617993, axis 0 0 1, limit lower=-0.1 upper=0.1 effort=30 velocity=1.0, mimic joint=right_hand_v2s_synergy_joint multiplier=0.4
- added joint right_hand_v2s_little_middle_joint: type revolute, parent right_hand_v2s_little_proximal_link, child right_hand_v2s_little_middle_link, origin xyz=0.022 0 0 rpy=0 0 0, axis 0 0 1, limit lower=-0.785398 upper=1.57 effort=30 velocity=1.0, mimic joint=right_hand_v2s_synergy_joint multiplier=0.7853981633974483
- added joint right_hand_v2s_little_proximal_joint: type revolute, parent right_hand_v2s_little_knuckle_link, child right_hand_v2s_little_proximal_link, origin xyz=0.0211 -0.0023 0 rpy=1.5707963 0 0, axis 0 0 1, limit lower=-0.785398 upper=1.57 effort=30 velocity=1.0, mimic joint=right_hand_v2s_synergy_joint multiplier=0.7853981633974483
- added joint right_hand_v2s_middle_distal_joint: type revolute, parent right_hand_v2s_middle_middle_link, child right_hand_v2s_middle_distal_link, origin xyz=0.022 0 0 rpy=0 0 0, axis 0 0 1, limit lower=-0.785398 upper=1.57 effort=30 velocity=1.0, mimic joint=right_hand_v2s_synergy_joint multiplier=0.7853981633974483
- added joint right_hand_v2s_middle_knuckle_joint: type revolute, parent right_hand_v2s_palm_link, child right_hand_v2s_middle_knuckle_link, origin xyz=0.104 -0.0075 0.00766056 rpy=0.0 0.0 0.0, axis 0 0 1, limit lower=-0.1 upper=0.1 effort=30 velocity=1.0, mimic joint=right_hand_v2s_synergy_joint multiplier=0.0
- added joint right_hand_v2s_middle_middle_joint: type revolute, parent right_hand_v2s_middle_proximal_link, child right_hand_v2s_middle_middle_link, origin xyz=0.022 0 0 rpy=0 0 0, axis 0 0 1, limit lower=-0.785398 upper=1.57 effort=30 velocity=1.0, mimic joint=right_hand_v2s_synergy_joint multiplier=0.7853981633974483
- added joint right_hand_v2s_middle_proximal_joint: type revolute, parent right_hand_v2s_middle_knuckle_link, child right_hand_v2s_middle_proximal_link, origin xyz=0.0211 0.0 0 rpy=1.5707963 0 0, axis 0 0 1, limit lower=-0.785398 upper=1.57 effort=30 velocity=1.0, mimic joint=right_hand_v2s_synergy_joint multiplier=0.7853981633974483
- added joint right_hand_v2s_palm_joint: type fixed, parent right_hand_v2s_palm_base, child right_hand_v2s_palm_link, origin xyz=0 0 0.00 rpy=0 -1.57 3.14159
- added joint right_hand_v2s_ring_distal_joint: type revolute, parent right_hand_v2s_ring_middle_link, child right_hand_v2s_ring_distal_link, origin xyz=0.022 0 0 rpy=0 0 0, axis 0 0 1, limit lower=-0.785398 upper=1.57 effort=30 velocity=1.0, mimic joint=right_hand_v2s_synergy_joint multiplier=0.7853981633974483
- added joint right_hand_v2s_ring_knuckle_joint: type revolute, parent right_hand_v2s_palm_link, child right_hand_v2s_ring_knuckle_link, origin xyz=0.099 0.0105 0.00766056 rpy=0 0 0.0872664, axis 0 0 1, limit lower=-0.1 upper=0.1 effort=30 velocity=1.0, mimic joint=right_hand_v2s_synergy_joint multiplier=0.2
- added joint right_hand_v2s_ring_middle_joint: type revolute, parent right_hand_v2s_ring_proximal_link, child right_hand_v2s_ring_middle_link, origin xyz=0.022 0 0 rpy=0 0 0, axis 0 0 1, limit lower=-0.785398 upper=1.57 effort=30 velocity=1.0, mimic joint=right_hand_v2s_synergy_joint multiplier=0.7853981633974483
- added joint right_hand_v2s_ring_proximal_joint: type revolute, parent right_hand_v2s_ring_knuckle_link, child right_hand_v2s_ring_proximal_link, origin xyz=0.0211 -0.0023 0 rpy=1.5707963 0 0, axis 0 0 1, limit lower=-0.785398 upper=1.57 effort=30 velocity=1.0, mimic joint=right_hand_v2s_synergy_joint multiplier=0.7853981633974483
- added joint right_hand_v2s_synergy_joint: type revolute, parent right_hand_v2s_palm_link, child right_hand_v2s_synergy_link, axis 0 0 1, limit lower=0.0 upper=1.0 effort=100 velocity=100000
- added joint right_hand_v2s_thumb_distal_joint: type revolute, parent right_hand_v2s_thumb_proximal_link, child right_hand_v2s_thumb_distal_link, origin xyz=0.022 0 0 rpy=0 0 0.3, axis 0 0 1, limit lower=-0.785398 upper=1.57 effort=30 velocity=1.0, mimic joint=right_hand_v2s_synergy_joint multiplier=0.7853981633974483
- added joint right_hand_v2s_thumb_knuckle_joint: type revolute, parent right_hand_v2s_palm_link, child right_hand_v2s_thumb_knuckle_link, origin xyz=0.06643 -0.0437097 0.0210 rpy=-1.5707963 -0.7 -1.0471972, axis 0 0 -1, limit lower=0 upper=1.57 effort=30 velocity=1.0, mimic joint=right_hand_v2s_synergy_joint multiplier=2.0420352248333655
- added joint right_hand_v2s_thumb_proximal_joint: type revolute, parent right_hand_v2s_thumb_knuckle_link, child right_hand_v2s_thumb_proximal_link, origin xyz=0.0235 -0.00343074 0.00392231  rpy=1.6580634 -0.3 0, axis 0 0 1, limit lower=-0.785398 upper=1.57 effort=30 velocity=1.0, mimic joint=right_hand_v2s_synergy_joint multiplier=1.0210176124166828
