Commit message: works up to real grasping

File: repair_urdf/urdf/repair_full.urdf (robot description, URDF)
Before this commit: robot repair_full, 83 links, 82 joints
Joints:
- joint left_hand_v2s_grasp_joint: origin xyz=0 0 0.07 rpy=0 0 0 -> xyz=0 0 0.09 rpy=0 0 0
- joint right_hand_v2s_grasp_joint: origin xyz=0 0 0.07 rpy=0 0 0 -> xyz=0 0 0.09 rpy=0 0 0
- joint right_hand_v2s_index_distal_joint: mimic joint=right_hand_v2s_synergy_joint multiplier=0.7853981633974483 -> joint=right_hand_v2s_synergy_joint multiplier=1.0
- joint right_hand_v2s_index_knuckle_joint: mimic joint=right_hand_v2s_synergy_joint multiplier=-0.2 -> joint=right_hand_v2s_synergy_joint multiplier=1.0
- joint right_hand_v2s_index_middle_joint: mimic joint=right_hand_v2s_synergy_joint multiplier=0.7853981633974483 -> joint=right_hand_v2s_synergy_joint multiplier=1.0
- joint right_hand_v2s_index_proximal_joint: mimic joint=right_hand_v2s_synergy_joint multiplier=0.7853981633974483 -> joint=right_hand_v2s_synergy_joint multiplier=1.0
- joint right_hand_v2s_little_distal_joint: mimic joint=right_hand_v2s_synergy_joint multiplier=0.7853981633974483 -> joint=right_hand_v2s_synergy_joint multiplier=1.0
- joint right_hand_v2s_little_knuckle_joint: mimic joint=right_hand_v2s_synergy_joint multiplier=0.4 -> joint=right_hand_v2s_synergy_joint multiplier=1.0
- joint right_hand_v2s_little_middle_joint: mimic joint=right_hand_v2s_synergy_joint multiplier=0.7853981633974483 -> joint=right_hand_v2s_synergy_joint multiplier=1.0
- joint right_hand_v2s_little_proximal_joint: mimic joint=right_hand_v2s_synergy_joint multiplier=0.7853981633974483 -> joint=right_hand_v2s_synergy_joint multiplier=1.0
- joint right_hand_v2s_middle_distal_joint: mimic joint=right_hand_v2s_synergy_joint multiplier=0.7853981633974483 -> joint=right_hand_v2s_synergy_joint multiplier=1.0
- joint right_hand_v2s_middle_knuckle_joint: mimic joint=right_hand_v2s_synergy_joint multiplier=0.0 -> joint=right_hand_v2s_synergy_joint multiplier=1.0
- joint right_hand_v2s_middle_middle_joint: mimic joint=right_hand_v2s_synergy_joint multiplier=0.7853981633974483 -> joint=right_hand_v2s_synergy_joint multiplier=1.0
- joint right_hand_v2s_middle_proximal_joint: mimic joint=right_hand_v2s_synergy_joint multiplier=0.7853981633974483 -> joint=right_hand_v2s_synergy_joint multiplier=1.0
- joint right_hand_v2s_ring_distal_joint: mimic joint=right_hand_v2s_synergy_joint multiplier=0.7853981633974483 -> joint=right_hand_v2s_synergy_joint multiplier=1.0
- joint right_hand_v2s_ring_knuckle_joint: mimic joint=right_hand_v2s_synergy_joint multiplier=0.2 -> joint=right_hand_v2s_synergy_joint multiplier=1.0
- joint right_hand_v2s_ring_middle_joint: mimic joint=right_hand_v2s_synergy_joint multiplier=0.7853981633974483 -> joint=right_hand_v2s_synergy_joint multiplier=1.0
- joint right_hand_v2s_ring_proximal_joint: mimic joint=right_hand_v2s_synergy_joint multiplier=0.7853981633974483 -> joint=right_hand_v2s_synergy_joint multiplier=1.0
- joint right_hand_v2s_thumb_distal_joint: mimic joint=right_hand_v2s_synergy_joint multiplier=0.7853981633974483 -> joint=right_hand_v2s_synergy_joint multiplier=1.0
- joint right_hand_v2s_thumb_knuckle_joint: mimic joint=right_hand_v2s_synergy_joint multiplier=2.0420352248333655 -> joint=right_hand_v2s_synergy_joint multiplier=1.0
- joint right_hand_v2s_thumb_proximal_joint: mimic joint=right_hand_v2s_synergy_joint multiplier=1.0210176124166828 -> joint=right_hand_v2s_synergy_joint multiplier=1.0
