Commit message: added new urdf version of arm and tried to use moveit; Bug: controller not stiff for initila gazebo pose

File: repair_urdf/urdf/repair_full.urdf (robot description, URDF)
Before this commit: robot repair_full, 83 links, 82 joints
Links:
- removed link left_hand_v2s_grasp_link
- removed link left_hand_v2s_index_distal_link
- removed link left_hand_v2s_index_knuckle_link
- removed link left_hand_v2s_index_middle_link
- removed link left_hand_v2s_index_proximal_link
- removed link left_hand_v2s_little_distal_link
- removed link left_hand_v2s_little_knuckle_link
- removed link left_hand_v2s_little_middle_link
- removed link left_hand_v2s_little_proximal_link
- removed link left_hand_v2s_middle_distal_link
- removed link left_hand_v2s_middle_knuckle_link
- removed link left_hand_v2s_middle_middle_link
- removed link left_hand_v2s_middle_proximal_link
- removed link left_hand_v2s_palm_base
- removed link left_hand_v2s_palm_link
- removed link left_hand_v2s_ring_distal_link
- removed link left_hand_v2s_ring_knuckle_link
- removed link left_hand_v2s_ring_middle_link
- removed link left_hand_v2s_ring_proximal_link
- removed link left_hand_v2s_synergy_link
- removed link left_hand_v2s_thumb_distal_link
- removed link left_hand_v2s_thumb_knuckle_link
- removed link left_hand_v2s_thumb_proximal_link
- removed link right_hand_v2s_grasp_link
- removed link right_hand_v2s_index_distal_link
- removed link right_hand_v2s_index_knuckle_link
- removed link right_hand_v2s_index_middle_link
- removed link right_hand_v2s_index_proximal_link
- removed link right_hand_v2s_little_distal_link
- removed link right_hand_v2s_little_knuckle_link
- removed link right_hand_v2s_little_middle_link
- removed link right_hand_v2s_little_proximal_link
- removed link right_hand_v2s_middle_distal_link
- removed link right_hand_v2s_middle_knuckle_link
- removed link right_hand_v2s_middle_middle_link
- removed link right_hand_v2s_middle_proximal_link
- removed link right_hand_v2s_palm_base
- removed link right_hand_v2s_palm_link
- removed link right_hand_v2s_ring_distal_link
- removed link right_hand_v2s_ring_knuckle_link
- removed link right_hand_v2s_ring_middle_link
- removed link right_hand_v2s_ring_proximal_link
- removed link right_hand_v2s_synergy_link
- removed link right_hand_v2s_thumb_distal_link
- removed link right_hand_v2s_thumb_knuckle_link
- removed link right_hand_v2s_thumb_proximal_link
- added link left_hand_v1s_grasp_link, mass 0.1
- added link left_hand_v1s_index_distal_link, mass 0.1; collision mesh filename=package://softhands_description/meshes/softhands/v1.0/commo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; visual mesh filename=package://softhands_description/meshes/softhands/v1.0/commo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
- added link left_hand_v1s_index_knuckle_link, mass 0.09; collision mesh filename=package://softhands_description/meshes/softhands/v1.0/commo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; visual mesh filename=package://softhands_description/meshes/softhands/v1.0/commo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
- added link left_hand_v1s_index_middle_link, mass 0.05; collision mesh filename=package://softhands_description/meshes/softhands/v1.0/commo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; visual mesh filename=package://softhands_description/meshes/softhands/v1.0/commo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
- added link left_hand_v1s_index_proximal_link, mass 0.05; collision mesh filename=package://softhands_description/meshes/softhands/v1.0/commo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; visual mesh filename=package://softhands_description/meshes/softhands/v1.0/commo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
- added link left_hand_v1s_little_distal_link, mass 0.1; collision mesh filename=package://softhands_description/meshes/softhands/v1.0/commo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; visual mesh filename=package://softhands_description/meshes/softhands/v1.0/commo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
- added link left_hand_v1s_little_knuckle_link, mass 0.09; collision mesh filename=package://softhands_description/meshes/softhands/v1.0/commo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; visual mesh filename=package://softhands_description/meshes/softhands/v1.0/commo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
- added link left_hand_v1s_little_middle_link, mass 0.05; collision mesh filename=package://softhands_description/meshes/softhands/v1.0/commo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; visual mesh filename=package://softhands_description/meshes/softhands/v1.0/commo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
- added link left_hand_v1s_little_proximal_link, mass 0.05; collision mesh filename=package://softhands_description/meshes/softhands/v1.0/commo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; visual mesh filename=package://softhands_description/meshes/softhands/v1.0/commo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
- added link left_hand_v1s_middle_distal_link, mass 0.1; collision mesh filename=package://softhands_description/meshes/softhands/v1.0/commo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; visual mesh filename=package://softhands_description/meshes/softhands/v1.0/commo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
- added link left_hand_v1s_middle_knuckle_link, mass 0.09; collision mesh filename=package://softhands_description/meshes/softhands/v1.0/commo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; visual mesh filename=package://softhands_description/meshes/softhands/v1.0/commo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
- added link left_hand_v1s_middle_middle_link, mass 0.05; collision mesh filename=package://softhands_description/meshes/softhands/v1.0/commo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; visual mesh filename=package://softhands_description/meshes/softhands/v1.0/commo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
- added link left_hand_v1s_middle_proximal_link, mass 0.05; collision mesh filename=package://softhands_description/meshes/softhands/v1.0/commo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; visual mesh filename=package://softhands_description/meshes/softhands/v1.0/commo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
- added link left_hand_v1s_palm_base
- added link left_hand_v1s_palm_link, mass 2.28; collision mesh filename=package://softhands_description/meshes/softhands/v1.0/left/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; collision mesh filename=package://softhands_description/meshes/softhands/v1.0/right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
- added link left_hand_v1s_ring_distal_link, mass 0.1; collision mesh filename=package://softhands_description/meshes/softhands/v1.0/commo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; visual mesh filename=package://softhands_description/meshes/softhands/v1.0/commo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
- added link left_hand_v1s_ring_knuckle_link, mass 0.09; collision mesh filename=package://softhands_description/meshes/softhands/v1.0/commo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; visual mesh filename=package://softhands_description/meshes/softhands/v1.0/commo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
- added link left_hand_v1s_ring_middle_link, mass 0.05; collision mesh filename=package://softhands_description/meshes/softhands/v1.0/commo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; visual mesh filename=package://softhands_description/meshes/softhands/v1.0/commo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
- added link left_hand_v1s_ring_proximal_link, mass 0.05; collision mesh filename=package://softhands_description/meshes/softhands/v1.0/commo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; visual mesh filename=package://softhands_description/meshes/softhands/v1.0/commo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
- added link left_hand_v1s_synergy_link, mass 0.1
- added link left_hand_v1s_thumb_distal_link, mass 0.1; collision mesh filename=package://softhands_description/meshes/softhands/v1.0/commo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; visual mesh filename=package://softhands_description/meshes/softhands/v1.0/commo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
- added link left_hand_v1s_thumb_knuckle_link, mass 0.09; collision mesh filename=package://softhands_description/meshes/softhands/v1.0/left/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; visual mesh filename=package://softhands_description/meshes/softhands/v1.0/left/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
- added link left_hand_v1s_thumb_proximal_link, mass 0.05; collision mesh filename=package://softhands_description/meshes/softhands/v1.0/commo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; visual mesh filename=package://softhands_description/meshes/softhands/v1.0/commo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
- added link right_hand_v1s_grasp_link, mass 0.1
- added link right_hand_v1s_index_distal_link, mass 0.1; collision mesh filename=package://softhands_description/meshes/softhands/v1.0/commo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; visual mesh filename=package://softhands_description/meshes/softhands/v1.0/commo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
- added link right_hand_v1s_index_knuckle_link, mass 0.09; collision mesh filename=package://softhands_description/meshes/softhands/v1.0/commo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; visual mesh filename=package://softhands_description/meshes/softhands/v1.0/commo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
- added link right_hand_v1s_index_middle_link, mass 0.05; collision mesh filename=package://softhands_description/meshes/softhands/v1.0/commo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; visual mesh filename=package://softhands_description/meshes/softhands/v1.0/commo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
- added link right_hand_v1s_index_proximal_link, mass 0.05; collision mesh filename=package://softhands_description/meshes/softhands/v1.0/commo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; visual mesh filename=package://softhands_description/meshes/softhands/v1.0/commo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
- added link right_hand_v1s_little_distal_link, mass 0.1; collision mesh filename=package://softhands_description/meshes/softhands/v1.0/commo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; visual mesh filename=package://softhands_description/meshes/softhands/v1.0/commo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
- added link right_hand_v1s_little_knuckle_link, mass 0.09; collision mesh filename=package://softhands_description/meshes/softhands/v1.0/commo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; visual mesh filename=package://softhands_description/meshes/softhands/v1.0/commo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
- added link right_hand_v1s_little_middle_link, mass 0.05; collision mesh filename=package://softhands_description/meshes/softhands/v1.0/commo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; visual mesh filename=package://softhands_description/meshes/softhands/v1.0/commo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
- added link right_hand_v1s_little_proximal_link, mass 0.05; collision mesh filename=package://softhands_description/meshes/softhands/v1.0/commo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; visual mesh filename=package://softhands_description/meshes/softhands/v1.0/commo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
- added link right_hand_v1s_middle_distal_link, mass 0.1; collision mesh filename=package://softhands_description/meshes/softhands/v1.0/commo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; visual mesh filename=package://softhands_description/meshes/softhands/v1.0/commo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
- added link right_hand_v1s_middle_knuckle_link, mass 0.09; collision mesh filename=package://softhands_description/meshes/softhands/v1.0/commo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; visual mesh filename=package://softhands_description/meshes/softhands/v1.0/commo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
- added link right_hand_v1s_middle_middle_link, mass 0.05; collision mesh filename=package://softhands_description/meshes/softhands/v1.0/commo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; visual mesh filename=package://softhands_description/meshes/softhands/v1.0/commo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
- added link right_hand_v1s_middle_proximal_link, mass 0.05; collision mesh filename=package://softhands_description/meshes/softhands/v1.0/commo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; visual mesh filename=package://softhands_description/meshes/softhands/v1.0/commo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
- added link right_hand_v1s_palm_base
- added link right_hand_v1s_palm_link, mass 2.28; collision mesh filename=package://softhands_description/meshes/softhands/v1.0/right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; collision mesh filename=package://softhands_description/meshes/softhands/v1.0/right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
- added link right_hand_v1s_ring_distal_link, mass 0.1; collision mesh filename=package://softhands_description/meshes/softhands/v1.0/commo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; visual mesh filename=package://softhands_description/meshes/softhands/v1.0/commo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
- added link right_hand_v1s_ring_knuckle_link, mass 0.09; collision mesh filename=package://softhands_description/meshes/softhands/v1.0/commo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; visual mesh filename=package://softhands_description/meshes/softhands/v1.0/commo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
- added link right_hand_v1s_ring_middle_link, mass 0.05; collision mesh filename=package://softhands_description/meshes/softhands/v1.0/commo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; visual mesh filename=package://softhands_description/meshes/softhands/v1.0/commo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
- added link right_hand_v1s_ring_proximal_link, mass 0.05; collision mesh filename=package://softhands_description/meshes/softhands/v1.0/commo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; visual mesh filename=package://softhands_description/meshes/softhands/v1.0/commo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
- added link right_hand_v1s_synergy_link, mass 0.1
- added link right_hand_v1s_thumb_distal_link, mass 0.1; collision mesh filename=package://softhands_description/meshes/softhands/v1.0/commo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; visual mesh filename=package://softhands_description/meshes/softhands/v1.0/commo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
- added link right_hand_v1s_thumb_knuckle_link, mass 0.09; collision mesh filename=package://softhands_description/meshes/softhands/v1.0/right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; visual mesh filename=package://softhands_description/meshes/softhands/v1.0/right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
- added link right_hand_v1s_thumb_proximal_link, mass 0.05; collision mesh filename=package://softhands_description/meshes/softhands/v1.0/commo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; visual mesh filename=package://softhands_description/meshes/softhands/v1.0/commo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
Joints:
- removed joint left_hand_v2s_base_joint
- removed joint left_hand_v2s_grasp_joint
- removed joint left_hand_v2s_index_distal_joint
- removed joint left_hand_v2s_index_knuckle_joint
- removed joint left_hand_v2s_index_middle_joint
- removed joint left_hand_v2s_index_proximal_joint
- removed joint left_hand_v2s_little_distal_joint
- removed joint left_hand_v2s_little_knuckle_joint
- removed joint left_hand_v2s_little_middle_joint
- removed joint left_hand_v2s_little_proximal_joint
- removed joint left_hand_v2s_middle_distal_joint
- removed joint left_hand_v2s_middle_knuckle_joint
- removed joint left_hand_v2s_middle_middle_joint
- removed joint left_hand_v2s_middle_proximal_joint
- removed joint left_hand_v2s_palm_joint
- removed joint left_hand_v2s_ring_distal_joint
- removed joint left_hand_v2s_ring_knuckle_joint
- removed joint left_hand_v2s_ring_middle_joint
- removed joint left_hand_v2s_ring_proximal_joint
- removed joint left_hand_v2s_synergy_joint
- removed joint left_hand_v2s_thumb_distal_joint
- removed joint left_hand_v2s_thumb_knuckle_joint
- removed joint left_hand_v2s_thumb_proximal_joint
- removed joint right_hand_v2s_base_joint
- removed joint right_hand_v2s_grasp_joint
- removed joint right_hand_v2s_index_distal_joint
- removed joint right_hand_v2s_index_knuckle_joint
- removed joint right_hand_v2s_index_middle_joint
- removed joint right_hand_v2s_index_proximal_joint
- removed joint right_hand_v2s_little_distal_joint
- removed joint right_hand_v2s_little_knuckle_joint
- removed joint right_hand_v2s_little_middle_joint
- removed joint right_hand_v2s_little_proximal_joint
- removed joint right_hand_v2s_middle_distal_joint
- removed joint right_hand_v2s_middle_knuckle_joint
- removed joint right_hand_v2s_middle_middle_joint
- removed joint right_hand_v2s_middle_proximal_joint
- removed joint right_hand_v2s_palm_joint
- removed joint right_hand_v2s_ring_distal_joint
- removed joint right_hand_v2s_ring_knuckle_joint
- removed joint right_hand_v2s_ring_middle_joint
- removed joint right_hand_v2s_ring_proximal_joint
- removed joint right_hand_v2s_synergy_joint
- removed joint right_hand_v2s_thumb_distal_joint
- removed joint right_hand_v2s_thumb_knuckle_joint
- removed joint right_hand_v2s_thumb_proximal_joint
- added joint left_hand_base_joint: type fixed, parent arm_2_link_7, child left_hand_v1s_palm_base, origin xyz=0 -0.013900 -0.015 rpy=0 0 0
- added joint left_hand_v1s_grasp_joint: type fixed, parent left_hand_v1s_palm_link, child left_hand_v1s_grasp_link, origin xyz=0.0 0.0 0.07 rpy=0 0 0
- added joint left_hand_v1s_index_distal_joint: type revolute, parent left_hand_v1s_index_middle_link, child left_hand_v1s_index_distal_link, origin xyz=0.020 0 0 rpy=0 0 0, axis 0 -1 0, limit lower=-1.57 upper=1.57 effort=30 velocity=1.0, mimic joint=left_hand_v1s_synergy_joint multiplier=1.2
- added joint left_hand_v1s_index_knuckle_joint: type revolute, parent left_hand_v1s_palm_link, child left_hand_v1s_index_knuckle_link, origin xyz=-0.0033 -0.0195 0.0936994 rpy=-1.5707963267948966 -1.4835299330931884 -1.5707963267948966, axis 0 0 -1, limit lower=-1.57 upper=1.57 effort=30 velocity=1.0, mimic joint=left_hand_v1s_synergy_joint multiplier=1.2
- added joint left_hand_v1s_index_middle_joint: type revolute, parent left_hand_v1s_index_proximal_link, child left_hand_v1s_index_middle_link, origin xyz=0.020 0 0 rpy=0 0 0, axis 0 -1 0, limit lower=-1.57 upper=1.57 effort=30 velocity=1.0, mimic joint=left_hand_v1s_synergy_joint multiplier=1.2
- added joint left_hand_v1s_index_proximal_joint: type revolute, parent left_hand_v1s_index_knuckle_link, child left_hand_v1s_index_proximal_link, origin xyz=0.020 0 0 rpy=0 0 0, axis 0 -1 0, limit lower=-1.57 upper=1.57 effort=30 velocity=1.0, mimic joint=left_hand_v1s_synergy_joint multiplier=1.2
- added joint left_hand_v1s_little_distal_joint: type revolute, parent left_hand_v1s_little_middle_link, child left_hand_v1s_little_distal_link, origin xyz=0.020 0 0 rpy=0 0 0, axis 0 -1 0, limit lower=-1.57 upper=1.57 effort=30 velocity=1.0, mimic joint=left_hand_v1s_synergy_joint multiplier=1.2
- added joint left_hand_v1s_little_knuckle_joint: type revolute, parent left_hand_v1s_palm_link, child left_hand_v1s_little_knuckle_link, origin xyz=-0.0033 0.039 0.0836994 rpy=1.5707963267948966 -1.4835299330931884 1.5707963267948966, axis 0 0 -1, limit lower=-1.57 upper=1.57 effort=30 velocity=1.0, mimic joint=left_hand_v1s_synergy_joint multiplier=1.2
- added joint left_hand_v1s_little_middle_joint: type revolute, parent left_hand_v1s_little_proximal_link, child left_hand_v1s_little_middle_link, origin xyz=0.020 0 0 rpy=0 0 0, axis 0 -1 0, limit lower=-1.57 upper=1.57 effort=30 velocity=1.0, mimic joint=left_hand_v1s_synergy_joint multiplier=1.2
- added joint left_hand_v1s_little_proximal_joint: type revolute, parent left_hand_v1s_little_knuckle_link, child left_hand_v1s_little_proximal_link, origin xyz=0.020 0 0 rpy=0 0 0, axis 0 -1 0, limit lower=-1.57 upper=1.57 effort=30 velocity=1.0, mimic joint=left_hand_v1s_synergy_joint multiplier=1.2
- added joint left_hand_v1s_middle_distal_joint: type revolute, parent left_hand_v1s_middle_middle_link, child left_hand_v1s_middle_distal_link, origin xyz=0.020 0 0 rpy=0 0 0, axis 0 -1 0, limit lower=-1.57 upper=1.57 effort=30 velocity=1.0, mimic joint=left_hand_v1s_synergy_joint multiplier=1.2
- added joint left_hand_v1s_middle_knuckle_joint: type revolute, parent left_hand_v1s_palm_link, child left_hand_v1s_middle_knuckle_link, origin xyz=-0.0033 0.0 0.100699 rpy=3.1415 -1.5707963267948966 0.0, axis 0 0 -1, limit lower=-1.57 upper=1.57 effort=30 velocity=1.0, mimic joint=left_hand_v1s_synergy_joint multiplier=1.2
- added joint left_hand_v1s_middle_middle_joint: type revolute, parent left_hand_v1s_middle_proximal_link, child left_hand_v1s_middle_middle_link, origin xyz=0.020 0 0 rpy=0 0 0, axis 0 -1 0, limit lower=-1.57 upper=1.57 effort=30 velocity=1.0, mimic joint=left_hand_v1s_synergy_joint multiplier=1.2
- added joint left_hand_v1s_middle_proximal_joint: type revolute, parent left_hand_v1s_middle_knuckle_link, child left_hand_v1s_middle_proximal_link, origin xyz=0.020 0 0 rpy=0 0 0, axis 0 -1 0, limit lower=-1.57 upper=1.57 effort=30 velocity=1.0, mimic joint=left_hand_v1s_synergy_joint multiplier=1.2
- added joint left_hand_v1s_palm_joint: type fixed, parent left_hand_v1s_palm_base, child left_hand_v1s_palm_link, origin xyz=0.002 0.00695 0.0535 rpy=0 0 0
- added joint left_hand_v1s_ring_distal_joint: type revolute, parent left_hand_v1s_ring_middle_link, child left_hand_v1s_ring_distal_link, origin xyz=0.020 0 0 rpy=0 0 0, axis 0 -1 0, limit lower=-1.57 upper=1.57 effort=30 velocity=1.0, mimic joint=left_hand_v1s_synergy_joint multiplier=1.2
- added joint left_hand_v1s_ring_knuckle_joint: type revolute, parent left_hand_v1s_palm_link, child left_hand_v1s_ring_knuckle_link, origin xyz=-0.0033 0.0195 0.0936994 rpy=1.5707963267948966 -1.5184364298870514 1.5707963267948966, axis 0 0 -1, limit lower=-1.57 upper=1.57 effort=30 velocity=1.0, mimic joint=left_hand_v1s_synergy_joint multiplier=1.2
- added joint left_hand_v1s_ring_middle_joint: type revolute, parent left_hand_v1s_ring_proximal_link, child left_hand_v1s_ring_middle_link, origin xyz=0.020 0 0 rpy=0 0 0, axis 0 -1 0, limit lower=-1.57 upper=1.57 effort=30 velocity=1.0, mimic joint=left_hand_v1s_synergy_joint multiplier=1.2
- added joint left_hand_v1s_ring_proximal_joint: type revolute, parent left_hand_v1s_ring_knuckle_link, child left_hand_v1s_ring_proximal_link, origin xyz=0.020 0 0 rpy=0 0 0, axis 0 -1 0, limit lower=-1.57 upper=1.57 effort=30 velocity=1.0, mimic joint=left_hand_v1s_synergy_joint multiplier=1.2
- added joint left_hand_v1s_synergy_joint: type revolute, parent left_hand_v1s_palm_link, child left_hand_v1s_synergy_link, axis 0 0 1, limit lower=0.0 upper=1.0 effort=100 velocity=100000
- added joint left_hand_v1s_thumb_distal_joint: type continuous, parent left_hand_v1s_thumb_proximal_link, child left_hand_v1s_thumb_distal_link, origin xyz=0.020 0 0.0 rpy=0 0 0, axis 0 -1 0, mimic joint=left_hand_v1s_synergy_joint multiplier=1.2
- added joint left_hand_v1s_thumb_knuckle_joint: type continuous, parent left_hand_v1s_palm_link, child left_hand_v1s_thumb_knuckle_link, origin xyz=0.005669722 -0.029616 0.055314 rpy=0.0 -0.38397275793662144 -1.5707963267948966, axis 0 0 1, mimic joint=left_hand_v1s_synergy_joint multiplier=1.3
- added joint left_hand_v1s_thumb_proximal_joint: type continuous, parent left_hand_v1s_thumb_knuckle_link, child left_hand_v1s_thumb_proximal_link, origin xyz=0.033500000 0.0033 0.0 rpy=-0.426627741408745 0 0.0, axis 0 -1 0, mimic joint=left_hand_v1s_synergy_joint multiplier=1.2
- added joint right_hand_base_joint: type fixed, parent arm_1_link_7, child right_hand_v1s_palm_base, origin xyz=0 0 -0.015 rpy=0 0.0 3.14159265359
- added joint right_hand_v1s_grasp_joint: type fixed, parent right_hand_v1s_palm_link, child right_hand_v1s_grasp_link, origin xyz=0.0 0.0 0.07 rpy=0 0 0
- added joint right_hand_v1s_index_distal_joint: type revolute, parent right_hand_v1s_index_middle_link, child right_hand_v1s_index_distal_link, origin xyz=0.020 0 0 rpy=0 0 0, axis 0 -1 0, limit lower=-1.57 upper=1.57 effort=30 velocity=1.0, mimic joint=right_hand_v1s_synergy_joint multiplier=1.2
- added joint right_hand_v1s_index_knuckle_joint: type revolute, parent right_hand_v1s_palm_link, child right_hand_v1s_index_knuckle_link, origin xyz=-0.0033 0.0195 0.0936994 rpy=1.5707963267948966 -1.4835299330931884 1.5707963267948966, axis 0 0 1, limit lower=-1.57 upper=1.57 effort=30 velocity=1.0, mimic joint=right_hand_v1s_synergy_joint multiplier=1.2
- added joint right_hand_v1s_index_middle_joint: type revolute, parent right_hand_v1s_index_proximal_link, child right_hand_v1s_index_middle_link, origin xyz=0.020 0 0 rpy=0 0 0, axis 0 -1 0, limit lower=-1.57 upper=1.57 effort=30 velocity=1.0, mimic joint=right_hand_v1s_synergy_joint multiplier=1.2
- added joint right_hand_v1s_index_proximal_joint: type revolute, parent right_hand_v1s_index_knuckle_link, child right_hand_v1s_index_proximal_link, origin xyz=0.020 0 0 rpy=0 0 0, axis 0 -1 0, limit lower=-1.57 upper=1.57 effort=30 velocity=1.0, mimic joint=right_hand_v1s_synergy_joint multiplier=1.2
- added joint right_hand_v1s_little_distal_joint: type revolute, parent right_hand_v1s_little_middle_link, child right_hand_v1s_little_distal_link, origin xyz=0.020 0 0 rpy=0 0 0, axis 0 -1 0, limit lower=-1.57 upper=1.57 effort=30 velocity=1.0, mimic joint=right_hand_v1s_synergy_joint multiplier=1.2
- added joint right_hand_v1s_little_knuckle_joint: type revolute, parent right_hand_v1s_palm_link, child right_hand_v1s_little_knuckle_link, origin xyz=-0.0033 -0.039 0.0836994 rpy=-1.5707963267948966 -1.4835299330931884 -1.5707963267948966, axis 0 0 1, limit lower=-1.57 upper=1.57 effort=30 velocity=1.0, mimic joint=right_hand_v1s_synergy_joint multiplier=1.2
- added joint right_hand_v1s_little_middle_joint: type revolute, parent right_hand_v1s_little_proximal_link, child right_hand_v1s_little_middle_link, origin xyz=0.020 0 0 rpy=0 0 0, axis 0 -1 0, limit lower=-1.57 upper=1.57 effort=30 velocity=1.0, mimic joint=right_hand_v1s_synergy_joint multiplier=1.2
- added joint right_hand_v1s_little_proximal_joint: type revolute, parent right_hand_v1s_little_knuckle_link, child right_hand_v1s_little_proximal_link, origin xyz=0.020 0 0 rpy=0 0 0, axis 0 -1 0, limit lower=-1.57 upper=1.57 effort=30 velocity=1.0, mimic joint=right_hand_v1s_synergy_joint multiplier=1.2
- added joint right_hand_v1s_middle_distal_joint: type revolute, parent right_hand_v1s_middle_middle_link, child right_hand_v1s_middle_distal_link, origin xyz=0.020 0 0 rpy=0 0 0, axis 0 -1 0, limit lower=-1.57 upper=1.57 effort=30 velocity=1.0, mimic joint=right_hand_v1s_synergy_joint multiplier=1.2
- added joint right_hand_v1s_middle_knuckle_joint: type revolute, parent right_hand_v1s_palm_link, child right_hand_v1s_middle_knuckle_link, origin xyz=-0.003300000 0.0 0.100699 rpy=3.141592 -1.5707963267948966 0.0, axis 0 0 1, limit lower=-1.57 upper=1.57 effort=30 velocity=1.0, mimic joint=right_hand_v1s_synergy_joint multiplier=1.2
- added joint right_hand_v1s_middle_middle_joint: type revolute, parent right_hand_v1s_middle_proximal_link, child right_hand_v1s_middle_middle_link, origin xyz=0.020 0 0 rpy=0 0 0, axis 0 -1 0, limit lower=-1.57 upper=1.57 effort=30 velocity=1.0, mimic joint=right_hand_v1s_synergy_joint multiplier=1.2
- added joint right_hand_v1s_middle_proximal_joint: type revolute, parent right_hand_v1s_middle_knuckle_link, child right_hand_v1s_middle_proximal_link, origin xyz=0.020 0 0 rpy=0 0 0, axis 0 -1 0, limit lower=-1.57 upper=1.57 effort=30 velocity=1.0, mimic joint=right_hand_v1s_synergy_joint multiplier=1.2
- added joint right_hand_v1s_palm_joint: type fixed, parent right_hand_v1s_palm_base, child right_hand_v1s_palm_link, origin xyz=0.002 0.00695 0.0535 rpy=0 0 0
- added joint right_hand_v1s_ring_distal_joint: type revolute, parent right_hand_v1s_ring_middle_link, child right_hand_v1s_ring_distal_link, origin xyz=0.020 0 0 rpy=0 0 0, axis 0 -1 0, limit lower=-1.57 upper=1.57 effort=30 velocity=1.0, mimic joint=right_hand_v1s_synergy_joint multiplier=1.2
- added joint right_hand_v1s_ring_knuckle_joint: type revolute, parent right_hand_v1s_palm_link, child right_hand_v1s_ring_knuckle_link, origin xyz=-0.0033 -0.0195 0.0936994 rpy=-1.5707963267948966 -1.5184364298870514 -1.5707963267948966, axis 0 0 1, limit lower=-1.57 upper=1.57 effort=30 velocity=1.0, mimic joint=right_hand_v1s_synergy_joint multiplier=1.2
- added joint right_hand_v1s_ring_middle_joint: type revolute, parent right_hand_v1s_ring_proximal_link, child right_hand_v1s_ring_middle_link, origin xyz=0.020 0 0 rpy=0 0 0, axis 0 -1 0, limit lower=-1.57 upper=1.57 effort=30 velocity=1.0, mimic joint=right_hand_v1s_synergy_joint multiplier=1.2
- added joint right_hand_v1s_ring_proximal_joint: type revolute, parent right_hand_v1s_ring_knuckle_link, child right_hand_v1s_ring_proximal_link, origin xyz=0.020 0 0 rpy=0 0 0, axis 0 -1 0, limit lower=-1.57 upper=1.57 effort=30 velocity=1.0, mimic joint=right_hand_v1s_synergy_joint multiplier=1.2
- added joint right_hand_v1s_synergy_joint: type revolute, parent right_hand_v1s_palm_link, child right_hand_v1s_synergy_link, axis 0 0 1, limit lower=0.0 upper=1.0 effort=100 velocity=100000
- added joint right_hand_v1s_thumb_distal_joint: type continuous, parent right_hand_v1s_thumb_proximal_link, child right_hand_v1s_thumb_distal_link, origin xyz=0.020 0 0.0 rpy=0 0 0, axis 0 -1 0, mimic joint=right_hand_v1s_synergy_joint multiplier=1.2
- added joint right_hand_v1s_thumb_knuckle_joint: type continuous, parent right_hand_v1s_palm_link, child right_hand_v1s_thumb_knuckle_link, origin xyz=0.00566972 0.0296160 0.0553140 rpy=0.0 -0.38397275793662144 1.5707963267948966, axis 0 0 -1, mimic joint=right_hand_v1s_synergy_joint multiplier=1.3
- added joint right_hand_v1s_thumb_proximal_joint: type continuous, parent right_hand_v1s_thumb_knuckle_link, child right_hand_v1s_thumb_proximal_link, origin xyz=0.033500000 -0.0033 0.0 rpy=0.426627741408745 0 0.0, axis 0 -1 0, mimic joint=right_hand_v1s_synergy_joint multiplier=1.2
