Commit message: added new urdf version of arm and tried to use moveit; Bug: controller not stiff for initila gazebo pose

File: repair_urdf/urdf/repair_full.urdf.xacro (robot description, xacro)
@@ -1,183 +1,27 @@
 <?xml version="1.0"?>
-<!-- xacro for generating the full urdf of the RePair platform (cage + bimanual robot) -->
-<!-- is_sliding_wrist: whether to add a sliding joint along the wrist second d.o.f.
-    (true -> yes), everything else -> no. This is used to generate the URDF for the optimization.  -->
-<!-- gen_coll: whether to add the approximate collision  model of the platform -->
-<!-- load_sol: whether to generate the URDF without the additional d.o.f. used by the co-design optimization.
-Setting it to "true", allow to fix the additional d.o.f. to desired values
-(specified in the repair_urdf/config/arm_opt_mount_vals.yaml file) -->
-<!-- use_updated_wrist: visual parameter. if true, we load the latest meshes (which are adapted to the
-results of the optimization), otherwise we go with the old ones (generated for a spherical wrist) -->
-<robot name = "repair_full" xmlns:xacro="http://ros.org/wiki/xacro">
-<xacro:arg name="is_sliding_wrist" default="true" />
-<xacro:arg name="gen_coll" default="false" />
-<xacro:arg name="load_sol" default="true" />
-<xacro:arg name="use_updated_wrist" default="false" />
-<xacro:arg name="gz_self_collide" default="true" />
-<xacro:arg name="xbot" default="true" />
-<xacro:arg name="fixed_hands" default="false" />
-<xacro:include filename="$(find repair_urdf)/urdf/repair_arm.urdf.xacro"/>
-<xacro:include filename="$(find repair_urdf)/urdf/repair_cage.urdf.xacro"/>
-<xacro:include filename="$(find repair_urdf)/urdf/repair_opt_mount_params.urdf.xacro"/>
-<xacro:include filename="$(find repair_urdf)/urdf/materials.gazebo.xacro"/>
-<xacro:include filename="$(find repair_urdf)/urdf/repair_hand_transmission.xacro" />
-<xacro:if value="$(arg xbot)">
-    <xacro:include filename="$(find repair_urdf)/urdf/xbot2.gazebo.xacro"/>
-</xacro:if>
-<xacro:if value="$(arg load_sol)">
-    <joint name="x_joint" type="prismatic">
-        <origin xyz="0.0 0.0 ${mount_h}" rpy="0.0 0.0 0.0"/>
-        <parent link="working_surface_link"/>
-        <child link="base_link"/>
-        <axis xyz="1 0 0"/>
-        <limit lower="${- cage_depth/2 + x_joint_limit_margin}" upper= "${cage_depth/2 - x_joint_limit_margin}" effort="1000.0" velocity="20.0"/>
-    </joint>
-    <transmission name="trans_x_joint">
-        <type>transmission_interface/SimpleTransmission</type>
-        <joint name="x_joint">
-            <hardwareInterface>hardware_interface/PositionJointInterface</hardwareInterface>
-        </joint>
-        <actuator name="x_joint_motor">
-            <hardwareInterface>hardware_interface/PositionJointInterface</hardwareInterface>
-            <mechanicalReduction>1</mechanicalReduction>
-        </actuator>
-    </transmission>
-    <link name="base_link">
-        <!-- torso inertias + stuff attached to the sliding guide -->
-        <inertial>
-          <mass value="${full_torso_mass}" />
-          <origin xyz="0 0 0" />
-          <inertia ixx="0" ixy="0"  ixz="0"
-                  iyy="0" iyz="0"
-                  izz="0" />
-        </inertial>
-        <xacro:if value="$(arg use_updated_wrist)">
-            <visual name="base_link_visual">
-                <geometry>
-                    <mesh filename="package://repair_urdf/meshes/optimized/link_0.stl" scale="${mmTom} ${mmTom} ${mmTom}"/>
-                </geometry>
-                <material name="dark"/>
-            </visual>
-        </xacro:if>
-    </link>
-    <joint name="r_arm_mount_joint" type="fixed">
-        <origin xyz="0.0 ${-should_w} 0.0" rpy="0 0 0"/>
-        <parent link="base_link"/>
-        <child link="dummy_r"/>
-    </joint>
-    <joint name="l_arm_mount_joint" type="fixed">
-        <origin xyz="0.0 ${should_w} 0.0" rpy="0 0 0"/>
-        <parent link="base_link"/>
-        <child link="dummy_l"/>
-    </joint>
-    <link name="dummy_r">
-    </link>
-    <link name="dummy_l">
-    </link>
-    <joint name="roll_r" type="fixed">
-        <origin xyz="0 0.0 0.0" rpy="${roll_mount} 0.0 0.0"/>
-        <parent link="dummy_r"/>
-        <child link="r_arm_mount_frame"/>
-    </joint>
-    <joint name="roll_l" type="fixed">
-        <origin xyz="0 0.0 0.0" rpy="${-roll_mount} 0.0 0.0"/>
-        <parent link="dummy_l"/>
-        <child link="l_arm_mount_frame"/>
-    </joint>
-    <link name="r_arm_mount_frame">
-        <xacro:aux_inertia cutoff_inertia="${gazebo_cutoff_inertia}"/>
-    </link>
-    <link name="l_arm_mount_frame">
-        <xacro:aux_inertia cutoff_inertia="${gazebo_cutoff_inertia}"/>
-    </link>
-</xacro:if>
-<xacro:unless value="$(arg load_sol)">
-    <joint name="x_joint" type="prismatic">
-        <origin xyz="0.0 0.0 0.0" rpy="0.0 0.0 0.0"/>
-        <parent link="working_surface_link"/>
-        <child link="dummy_link"/>
-        <axis xyz="1 0 0"/>
-        <limit lower="${- cage_depth/2 + x_joint_limit_margin}" upper= "${cage_depth/2 - x_joint_limit_margin}" effort="1000.0" velocity="20.0"/>
-    </joint>
-    <link name="dummy_link">
-    </link>
-    <joint name="z_joint" type="prismatic">
-        <origin xyz="0.0 0.0 0.0" rpy="0.0 0.0 0.0"/>
-        <parent link="dummy_link"/>
-        <child link="base_link"/>
-        <axis xyz="0 0 1"/>
-        <limit lower="${z_joint_lb}" upper= "2" effort="1000.0" velocity="20.0"/>
-    </joint>
-    <!-- RePAIR assembly (two arms) -->
-    <link name="base_link">
-        <!-- torso inertias + stuff attached to the sliding guide -->
-        <inertial>
-            <mass value="${full_torso_mass}" />
-            <origin xyz="0 0 0" />
-            <inertia ixx="0" ixy="0"  ixz="0"
-                    iyy="0" iyz="0"
-                    izz="0" />
-          </inertial>
-        <xacro:if value="$(arg use_updated_wrist)">
-            <visual name="base_link_visual">
-                <geometry>
-                    <mesh filename="package://repair_urdf/meshes/optimized/link_0.stl" scale="${mmTom} ${mmTom} ${mmTom}"/>
-                </geometry>
-                <material name="dark"/>
-            </visual>
-        </xacro:if>
-    </link>
-    <link name="dummy_r">
-    </link>
-    <link name="dummy_l">
-    </link>
-    <joint name="r_arm_mount_joint" type="prismatic">
-        <origin xyz="0.0 0.0 0.0" rpy="0 0 0"/>
-        <parent link="base_link"/>
-        <child link="dummy_r"/>
-        <axis xyz="0 -1 0"/>
-        <limit lower="${shoulder_width_lb}" upper= "${shoulder_width_ub}" effort="1000.0" velocity="20.0"/>
-    </joint>
-    <joint name="l_arm_mount_joint" type="prismatic">
-        <origin xyz="0.0 0.0 0.0" rpy="0 0 0"/>
-        <parent link="base_link"/>
-        <child link="dummy_l"/>
-        <axis xyz="0 1 0"/>
-        <limit lower="${shoulder_width_lb}" upper= "${shoulder_width_ub}" effort="1000.0" velocity="20.0"/>
-    </joint>
-    <joint name="roll_r" type="revolute">
-        <origin xyz="0.0 0.0 0.0" rpy="0.0 0.0 0.0"/>
-        <parent link="dummy_r"/>
-        <child link="r_arm_mount_frame"/>
-        <axis xyz="1 0 0"/>
-        <limit lower="${shoulder_roll_lb}" upper="${shoulder_roll_ub}" effort="0.0" velocity="0.0"/>
-    </joint>
-    <joint name="roll_l" type="revolute">
-        <origin xyz="0.0 0.0 0.0" rpy="0.0 0.0 0.0"/>
-        <parent link="dummy_l"/>
-        <child link="l_arm_mount_frame"/>
-        <axis xyz="-1 0 0"/>
-        <limit lower="${shoulder_roll_lb}" upper="${shoulder_roll_ub}" effort="0.0" velocity="0.0"/>
-    </joint>
-    <link name="r_arm_mount_frame">
-    </link>
-    <link name="l_arm_mount_frame">
-    </link>
-</xacro:unless>
-<xacro:repair_arm base_link="r_arm_mount_frame" id="1" is_sliding_wrist="$(arg is_sliding_wrist)"
-gen_coll="$(arg gen_coll)" load_sol="$(arg load_sol)" use_updated_wrist ="$(arg use_updated_wrist)"
-gz_self_collide ="$(arg gz_self_collide)" fixed_hands ="$(arg fixed_hands)" />
-<xacro:repair_arm base_link="l_arm_mount_frame" id="2" is_sliding_wrist="$(arg is_sliding_wrist)"
-gen_coll="$(arg gen_coll)" load_sol="$(arg load_sol)" use_updated_wrist ="$(arg use_updated_wrist)"
-gz_self_collide ="$(arg gz_self_collide)" fixed_hands ="$(arg fixed_hands)" />
-<xacro:repair_arm_materials id="1" />
-<xacro:repair_arm_materials id="2" />
-<xacro:repair_torso_materials />
-<xacro:if value="$(arg gz_self_collide)">
-    <gazebo reference="table_top_link">
-        <selfCollide> 1 </selfCollide>
-    </gazebo>
-</xacro:if>
-<xacro:repair_hand_transmission id="left" />
-<xacro:repair_hand_transmission id="right" />
+<robot xmlns:xacro="http://ros.org/wiki/xacro" name="repair_full">
+    <xacro:include filename="$(find repair_urdf)/urdf/conversions.urdf.xacro" />
+    <xacro:include filename="$(find repair_urdf)/urdf/materials.urdf.xacro" />
+    <xacro:include filename="$(find repair_urdf)/urdf/repair_arm_macro.urdf.xacro" />
+    <xacro:include filename="$(find repair_urdf)/urdf/repair_torso_macro.urdf.xacro"/>
+    <xacro:include filename="$(find repair_urdf)/urdf/repair_cage_macro.urdf.xacro"/>
+    <xacro:include filename="$(find repair_urdf)/urdf/kinematics_properties.urdf.xacro" />
+    <xacro:include filename="$(find repair_urdf)/urdf/inertial_properties.urdf.xacro" />
+    <xacro:include filename="$(find repair_urdf)/urdf/limits.urdf.xacro" />
+    <xacro:include filename="$(find repair_urdf)/urdf/gazebo/xbot.gazebo.xacro" />
+    <link name="world"/>
+    <xacro:repair_cage parent="world">
+    </xacro:repair_cage>
+    <xacro:repair_torso parent="sliding_guide_link">
+    <origin xyz="${Torso_Ox} ${Torso_Oy} ${Torso_Oz}"
+            rpy="${Torso_roll} ${Torso_pitch} ${Torso_yaw}" />
+    </xacro:repair_torso>
+    <xacro:repair_arm id="2"  rot="1"  parent="torso_1">
+      <origin xyz="${Shoulder_1_Ox} ${Shoulder_1_Oy} ${Shoulder_1_Oz}"
+              rpy="${Shoulder_1_roll} ${Shoulder_1_pitch} ${Shoulder_1_yaw}" />
+    </xacro:repair_arm>
+    <xacro:repair_arm id="1"  rot="-1"  parent="torso_1">
+        <origin xyz="${Shoulder_1_Ox} ${-Shoulder_1_Oy} ${Shoulder_1_Oz}"
+                rpy="${-Shoulder_1_roll} ${Shoulder_1_pitch} ${Shoulder_1_yaw}" />
+      </xacro:repair_arm>
 </robot>

Commit message: Launch with local xbot dummy works

File: repair_urdf/urdf/repair_full.urdf (robot description, URDF)
Before this commit: robot repair_full, 75 links, 74 joints
Joints:
- joint left_hand_v1s_index_distal_joint: type revolute -> fixed
- joint left_hand_v1s_index_knuckle_joint: type revolute -> fixed
- joint left_hand_v1s_index_middle_joint: type revolute -> fixed
- joint left_hand_v1s_index_proximal_joint: type revolute -> fixed
- joint left_hand_v1s_little_distal_joint: type revolute -> fixed
- joint left_hand_v1s_little_knuckle_joint: type revolute -> fixed
- joint left_hand_v1s_little_middle_joint: type revolute -> fixed
- joint left_hand_v1s_little_proximal_joint: type revolute -> fixed
- joint left_hand_v1s_middle_distal_joint: type revolute -> fixed
- joint left_hand_v1s_middle_knuckle_joint: type revolute -> fixed
- joint left_hand_v1s_middle_middle_joint: type revolute -> fixed
- joint left_hand_v1s_middle_proximal_joint: type revolute -> fixed
- joint left_hand_v1s_ring_distal_joint: type revolute -> fixed
- joint left_hand_v1s_ring_knuckle_joint: type revolute -> fixed
- joint left_hand_v1s_ring_middle_joint: type revolute -> fixed
- joint left_hand_v1s_ring_proximal_joint: type revolute -> fixed
- joint left_hand_v1s_thumb_distal_joint: type continuous -> fixed
- joint left_hand_v1s_thumb_knuckle_joint: type continuous -> fixed
- joint left_hand_v1s_thumb_proximal_joint: type continuous -> fixed
- joint right_hand_v1s_index_distal_joint: type revolute -> fixed
- joint right_hand_v1s_index_knuckle_joint: type revolute -> fixed
- joint right_hand_v1s_index_middle_joint: type revolute -> fixed
- joint right_hand_v1s_index_proximal_joint: type revolute -> fixed
- joint right_hand_v1s_little_distal_joint: type revolute -> fixed
- joint right_hand_v1s_little_knuckle_joint: type revolute -> fixed
- joint right_hand_v1s_little_middle_joint: type revolute -> fixed
- joint right_hand_v1s_little_proximal_joint: type revolute -> fixed
- joint right_hand_v1s_middle_distal_joint: type revolute -> fixed
- joint right_hand_v1s_middle_knuckle_joint: type revolute -> fixed
- joint right_hand_v1s_middle_middle_joint: type revolute -> fixed
- joint right_hand_v1s_middle_proximal_joint: type revolute -> fixed
- joint right_hand_v1s_ring_distal_joint: type revolute -> fixed
- joint right_hand_v1s_ring_knuckle_joint: type revolute -> fixed
- joint right_hand_v1s_ring_middle_joint: type revolute -> fixed
- joint right_hand_v1s_ring_proximal_joint: type revolute -> fixed
- joint right_hand_v1s_thumb_distal_joint: type continuous -> fixed
- joint right_hand_v1s_thumb_knuckle_joint: type continuous -> fixed
- joint right_hand_v1s_thumb_proximal_joint: type continuous -> fixed

File: repair_urdf/urdf/repair_full.urdf.xacro (robot description, xacro)
@@ -38,5 +38,5 @@
         translation="0"
         operation_mode="0"
-        fixed_hands="false">
+        fixed_hands="true">
     </xacro:softhands>
     <xacro:softhands type="right"
@@ -47,5 +47,5 @@
         translation="0"
         operation_mode="0"
-        fixed_hands="false">
+        fixed_hands="true">
     </xacro:softhands>
     <!-- <gazebo reference="table_top_link">

Commit message: Fragment scanner demo works

File: repair_urdf/urdf/repair_full.urdf (robot description, URDF)
Before this commit: robot repair_full, 75 links, 74 joints
Links:
- added link camera_bottom_screw_frame
- added link camera_color_frame
- added link camera_color_optical_frame
- added link camera_depth_frame
- added link camera_depth_optical_frame
- added link camera_left_ir_frame
- added link camera_left_ir_optical_frame
- added link camera_link, mass 0.564; collision box size=0.02505 0.09 0.025; visual mesh filename=/home/bk/ros1/repair_robot_ws/src/repair_ros_robot/repair_u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
- added link camera_right_ir_frame
- added link camera_right_ir_optical_frame
- added link left_hand_v1s_grasp_link
- added link right_hand_v1s_grasp_link
Joints:
- added joint camera_color_joint: type fixed, parent camera_depth_frame, child camera_color_frame, origin xyz=0 0.015 0 rpy=0 0 0
- added joint camera_color_optical_joint: type fixed, parent camera_color_frame, child camera_color_optical_frame, origin xyz=0 0 0 rpy=-1.5707963267948966 0 -1.5707963267948966
- added joint camera_depth_joint: type fixed, parent camera_link, child camera_depth_frame, origin xyz=0 0 0 rpy=0 0 0
- added joint camera_depth_optical_joint: type fixed, parent camera_depth_frame, child camera_depth_optical_frame, origin xyz=0 0 0 rpy=-1.5707963267948966 0 -1.5707963267948966
- added joint camera_joint: type fixed, parent torso_1, child camera_bottom_screw_frame, origin xyz=0.0857 0.0000476009 -0.273184 rpy=0.0009783 1.1836725 0
- added joint camera_left_ir_joint: type fixed, parent camera_depth_frame, child camera_left_ir_frame, origin xyz=0 0.0 0 rpy=0 0 0
- added joint camera_left_ir_optical_joint: type fixed, parent camera_left_ir_frame, child camera_left_ir_optical_frame, origin xyz=0 0 0 rpy=-1.5707963267948966 0 -1.5707963267948966
- added joint camera_link_joint: type fixed, parent camera_bottom_screw_frame, child camera_link, origin xyz=0 0.0175 0.0125 rpy=0 0 0
- added joint camera_right_ir_joint: type fixed, parent camera_depth_frame, child camera_right_ir_frame, origin xyz=0 -0.05 0 rpy=0 0 0
- added joint camera_right_ir_optical_joint: type fixed, parent camera_right_ir_frame, child camera_right_ir_optical_frame, origin xyz=0 0 0 rpy=-1.5707963267948966 0 -1.5707963267948966
- added joint left_hand_v1s_grasp_joint: type fixed, parent left_hand_v1s_palm_link, child left_hand_v1s_grasp_link, origin xyz=0.03 -0.06 0.10 rpy=0 0 0
- added joint right_hand_v1s_grasp_joint: type fixed, parent right_hand_v1s_palm_link, child right_hand_v1s_grasp_link, origin xyz=0.03 0.06 0.10 rpy=0 0 0
- joint left_hand_base_joint: origin xyz=0 0 -0.015 rpy=0 0.0 3.14159265359 -> xyz=0 0 0 rpy=0 0.0 1.570796326795
- joint left_hand_v1s_index_distal_joint: type fixed -> revolute
- joint left_hand_v1s_index_knuckle_joint: type fixed -> revolute
- joint left_hand_v1s_index_middle_joint: type fixed -> revolute
- joint left_hand_v1s_index_proximal_joint: type fixed -> revolute
- joint left_hand_v1s_little_distal_joint: type fixed -> revolute
- joint left_hand_v1s_little_knuckle_joint: type fixed -> revolute
- joint left_hand_v1s_little_middle_joint: type fixed -> revolute
- joint left_hand_v1s_little_proximal_joint: type fixed -> revolute
- joint left_hand_v1s_middle_distal_joint: type fixed -> revolute
- joint left_hand_v1s_middle_knuckle_joint: type fixed -> revolute
- joint left_hand_v1s_middle_middle_joint: type fixed -> revolute
- joint left_hand_v1s_middle_proximal_joint: type fixed -> revolute
- joint left_hand_v1s_ring_distal_joint: type fixed -> revolute
- joint left_hand_v1s_ring_knuckle_joint: type fixed -> revolute
- joint left_hand_v1s_ring_middle_joint: type fixed -> revolute
- joint left_hand_v1s_ring_proximal_joint: type fixed -> revolute
- joint left_hand_v1s_thumb_distal_joint: type fixed -> continuous
- joint left_hand_v1s_thumb_knuckle_joint: type fixed -> continuous
- joint left_hand_v1s_thumb_proximal_joint: type fixed -> continuous
- joint right_hand_base_joint: origin xyz=0 -0.013900 -0.015 rpy=0 0 3.14159265359 -> xyz=0 0 0 rpy=0 0 -1.570796326795
- joint right_hand_v1s_index_distal_joint: type fixed -> revolute
- joint right_hand_v1s_index_knuckle_joint: type fixed -> revolute
- joint right_hand_v1s_index_middle_joint: type fixed -> revolute
- joint right_hand_v1s_index_proximal_joint: type fixed -> revolute
- joint right_hand_v1s_little_distal_joint: type fixed -> revolute
- joint right_hand_v1s_little_knuckle_joint: type fixed -> revolute
- joint right_hand_v1s_little_middle_joint: type fixed -> revolute
- joint right_hand_v1s_little_proximal_joint: type fixed -> revolute
- joint right_hand_v1s_middle_distal_joint: type fixed -> revolute
- joint right_hand_v1s_middle_knuckle_joint: type fixed -> revolute
- joint right_hand_v1s_middle_middle_joint: type fixed -> revolute
- joint right_hand_v1s_middle_proximal_joint: type fixed -> revolute
- joint right_hand_v1s_ring_distal_joint: type fixed -> revolute
- joint right_hand_v1s_ring_knuckle_joint: type fixed -> revolute
- joint right_hand_v1s_ring_middle_joint: type fixed -> revolute
- joint right_hand_v1s_ring_proximal_joint: type fixed -> revolute
- joint right_hand_v1s_thumb_distal_joint: type fixed -> continuous
- joint right_hand_v1s_thumb_knuckle_joint: type fixed -> continuous
- joint right_hand_v1s_thumb_proximal_joint: type fixed -> continuous

File: repair_urdf/urdf/repair_full.urdf.xacro (robot description, xacro)
@@ -38,6 +38,6 @@
         version="v1.0_simple"
         parent="arm_1_7"
-        position="0 0 -0.015"
-        orientation="0 0.0 ${PI}"
+        position="0 0 0"
+        orientation="0 0.0 ${PI/2}"
         translation="0"
         operation_mode="0"
@@ -47,6 +47,6 @@
         version="v1.0_simple"
         parent="arm_2_7"
-        position="0 -0.013900 -0.015"
-        orientation="0 0 ${PI}"
+        position="0 0 0"
+        orientation="0 0 ${-PI/2}"
         translation="0"
         operation_mode="0"

Commit message: Regenerated urdf so that it works with xbot dummy

File: repair_urdf/urdf/repair_full.urdf (robot description, URDF)
Before this commit: robot repair_full, 87 links, 86 joints
Joints:
- joint left_hand_v1s_index_distal_joint: type revolute -> fixed
- joint left_hand_v1s_index_knuckle_joint: type revolute -> fixed
- joint left_hand_v1s_index_middle_joint: type revolute -> fixed
- joint left_hand_v1s_index_proximal_joint: type revolute -> fixed
- joint left_hand_v1s_little_distal_joint: type revolute -> fixed
- joint left_hand_v1s_little_knuckle_joint: type revolute -> fixed
- joint left_hand_v1s_little_middle_joint: type revolute -> fixed
- joint left_hand_v1s_little_proximal_joint: type revolute -> fixed
- joint left_hand_v1s_middle_distal_joint: type revolute -> fixed
- joint left_hand_v1s_middle_knuckle_joint: type revolute -> fixed
- joint left_hand_v1s_middle_middle_joint: type revolute -> fixed
- joint left_hand_v1s_middle_proximal_joint: type revolute -> fixed
- joint left_hand_v1s_ring_distal_joint: type revolute -> fixed
- joint left_hand_v1s_ring_knuckle_joint: type revolute -> fixed
- joint left_hand_v1s_ring_middle_joint: type revolute -> fixed
- joint left_hand_v1s_ring_proximal_joint: type revolute -> fixed
- joint left_hand_v1s_thumb_distal_joint: type continuous -> fixed
- joint left_hand_v1s_thumb_knuckle_joint: type continuous -> fixed
- joint left_hand_v1s_thumb_proximal_joint: type continuous -> fixed
- joint right_hand_v1s_index_distal_joint: type revolute -> fixed
- joint right_hand_v1s_index_knuckle_joint: type revolute -> fixed
- joint right_hand_v1s_index_middle_joint: type revolute -> fixed
- joint right_hand_v1s_index_proximal_joint: type revolute -> fixed
- joint right_hand_v1s_little_distal_joint: type revolute -> fixed
- joint right_hand_v1s_little_knuckle_joint: type revolute -> fixed
- joint right_hand_v1s_little_middle_joint: type revolute -> fixed
- joint right_hand_v1s_little_proximal_joint: type revolute -> fixed
- joint right_hand_v1s_middle_distal_joint: type revolute -> fixed
- joint right_hand_v1s_middle_knuckle_joint: type revolute -> fixed
- joint right_hand_v1s_middle_middle_joint: type revolute -> fixed
- joint right_hand_v1s_middle_proximal_joint: type revolute -> fixed
- joint right_hand_v1s_ring_distal_joint: type revolute -> fixed
- joint right_hand_v1s_ring_knuckle_joint: type revolute -> fixed
- joint right_hand_v1s_ring_middle_joint: type revolute -> fixed
- joint right_hand_v1s_ring_proximal_joint: type revolute -> fixed
- joint right_hand_v1s_thumb_distal_joint: type continuous -> fixed
- joint right_hand_v1s_thumb_knuckle_joint: type continuous -> fixed
- joint right_hand_v1s_thumb_proximal_joint: type continuous -> fixed
