Commit message: l515 camera support for gazebo

File: repair_urdf/urdf/repair_full.urdf (robot description, URDF)
Before this commit: robot repair_full, 87 links, 86 joints
Links:
- removed link camera_left_ir_frame
- removed link camera_left_ir_optical_frame
- removed link camera_right_ir_frame
- removed link camera_right_ir_optical_frame
- added link camera_accel_frame
- added link camera_accel_optical_frame
- added link camera_gyro_frame
- added link camera_gyro_optical_frame
- added link camera_infra_frame
- added link camera_infra_optical_frame
- added link camera_lower_mount
- added link camera_upper_mount
- link camera_link: mass 0.564 -> 0.095; geometry collision cylinder length=0.026 radius=0.0305; visual mesh filename=package://realsense_description_l515/meshes/l515.dae
Joints:
- removed joint camera_left_ir_joint
- removed joint camera_left_ir_optical_joint
- removed joint camera_right_ir_joint
- removed joint camera_right_ir_optical_joint
- added joint camera_accel_joint: type fixed, parent camera_color_frame, child camera_accel_frame, origin xyz=-0.00410137791186571 -0.0129784867167473 0.00256138201802969 rpy=-0.006161012 0.020193459 0.016301375
- added joint camera_accel_optical_joint: type fixed, parent camera_accel_frame, child camera_accel_optical_frame, origin xyz=0 0 0 rpy=-1.5707963267948966 0 -1.5707963267948966
- added joint camera_gyro_joint: type fixed, parent camera_color_frame, child camera_gyro_frame, origin xyz=-0.00410137791186571 -0.0129784867167473 0.00256138201802969 rpy=-0.006161012 0.020193459 0.016301375
- added joint camera_gyro_optical_joint: type fixed, parent camera_gyro_frame, child camera_gyro_optical_frame, origin xyz=0 0 0 rpy=-1.5707963267948966 0 -1.5707963267948966
- added joint camera_infra_joint: type fixed, parent camera_link, child camera_infra_frame, origin xyz=0 0.0 0 rpy=0 0 0
- added joint camera_infra_optical_joint: type fixed, parent camera_infra_frame, child camera_infra_optical_frame, origin xyz=0 0 0 rpy=-1.5707963267948966 0 -1.5707963267948966
- added joint camera_lower_mount_joint: type fixed, parent camera_bottom_screw_frame, child camera_lower_mount, origin xyz=-0.013999999999999999 0 0.01015 rpy=0 0 0
- added joint camera_upper_mount_joint: type fixed, parent camera_bottom_screw_frame, child camera_upper_mount, origin xyz=-0.013999999999999999 0 0.05015 rpy=0 0 0
- joint camera_color_joint: origin xyz=0 0.015 0 rpy=0 0 0 -> xyz=0 0 0.024 rpy=0 0 0; parent camera_depth_frame -> camera_link
- joint camera_joint: origin xyz=0.0857 0.0000476009 -0.273184 rpy=0.0009783 1.1836725 0 -> xyz=0.0857 0.0000476009 -0.268184 rpy=0.0009783 1.1836725 0
- joint camera_link_joint: origin xyz=0 0.0175 0.0125 rpy=0 0 0 -> xyz=0.007500000000000001 0.0 0.021150000000000002 rpy=0 0 0
- joint left_hand_v1s_index_distal_joint: type fixed -> revolute
- joint left_hand_v1s_index_knuckle_joint: type fixed -> revolute
- joint left_hand_v1s_index_middle_joint: type fixed -> revolute
- joint left_hand_v1s_index_proximal_joint: type fixed -> revolute
- joint left_hand_v1s_little_distal_joint: type fixed -> revolute
- joint left_hand_v1s_little_knuckle_joint: type fixed -> revolute
- joint left_hand_v1s_little_middle_joint: type fixed -> revolute
- joint left_hand_v1s_little_proximal_joint: type fixed -> revolute
- joint left_hand_v1s_middle_distal_joint: type fixed -> revolute
- joint left_hand_v1s_middle_knuckle_joint: type fixed -> revolute
- joint left_hand_v1s_middle_middle_joint: type fixed -> revolute
- joint left_hand_v1s_middle_proximal_joint: type fixed -> revolute
- joint left_hand_v1s_ring_distal_joint: type fixed -> revolute
- joint left_hand_v1s_ring_knuckle_joint: type fixed -> revolute
- joint left_hand_v1s_ring_middle_joint: type fixed -> revolute
- joint left_hand_v1s_ring_proximal_joint: type fixed -> revolute
- joint left_hand_v1s_thumb_distal_joint: type fixed -> continuous
- joint left_hand_v1s_thumb_knuckle_joint: type fixed -> continuous
- joint left_hand_v1s_thumb_proximal_joint: type fixed -> continuous
- joint right_hand_v1s_index_distal_joint: type fixed -> revolute
- joint right_hand_v1s_index_knuckle_joint: type fixed -> revolute
- joint right_hand_v1s_index_middle_joint: type fixed -> revolute
- joint right_hand_v1s_index_proximal_joint: type fixed -> revolute
- joint right_hand_v1s_little_distal_joint: type fixed -> revolute
- joint right_hand_v1s_little_knuckle_joint: type fixed -> revolute
- joint right_hand_v1s_little_middle_joint: type fixed -> revolute
- joint right_hand_v1s_little_proximal_joint: type fixed -> revolute
- joint right_hand_v1s_middle_distal_joint: type fixed -> revolute
- joint right_hand_v1s_middle_knuckle_joint: type fixed -> revolute
- joint right_hand_v1s_middle_middle_joint: type fixed -> revolute
- joint right_hand_v1s_middle_proximal_joint: type fixed -> revolute
- joint right_hand_v1s_ring_distal_joint: type fixed -> revolute
- joint right_hand_v1s_ring_knuckle_joint: type fixed -> revolute
- joint right_hand_v1s_ring_middle_joint: type fixed -> revolute
- joint right_hand_v1s_ring_proximal_joint: type fixed -> revolute
- joint right_hand_v1s_thumb_distal_joint: type fixed -> continuous
- joint right_hand_v1s_thumb_knuckle_joint: type fixed -> continuous
- joint right_hand_v1s_thumb_proximal_joint: type fixed -> continuous

File: repair_urdf/urdf/repair_full.urdf.xacro (robot description, xacro)
@@ -11,4 +11,5 @@
     <xacro:include filename="$(find repair_urdf)/urdf/limits.urdf.xacro" />
     <xacro:include filename="$(find repair_urdf)/urdf/_d435.urdf.xacro"/>
+    <xacro:include filename="$(find repair_urdf)/urdf/_l515.urdf.xacro"/>
     <!-- Only when working with Gazebo Xbot Control -->
     <!-- DO NOT USE WITH ROS_CONTROL AND MOVEIT -->
@@ -20,7 +21,11 @@
     <xacro:repair_cage parent="world">
     </xacro:repair_cage>
-    <xacro:sensor_d435 parent='torso_1'>
+    <!-- <xacro:sensor_d435 parent='torso_1'>
         <origin xyz="0.0857 0.0000476009 -0.273184" rpy="0.0009783 1.1836725 0" />
-    </xacro:sensor_d435>
+    </xacro:sensor_d435> -->
+    <xacro:sensor_l515 parent='torso_1' use_nominal_extrinsics='true'>
+        <!-- <origin xyz="0.0857 0.0000476009 -0.273184" rpy="0.0009783 1.1836725 0" /> -->
+        <origin xyz="0.0857 0.0000476009 -0.268184" rpy="0.0009783 1.1836725 0" />
+    </xacro:sensor_l515>
     <xacro:repair_torso parent="sliding_guide_link">
     <origin xyz="${Torso_Ox} ${Torso_Oy} ${Torso_Oz}"

Commit message: modified ecat and full xacro with v1_2_research

File: repair_urdf/urdf/repair_full.urdf (robot description, URDF)
Before this commit: robot repair_full, 115 links, 114 joints
Links:
- link camera_link: geometry collision box size=0.02505 0.09 0.025; visual mesh filename=/home/embedded/forest_ws/ros_src/repair_ros_robot/repair_ur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
Joints:
- joint left_hand_v1_2_research_grasp_joint: origin xyz=0.03 0.06 0.10 rpy=0 0 0 -> xyz=0.06 0.03 0.16 rpy=0 0 1.57
- joint left_hand_v1_2_research_index_distal_joint: type revolute -> fixed
- joint left_hand_v1_2_research_index_distal_virtual_joint: type revolute -> fixed
- joint left_hand_v1_2_research_index_knuckle_joint: type revolute -> fixed
- joint left_hand_v1_2_research_index_middle_joint: type revolute -> fixed
- joint left_hand_v1_2_research_index_middle_virtual_joint: type revolute -> fixed
- joint left_hand_v1_2_research_index_proximal_joint: type revolute -> fixed
- joint left_hand_v1_2_research_index_proximal_virtual_joint: type revolute -> fixed
- joint left_hand_v1_2_research_iso_joint: origin xyz=0 -0. 0.00 rpy=0 0 1.570796326795 -> xyz=0 0 0.00 rpy=0 0 0
- joint left_hand_v1_2_research_little_distal_joint: type revolute -> fixed
- joint left_hand_v1_2_research_little_distal_virtual_joint: type revolute -> fixed
- joint left_hand_v1_2_research_little_knuckle_joint: type revolute -> fixed
- joint left_hand_v1_2_research_little_middle_joint: type revolute -> fixed
- joint left_hand_v1_2_research_little_middle_virtual_joint: type revolute -> fixed
- joint left_hand_v1_2_research_little_proximal_joint: type revolute -> fixed
- joint left_hand_v1_2_research_little_proximal_virtual_joint: type revolute -> fixed
- joint left_hand_v1_2_research_middle_distal_joint: type revolute -> fixed
- joint left_hand_v1_2_research_middle_distal_virtual_joint: type revolute -> fixed
- joint left_hand_v1_2_research_middle_knuckle_joint: type revolute -> fixed
- joint left_hand_v1_2_research_middle_middle_joint: type revolute -> fixed
- joint left_hand_v1_2_research_middle_middle_virtual_joint: type revolute -> fixed
- joint left_hand_v1_2_research_middle_proximal_joint: type revolute -> fixed
- joint left_hand_v1_2_research_middle_proximal_virtual_joint: type revolute -> fixed
- joint left_hand_v1_2_research_ring_distal_joint: type revolute -> fixed
- joint left_hand_v1_2_research_ring_distal_virtual_joint: type revolute -> fixed
- joint left_hand_v1_2_research_ring_knuckle_joint: type revolute -> fixed
- joint left_hand_v1_2_research_ring_middle_joint: type revolute -> fixed
- joint left_hand_v1_2_research_ring_middle_virtual_joint: type revolute -> fixed
- joint left_hand_v1_2_research_ring_proximal_joint: type revolute -> fixed
- joint left_hand_v1_2_research_ring_proximal_virtual_joint: type revolute -> fixed
- joint left_hand_v1_2_research_thumb_distal_joint: type revolute -> fixed
- joint left_hand_v1_2_research_thumb_distal_virtual_joint: type revolute -> fixed
- joint left_hand_v1_2_research_thumb_knuckle_joint: type revolute -> fixed
- joint left_hand_v1_2_research_thumb_proximal_joint: type revolute -> fixed
- joint left_hand_v1_2_research_thumb_proximal_virtual_joint: type revolute -> fixed
- joint right_hand_v1_2_research_grasp_joint: origin xyz=0.03 0.06 0.10 rpy=0 0 0 -> xyz=-0.06 0.03 0.16 rpy=0 0 1.57
- joint right_hand_v1_2_research_index_distal_joint: type revolute -> fixed
- joint right_hand_v1_2_research_index_distal_virtual_joint: type revolute -> fixed
- joint right_hand_v1_2_research_index_knuckle_joint: type revolute -> fixed
- joint right_hand_v1_2_research_index_middle_joint: type revolute -> fixed
- joint right_hand_v1_2_research_index_middle_virtual_joint: type revolute -> fixed
- joint right_hand_v1_2_research_index_proximal_joint: type revolute -> fixed
- joint right_hand_v1_2_research_index_proximal_virtual_joint: type revolute -> fixed
- joint right_hand_v1_2_research_iso_joint: origin xyz=0 0.0 0.00 rpy=0 0 1.570796326795 -> xyz=0 0.0 0.00 rpy=0 0 3.14
- joint right_hand_v1_2_research_little_distal_joint: type revolute -> fixed
- joint right_hand_v1_2_research_little_distal_virtual_joint: type revolute -> fixed
- joint right_hand_v1_2_research_little_knuckle_joint: type revolute -> fixed
- joint right_hand_v1_2_research_little_middle_joint: type revolute -> fixed
- joint right_hand_v1_2_research_little_middle_virtual_joint: type revolute -> fixed
- joint right_hand_v1_2_research_little_proximal_joint: type revolute -> fixed
- joint right_hand_v1_2_research_little_proximal_virtual_joint: type revolute -> fixed
- joint right_hand_v1_2_research_middle_distal_joint: type revolute -> fixed
- joint right_hand_v1_2_research_middle_distal_virtual_joint: type revolute -> fixed
- joint right_hand_v1_2_research_middle_knuckle_joint: type revolute -> fixed
- joint right_hand_v1_2_research_middle_middle_joint: type revolute -> fixed
- joint right_hand_v1_2_research_middle_middle_virtual_joint: type revolute -> fixed
- joint right_hand_v1_2_research_middle_proximal_joint: type revolute -> fixed
- joint right_hand_v1_2_research_middle_proximal_virtual_joint: type revolute -> fixed
- joint right_hand_v1_2_research_ring_distal_joint: type revolute -> fixed
- joint right_hand_v1_2_research_ring_distal_virtual_joint: type revolute -> fixed
- joint right_hand_v1_2_research_ring_knuckle_joint: type revolute -> fixed
- joint right_hand_v1_2_research_ring_middle_joint: type revolute -> fixed
- joint right_hand_v1_2_research_ring_middle_virtual_joint: type revolute -> fixed
- joint right_hand_v1_2_research_ring_proximal_joint: type revolute -> fixed
- joint right_hand_v1_2_research_ring_proximal_virtual_joint: type revolute -> fixed
- joint right_hand_v1_2_research_thumb_distal_joint: type revolute -> fixed
- joint right_hand_v1_2_research_thumb_distal_virtual_joint: type revolute -> fixed
- joint right_hand_v1_2_research_thumb_knuckle_joint: type revolute -> fixed
- joint right_hand_v1_2_research_thumb_proximal_joint: type revolute -> fixed
- joint right_hand_v1_2_research_thumb_proximal_virtual_joint: type revolute -> fixed

File: repair_urdf/urdf/repair_full.urdf.xacro (robot description, xacro)
@@ -39,6 +39,6 @@
         version="v1_2_research"
         position="0 0 0"
-        orientation="${PI/2}"
-        fixed_hands="false">
+        orientation="${PI}"
+        fixed_hands="true">
     </xacro:softhands>
     <gazebo reference="table_top_link">

Commit message: thursday changes from thinkstation

File: repair_urdf/urdf/repair_full.urdf (robot description, URDF)
Before this commit: robot repair_full, 123 links, 122 joints
Links:
- added link dummy_prismatic_link
- link arm_1_1: geometry collision mesh filename=package://repair_urdf/meshes/simplified/mesh_sh-pitch.stl scale=0.001 -0.001 0.001; visual mesh filename=package://repair_urdf/meshes/simplified/mesh_sh-pitch.stl scale=0.001 -0.001 0.001
- link arm_1_2: geometry collision mesh filename=package://repair_urdf/meshes/simplified/mesh_sh-roll.stl scale=0.001 -0.001 0.001; visual mesh filename=package://repair_urdf/meshes/simplified/mesh_sh-roll.stl scale=0.001 -0.001 0.001
- link arm_1_3: geometry collision mesh filename=package://repair_urdf/meshes/simplified/mesh_sh-yaw.stl scale=0.001 -0.001 0.001; visual mesh filename=package://repair_urdf/meshes/simplified/mesh_sh-yaw.stl scale=0.001 -0.001 0.001
- link arm_1_4: geometry collision mesh filename=package://repair_urdf/meshes/simplified/mesh_elbow.stl scale=0.001 -0.001 0.001; visual mesh filename=package://repair_urdf/meshes/simplified/mesh_elbow.stl scale=0.001 -0.001 0.001
- link arm_1_5: geometry collision mesh filename=package://repair_urdf/meshes/simplified/mesh_forearm-yaw.stl scale=0.001 -0.001 0.001; visual mesh filename=package://repair_urdf/meshes/simplified/mesh_forearm-yaw.stl scale=0.001 -0.001 0.001
- link arm_1_6: geometry collision mesh filename=package://repair_urdf/meshes/simplified/mesh_wrist-pitch.stl scale=0.001 -0.001 0.001; visual mesh filename=package://repair_urdf/meshes/simplified/mesh_wrist-pitch.stl scale=0.001 -0.001 0.001
- link arm_1_7: geometry collision mesh filename=package://repair_urdf/meshes/simplified/mesh_wrist-roll.stl scale=0.001 -0.001 0.001; visual mesh filename=package://repair_urdf/meshes/simplified/mesh_wrist-roll.stl scale=0.001 -0.001 0.001
- link arm_2_1: geometry collision mesh filename=package://repair_urdf/meshes/simplified/mesh_sh-pitch.stl scale=0.001 0.001 0.001; visual mesh filename=package://repair_urdf/meshes/simplified/mesh_sh-pitch.stl scale=0.001 0.001 0.001
- link arm_2_2: geometry collision mesh filename=package://repair_urdf/meshes/simplified/mesh_sh-roll.stl scale=0.001 0.001 0.001; visual mesh filename=package://repair_urdf/meshes/simplified/mesh_sh-roll.stl scale=0.001 0.001 0.001
- link arm_2_3: geometry collision mesh filename=package://repair_urdf/meshes/simplified/mesh_sh-yaw.stl scale=0.001 0.001 0.001; visual mesh filename=package://repair_urdf/meshes/simplified/mesh_sh-yaw.stl scale=0.001 0.001 0.001
- link arm_2_4: geometry collision mesh filename=package://repair_urdf/meshes/simplified/mesh_elbow.stl scale=0.001 0.001 0.001; visual mesh filename=package://repair_urdf/meshes/simplified/mesh_elbow.stl scale=0.001 0.001 0.001
- link arm_2_5: geometry collision mesh filename=package://repair_urdf/meshes/simplified/mesh_forearm-yaw.stl scale=0.001 0.001 0.001; visual mesh filename=package://repair_urdf/meshes/simplified/mesh_forearm-yaw.stl scale=0.001 0.001 0.001
- link arm_2_6: geometry collision mesh filename=package://repair_urdf/meshes/simplified/mesh_wrist-pitch.stl scale=0.001 0.001 0.001; visual mesh filename=package://repair_urdf/meshes/simplified/mesh_wrist-pitch.stl scale=0.001 0.001 0.001
- link arm_2_7: geometry collision mesh filename=package://repair_urdf/meshes/simplified/mesh_wrist-roll.stl scale=0.001 0.001 0.001; visual mesh filename=package://repair_urdf/meshes/simplified/mesh_wrist-roll.stl scale=0.001 0.001 0.001
Joints:
- removed joint left_hand_v1_2_research_grasp_joint
- added joint j_sliding_guide: type fixed, parent sliding_guide_link, child dummy_prismatic_link, origin xyz=0 0 0 rpy=0 0 0
- added joint left_hand_v1_wide_grasp_joint: type fixed, parent left_hand_v1_wide_palm_central_link, child left_hand_v1_wide_grasp_link, origin xyz=0.03 -0.10 0.15 rpy=0 0 0
- joint j_torso_1: axis 0 0 1 -> (none); limit lower=-2.6 upper=2.6 effort=147.0 velocity=3.86 -> (none); parent sliding_guide_link -> dummy_prismatic_link; type revolute -> fixed
- joint left_hand_v1_wide_palm_central_joint: child left_hand_v1_2_research_iso_link -> left_hand_v1_wide_palm_central_link; origin xyz=0 -0. 0.00 rpy=0 0 3.14159265359 -> xyz=0 0 0.0 rpy=0 0 1.570796326795
- joint right_hand_v1_2_research_grasp_joint: origin xyz=0.03 0.06 0.10 rpy=0 0 1.57 -> xyz=-0.06 0.03 0.16 rpy=0 0 1.57

File: repair_urdf/urdf/repair_full.urdf.xacro (robot description, xacro)
@@ -1,5 +1,5 @@
 <?xml version="1.0"?>
 <robot xmlns:xacro="http://ros.org/wiki/xacro" name="repair_full">
-    <xacro:arg name="sh_version" default="v1_2_research"/>
+    <xacro:arg name="sh_version" default="mixed_hands"/>
     <xacro:arg name="fixed_hands" default="true"/>
     <xacro:include filename="$(find softhands_description)/urdf/softhands.xacro" />
