Commit message: last day updates

File: repair_urdf/urdf/repair_full.urdf (robot description, URDF)
Before this commit: robot repair_full, 124 links, 123 joints
Links:
- added link arm_1_angle_flange; collision mesh filename=package://repair_urdf/meshes/angle_flange_90.stl scale=0.001 0.001 0.001; visual mesh filename=package://repair_urdf/meshes/angle_flange_90.stl scale=0.001 0.001 0.001
- added link arm_1_camera_mount; collision mesh filename=package://repair_urdf/meshes/camera_supp_cover_wide_left.stl scale=0.001 0.001 0.001; visual mesh filename=package://repair_urdf/meshes/camera_supp_cover_wide_left.stl scale=0.001 0.001 0.001
- added link arm_2_angle_flange; collision mesh filename=package://repair_urdf/meshes/angle_flange_90.stl scale=0.001 0.001 0.001; visual mesh filename=package://repair_urdf/meshes/angle_flange_90.stl scale=0.001 0.001 0.001
- added link arm_2_camera_mount; collision mesh filename=package://repair_urdf/meshes/camera_supp_cover_sh1p2.stl scale=0.001 0.001 0.001; visual mesh filename=package://repair_urdf/meshes/camera_supp_cover_sh1p2.stl scale=0.001 0.001 0.001
- link leg1_link: geometry collision cylinder length=0.978 radius=0.02; visual cylinder length=0.978 radius=0.02
- link leg2_link: geometry collision cylinder length=0.978 radius=0.02; visual cylinder length=0.978 radius=0.02
- link leg3_link: geometry collision cylinder length=0.978 radius=0.02; visual cylinder length=0.978 radius=0.02
- link leg4_link: geometry collision cylinder length=0.978 radius=0.02; visual cylinder length=0.978 radius=0.02
- link sliding_guide_link: geometry collision box size=0.001 1.0 2.5; visual box size=0.001 0.4 2.5
- link table_top_link: geometry collision box size=1.0 2.5 0.028; visual box size=1.0 2.5 0.028
Joints:
- added joint arm_1_angle_flange_joint: type fixed, parent arm_1_7, child arm_1_angle_flange, origin xyz=0.0425 0 0.0430 rpy=0 1.5707963 0
- added joint arm_1_camera_mount_joint: type fixed, parent arm_1_7, child arm_1_camera_mount, origin xyz=0.17545 0.016874 -0.01 rpy=0 1.5707963 0
- added joint arm_2_angle_flange_joint: type fixed, parent arm_2_7, child arm_2_angle_flange, origin xyz=0.0425 0 0.0380 rpy=0 1.5707963 0
- added joint arm_2_camera_mount_joint: type fixed, parent arm_2_7, child arm_2_camera_mount, origin xyz=0.18145 0.00528118 -0.01350 rpy=0 1.5707963 0
- joint left_hand_v1_wide_palm_central_joint: origin xyz=0 0 0.0 rpy=0 0 1.570796326795 -> xyz=0.005 0 0 rpy=0 0 3.14159265359; parent arm_1_7 -> arm_1_angle_flange
- joint leg1_joint: origin xyz=0.5 1.25 1.0 rpy=0 0 0 -> xyz=0.5 1.25 0.978 rpy=0 0 0
- joint leg2_joint: origin xyz=-0.5 1.25 1.0 rpy=0 0 0 -> xyz=-0.5 1.25 0.978 rpy=0 0 0
- joint leg3_joint: origin xyz=0.5 -1.25 1.0 rpy=0 0 0 -> xyz=0.5 -1.25 0.978 rpy=0 0 0
- joint leg4_joint: origin xyz=-0.5 -1.25 1.0 rpy=0 0 0 -> xyz=-0.5 -1.25 0.978 rpy=0 0 0
- joint right_hand_v1_2_research_iso_joint: origin xyz=0 0.0 0.00 rpy=0 0 3.14159265359 -> xyz=0.005 0 0 rpy=0 0 1.570796326795; parent arm_2_7 -> arm_2_angle_flange

File: repair_urdf/urdf/repair_full.urdf.xacro (robot description, xacro)
@@ -43,10 +43,95 @@
         <origin xyz="${Shoulder_1_Ox} ${-Shoulder_1_Oy} ${Shoulder_1_Oz}"
                 rpy="${-Shoulder_1_roll} ${Shoulder_1_pitch} ${Shoulder_1_yaw}" />
-      </xacro:repair_arm>
-    <!--QUIRINO/GIANNIROS: here change the version for v1_2_research (small hand) or v1_wide (wide hand) and mixed-->
+    </xacro:repair_arm>
+    <!-- add end-effector mount for both arms -->
+    <link name="arm_1_angle_flange" >
+        <visual>
+            <origin xyz="0.0425 0 -0.0430" rpy="0 -1.5707963 0"/>
+            <geometry>
+                <mesh filename="package://repair_urdf/meshes/angle_flange_90.stl" scale="0.001 0.001 0.001"/>
+            </geometry>
+            <material name="dark"/>
+        </visual>
+        <collision>
+            <origin xyz="0.0425 0 -0.0430" rpy="0 -1.5707963 0"/>
+            <geometry>
+                <mesh filename="package://repair_urdf/meshes/angle_flange_90.stl" scale="0.001 0.001 0.001"/>
+            </geometry>
+        </collision>
+    </link>
+    <joint name="arm_1_angle_flange_joint" type="fixed">
+        <parent link="arm_1_7"/>
+        <child link="arm_1_angle_flange"/>
+        <origin xyz="0.0425 0 0.0430" rpy="0 1.5707963 0"/>
+    </joint>
+    <link name="arm_2_angle_flange" >
+        <visual>
+            <origin xyz="0.0425 0 -0.0430" rpy="0 -1.5707963 0"/>
+            <geometry>
+                <mesh filename="package://repair_urdf/meshes/angle_flange_90.stl" scale="0.001 0.001 0.001"/>
+            </geometry>
+            <material name="dark"/>
+        </visual>
+        <collision>
+            <origin xyz="0.0425 0 -0.0430" rpy="0 -1.5707963 0"/>
+            <geometry>
+                <mesh filename="package://repair_urdf/meshes/angle_flange_90.stl" scale="0.001 0.001 0.001"/>
+            </geometry>
+        </collision>
+    </link>
+    <joint name="arm_2_angle_flange_joint" type="fixed">
+        <parent link="arm_2_7"/>
+        <child link="arm_2_angle_flange"/>
+        <origin xyz="0.0425 0 0.0380" rpy="0 1.5707963 0"/>
+    </joint>
+    <!-- add camera mounts -->
+    <link name="arm_1_camera_mount" >
+        <visual>
+            <origin xyz="0.0 0.0 0.0" rpy="0 0.0 0"/>
+            <geometry>
+                <mesh filename="package://repair_urdf/meshes/camera_supp_cover_wide_left.stl" scale="0.001 0.001 0.001"/>
+            </geometry>
+            <material name="dark"/>
+        </visual>
+        <collision>
+            <origin xyz="0.0 0.0 0.0" rpy="0 0.0 0"/>
+            <geometry>
+                <mesh filename="package://repair_urdf/meshes/camera_supp_cover_wide_left.stl" scale="0.001 0.001 0.001"/>
+            </geometry>
+        </collision>
+    </link>
+    <joint name="arm_1_camera_mount_joint" type="fixed">
+        <parent link="arm_1_7"/>
+        <child link="arm_1_camera_mount"/>
+        <origin xyz="0.17545 0.016874 -0.01" rpy="0 1.5707963 0"/>
+    </joint>
+    <link name="arm_2_camera_mount" >
+        <visual>
+            <origin xyz="0.0 0.0 0.0" rpy="0 0.0 0"/>
+            <geometry>
+                <mesh filename="package://repair_urdf/meshes/camera_supp_cover_sh1p2.stl" scale="0.001 0.001 0.001"/>
+            </geometry>
+            <material name="dark"/>
+        </visual>
+        <collision>
+            <origin xyz="0.0 0.0 0.0" rpy="0 0.0 0"/>
+            <geometry>
+                <mesh filename="package://repair_urdf/meshes/camera_supp_cover_sh1p2.stl" scale="0.001 0.001 0.001"/>
+            </geometry>
+        </collision>
+    </link>
+    <joint name="arm_2_camera_mount_joint" type="fixed">
+        <parent link="arm_2_7"/>
+        <child link="arm_2_camera_mount"/>
+        <!-- <origin xyz="0.2016 0.0168740 -0.00950" rpy="0 1.5707963 0"/> -->
+        <origin xyz="0.18145 0.00528118 -0.01350" rpy="0 1.5707963 0"/>
+    </joint>
+    <!--QUIRINO/GIANNIROS: here change the version for v1_2_research (small hand) or v1_wide (wide hand) and mixed_hands-->
     <xacro:softhands
         version="$(arg sh_version)"
-        position="0 0 0"
+        position="0.005 0 0"
         orientation="${PI}"
+        arm_1_parent="arm_1_angle_flange"
+        arm_2_parent="arm_2_angle_flange"
         fixed_hands="$(arg fixed_hands)">
     </xacro:softhands>

Commit message: old URDF for bimanual manipulation

File: repair_urdf/urdf/repair_full.urdf (robot description, URDF)
Before this commit: robot repair_full, 116 links, 115 joints
Joints:
- joint j_torso_base: limit lower=-0.8 upper=0.8 effort=147 velocity=2.0 -> lower=-0.8 upper=0.8 effort=147 velocity=2.2

Commit message: changes thursday morning

File: repair_urdf/urdf/repair_full.urdf (robot description, URDF)
Before this commit: robot repair_full, 128 links, 127 joints
Joints:
- joint left_hand_v1_wide_grasp_joint: origin xyz=0.03 -0.10 0.15 rpy=0 0 0 -> xyz=0.05 0 0.12 rpy=0 0 0
- joint right_hand_v1_2_research_grasp_joint: origin xyz=-0.06 0.03 0.16 rpy=0 0 1.57 -> xyz=-0.0 0.03 0.12 rpy=0 0 1.57
