Commit message: added new SoftHand submodule for v1.2 and wide hand

File: repair_urdf/urdf/gazebo/ignore_joint_softhand.xbot.xacro (robot description, xacro)
@@ -7,23 +7,44 @@
     <!--SUBGROUPS: Groups can also be formed by referencing to already defined group names-->
     <xacro:macro name="ignore_softhand_jnts" params="side type" >
-        <joint name="${side}_hand_${type}_thumb_knuckle_joint"/>
-        <joint name="${side}_hand_${type}_thumb_proximal_joint"/>
-        <joint name="${side}_hand_${type}_thumb_distal_joint"/>
-        <joint name="${side}_hand_${type}_index_distal_joint"/>
-        <joint name="${side}_hand_${type}_index_proximal_joint"/>
-        <joint name="${side}_hand_${type}_index_middle_joint"/>
-        <joint name="${side}_hand_${type}_index_distal_joint"/>
-        <joint name="${side}_hand_${type}_middle_distal_joint"/>
-        <joint name="${side}_hand_${type}_middle_proximal_joint"/>
-        <joint name="${side}_hand_${type}_middle_middle_joint"/>
-        <joint name="${side}_hand_${type}_middle_distal_joint"/>
-        <joint name="${side}_hand_${type}_ring_distal_joint"/>
-        <joint name="${side}_hand_${type}_ring_proximal_joint"/>
-        <joint name="${side}_hand_${type}_ring_middle_joint"/>
-        <joint name="${side}_hand_${type}_ring_distal_joint"/>
-        <joint name="${side}_hand_${type}_little_distal_joint"/>
-        <joint name="${side}_hand_${type}_little_proximal_joint"/>
-        <joint name="${side}_hand_${type}_little_middle_joint"/>
-        <joint name="${side}_hand_${type}_little_distal_joint"/>
+        <!--QUIRINO/GIANNIROS: modified joints that XBot ignores-->
+        <!-- V1_wide -->
+        <joint name="${side}hand${type}_palm_central_little_joint"/>
+        <joint name="${side}hand${type}_palm_central_thumb_joint"/>
+        <joint name="${side}hand${type}_palm_central_thumb_virtual_joint"/>
+        <joint name="${side}hand${type}_palm_central_little_virtual_joint"/>
+        <!-- V1_2_research -->
+        <joint name="${side}hand${type}_thumb_knuckle_joint"/>
+        <joint name="${side}hand${type}_thumb_proximal_joint"/>
+        <joint name="${side}hand${type}_thumb_proximal_virtual_joint"/>
+        <joint name="${side}hand${type}_thumb_distal_joint"/>
+        <joint name="${side}hand${type}_thumb_distal_virtual_joint"/>
+        <joint name="${side}hand${type}_index_knuckle_joint"/>
+        <joint name="${side}hand${type}_index_proximal_joint"/>
+        <joint name="${side}hand${type}_index_middle_joint"/>
+        <joint name="${side}hand${type}_index_distal_joint"/>
+        <joint name="${side}hand${type}_index_proximal_virtual_joint"/>
+        <joint name="${side}hand${type}_index_middle_virtual_joint"/>
+        <joint name="${side}hand${type}_index_distal_virtual_joint"/>
+        <joint name="${side}hand${type}_middle_knuckle_joint"/>
+        <joint name="${side}hand${type}_middle_proximal_joint"/>
+        <joint name="${side}hand${type}_middle_middle_joint"/>
+        <joint name="${side}hand${type}_middle_distal_joint"/>
+        <joint name="${side}hand${type}_middle_proximal_virtual_joint"/>
+        <joint name="${side}hand${type}_middle_middle_virtual_joint"/>
+        <joint name="${side}hand${type}_middle_distal_virtual_joint"/>
+        <joint name="${side}hand${type}_ring_knuckle_joint"/>
+        <joint name="${side}hand${type}_ring_proximal_joint"/>
+        <joint name="${side}hand${type}_ring_middle_joint"/>
+        <joint name="${side}hand${type}_ring_distal_joint"/>
+        <joint name="${side}hand${type}_ring_proximal_virtual_joint"/>
+        <joint name="${side}hand${type}_ring_middle_virtual_joint"/>
+        <joint name="${side}hand${type}_ring_distal_virtual_joint"/>
+        <joint name="${side}hand${type}_little_knuckle_joint"/>
+        <joint name="${side}hand${type}_little_proximal_joint"/>
+        <joint name="${side}hand${type}_little_middle_joint"/>
+        <joint name="${side}hand${type}_little_distal_joint"/>
+        <joint name="${side}hand${type}_little_proximal_virtual_joint"/>
+        <joint name="${side}hand${type}_little_middle_virtual_joint"/>
+        <joint name="${side}hand${type}_little_distal_virtual_joint"/>
     </xacro:macro>
 </robot>

File: repair_urdf/urdf/gazebo/xbot.gazebo.xacro (robot description, xacro)
@@ -24,7 +24,9 @@
             <pid name="j_arm_2_7" profile="small_mot"/>
         </pid>
-        <ignore_joints>
-            <xacro:ignore_softhand_jnts side="right" type="v1s"/>
-            <xacro:ignore_softhand_jnts side="left" type="v1s"/>
+         <ignore_joints>
+            <xacro:ignore_softhand_jnts side="right" type="v1_2_research"/>
+            <xacro:ignore_softhand_jnts side="left" type="v1_2_research"/>
+            <xacro:ignore_softhand_jnts side="right" type="v1_wide"/>
+            <xacro:ignore_softhand_jnts side="left" type="v1_wide"/>
         </ignore_joints>
     </plugin>

File: repair_urdf/urdf/repair_full.urdf.xacro (robot description, xacro)
@@ -35,5 +35,5 @@
                 rpy="${-Shoulder_1_roll} ${Shoulder_1_pitch} ${Shoulder_1_yaw}" />
       </xacro:repair_arm>
-    <xacro:softhands type="left"
+    <!-- <xacro:softhands type="left"
         version="v1.0_simple"
         parent="arm_1_7"
@@ -52,4 +52,11 @@
         operation_mode="0"
         fixed_hands="false">
+    </xacro:softhands> -->
+    <!--QUIRINO/GIANNIROS: here change the version for v1_2_research (small hand) or v1_wide (wide hand)-->
+    <xacro:softhands
+        version="v1_wide"
+        position="0 0 0"
+        orientation="${PI/2}"
+        fixed_hands="false">
     </xacro:softhands>
     <!-- <gazebo reference="table_top_link">
