Commit message: merged with mixed hands plugin

File: repair_moveit_config_v2/config/repair_full.srdf.xacro (robot description, xacro)
@@ -4,5 +4,6 @@
     A URDF file must exist for this robot as well, where the joints and the links that are referenced are defined
 -->
-<robot name="repair_full">
+<robot  xmlns:xacro="http://ros.org/wiki/xacro" name="repair_full">
+    <xacro:property name="sh_version" default="v1_2_research"/>
     <!--GROUPS: Representation of a set of joints and links. This can be useful for specifying DOF to plan for, defining arms, end effectors, etc-->
     <!--LINKS: When a link is specified, the parent joint of that link (if it exists) is automatically included-->

File: repair_srdf/srdf/repair_full.srdf.xacro (robot description, xacro)
@@ -33,17 +33,17 @@
     <group_state name="home" group="chains">
         <joint name="j_arm_1_1" value="-0.5"/>
-        <joint name="j_arm_1_2" value="-0.5"/>
+        <joint name="j_arm_1_2" value="-0.7"/>
         <joint name="j_arm_1_3" value="0.5"/>
-        <joint name="j_arm_1_4" value="-1.0"/>
+        <joint name="j_arm_1_4" value="-1.2"/>
         <joint name="j_arm_1_5" value="-0.5"/>
-        <joint name="j_arm_1_6" value="-0.5"/>
-        <joint name="j_arm_1_7" value="-1.0"/>
+        <joint name="j_arm_1_6" value="0.5"/>
+        <joint name="j_arm_1_7" value="0.5"/>
         <joint name="j_arm_2_1" value="0.5"/>
-        <joint name="j_arm_2_2" value="0.5"/>
+        <joint name="j_arm_2_2" value="0.7"/>
         <joint name="j_arm_2_3" value="-0.5"/>
-        <joint name="j_arm_2_4" value="1.0"/>
+        <joint name="j_arm_2_4" value="1.2"/>
         <joint name="j_arm_2_5" value="0.5"/>
-        <joint name="j_arm_2_6" value="0.5"/>
-        <joint name="j_arm_2_7" value="1.0"/>
+        <joint name="j_arm_2_6" value="-0.5"/>
+        <joint name="j_arm_2_7" value="-0.5"/>
         <!-- <xacro:softhand_homing side="right" type="v1s"/>
         <xacro:softhand_homing side="left" type="v1s"/> -->
