Commit message: merged with mixed hands plugin

File: repair_urdf/urdf/repair_full.urdf.xacro (robot description, xacro)
@@ -1,4 +1,5 @@
 <?xml version="1.0"?>
 <robot xmlns:xacro="http://ros.org/wiki/xacro" name="repair_full">
+    <xacro:arg name="sh_version" default="mixed_hands"/>
     <xacro:include filename="$(find softhands_description)/urdf/softhands.xacro" />
     <xacro:include filename="$(find repair_urdf)/urdf/conversions.urdf.xacro" />
@@ -35,7 +36,7 @@
                 rpy="${-Shoulder_1_roll} ${Shoulder_1_pitch} ${Shoulder_1_yaw}" />
       </xacro:repair_arm>
-    <!--QUIRINO/GIANNIROS: here change the version for v1_2_research (small hand) or v1_wide (wide hand)-->
+    <!--QUIRINO/GIANNIROS: here change the version for v1_2_research (small hand) or v1_wide (wide hand) and mixed-->
     <xacro:softhands
-        version="v1_2_research"
+        version="$(arg sh_version)"
         position="0 0 0"
         orientation="${PI/2}"

Commit message: fixed sh_version property for xacro:if in repair_full.srdf.xacro

File: repair_moveit_config_v2/config/repair_full.srdf.xacro (robot description, xacro)
@@ -5,5 +5,6 @@
 -->
 <robot  xmlns:xacro="http://ros.org/wiki/xacro" name="repair_full">
-    <xacro:property name="sh_version" default="v1_2_research"/>
+  <!-- QUIRINO: replaced default with arg value for xacro:if-->
+  <xacro:property name="sh_version" value="$(arg sh_version)"/>
     <!--GROUPS: Representation of a set of joints and links. This can be useful for specifying DOF to plan for, defining arms, end effectors, etc-->
     <!--LINKS: When a link is specified, the parent joint of that link (if it exists) is automatically included-->
