Commit message: bug fix

File: repair_moveit_config_v2/config/gazebo_repair_full.urdf (robot description, URDF)
Before this commit: robot repair_full, 75 links, 74 joints
Links:
- added link camera_bottom_screw_frame
- added link camera_color_frame
- added link camera_color_optical_frame
- added link camera_depth_frame
- added link camera_depth_optical_frame
- added link camera_left_ir_frame
- added link camera_left_ir_optical_frame
- added link camera_link, mass 0.564; collision box size=0.02505 0.09 0.025; visual mesh filename=package://repair_urdf/meshes/d435.dae
- added link camera_right_ir_frame
- added link camera_right_ir_optical_frame
- added link left_hand_v1s_grasp_link
- added link right_hand_v1s_grasp_link
- link arm_1_1: geometry collision sphere radius=0.05; collision sphere radius=0.05
- link arm_1_2: geometry collision sphere radius=0.05; collision sphere radius=0.05
- link arm_1_3: geometry collision sphere radius=0.05; collision sphere radius=0.05
- link arm_1_4: geometry collision sphere radius=0.05; collision sphere radius=0.05
- link arm_1_5: geometry collision sphere radius=0.05; collision sphere radius=0.05
- link arm_1_6: geometry collision sphere radius=0.07; visual mesh filename=package://repair_urdf/meshes/simplified/mesh_wrist-pitch.stl scale=0.001 -0.001 0.001
- link arm_1_7: geometry collision sphere radius=0.07; collision sphere radius=0.11
- link arm_2_1: geometry collision sphere radius=0.05; collision sphere radius=0.05
- link arm_2_2: geometry collision sphere radius=0.05; collision sphere radius=0.05
- link arm_2_3: geometry collision sphere radius=0.05; collision sphere radius=0.05
- link arm_2_4: geometry collision sphere radius=0.05; collision sphere radius=0.05
- link arm_2_5: geometry collision sphere radius=0.05; collision sphere radius=0.05
- link arm_2_6: geometry collision sphere radius=0.07; visual mesh filename=package://repair_urdf/meshes/simplified/mesh_wrist-pitch.stl scale=0.001 0.001 0.001
- link arm_2_7: geometry collision sphere radius=0.07; collision sphere radius=0.11
- link left_hand_v1s_index_distal_link: geometry visual mesh filename=package://softhands_description/meshes/softhands/v1.0/commo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
- link left_hand_v1s_index_knuckle_link: geometry visual mesh filename=package://softhands_description/meshes/softhands/v1.0/commo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
- link left_hand_v1s_index_middle_link: geometry visual mesh filename=package://softhands_description/meshes/softhands/v1.0/commo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
- link left_hand_v1s_index_proximal_link: geometry visual mesh filename=package://softhands_description/meshes/softhands/v1.0/commo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
- link left_hand_v1s_little_distal_link: geometry visual mesh filename=package://softhands_description/meshes/softhands/v1.0/commo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
- link left_hand_v1s_little_knuckle_link: geometry visual mesh filename=package://softhands_description/meshes/softhands/v1.0/commo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
- link left_hand_v1s_little_middle_link: geometry visual mesh filename=package://softhands_description/meshes/softhands/v1.0/commo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
- link left_hand_v1s_little_proximal_link: geometry visual mesh filename=package://softhands_description/meshes/softhands/v1.0/commo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
- link left_hand_v1s_middle_distal_link: geometry visual mesh filename=package://softhands_description/meshes/softhands/v1.0/commo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
- link left_hand_v1s_middle_knuckle_link: geometry visual mesh filename=package://softhands_description/meshes/softhands/v1.0/commo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
- link left_hand_v1s_middle_middle_link: geometry visual mesh filename=package://softhands_description/meshes/softhands/v1.0/commo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
- link left_hand_v1s_middle_proximal_link: geometry visual mesh filename=package://softhands_description/meshes/softhands/v1.0/commo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
- link left_hand_v1s_palm_link: geometry visual mesh filename=package://softhands_description/meshes/softhands/v1.0/left/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; visual mesh filename=package://softhands_description/meshes/softhands/v1.0/left/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
- link left_hand_v1s_ring_distal_link: geometry visual mesh filename=package://softhands_description/meshes/softhands/v1.0/commo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
- link left_hand_v1s_ring_knuckle_link: geometry visual mesh filename=package://softhands_description/meshes/softhands/v1.0/commo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
- link left_hand_v1s_ring_middle_link: geometry visual mesh filename=package://softhands_description/meshes/softhands/v1.0/commo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
- link left_hand_v1s_ring_proximal_link: geometry visual mesh filename=package://softhands_description/meshes/softhands/v1.0/commo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
- link left_hand_v1s_thumb_distal_link: geometry visual mesh filename=package://softhands_description/meshes/softhands/v1.0/commo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
- link left_hand_v1s_thumb_knuckle_link: geometry visual mesh filename=package://softhands_description/meshes/softhands/v1.0/left/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
- link left_hand_v1s_thumb_proximal_link: geometry visual mesh filename=package://softhands_description/meshes/softhands/v1.0/commo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
- link right_hand_v1s_index_distal_link: geometry visual mesh filename=package://softhands_description/meshes/softhands/v1.0/commo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
- link right_hand_v1s_index_knuckle_link: geometry visual mesh filename=package://softhands_description/meshes/softhands/v1.0/commo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
- link right_hand_v1s_index_middle_link: geometry visual mesh filename=package://softhands_description/meshes/softhands/v1.0/commo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
- link right_hand_v1s_index_proximal_link: geometry visual mesh filename=package://softhands_description/meshes/softhands/v1.0/commo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
- link right_hand_v1s_little_distal_link: geometry visual mesh filename=package://softhands_description/meshes/softhands/v1.0/commo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
- link right_hand_v1s_little_knuckle_link: geometry visual mesh filename=package://softhands_description/meshes/softhands/v1.0/commo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
- link right_hand_v1s_little_middle_link: geometry visual mesh filename=package://softhands_description/meshes/softhands/v1.0/commo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
- link right_hand_v1s_little_proximal_link: geometry visual mesh filename=package://softhands_description/meshes/softhands/v1.0/commo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
- link right_hand_v1s_middle_distal_link: geometry visual mesh filename=package://softhands_description/meshes/softhands/v1.0/commo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
- link right_hand_v1s_middle_knuckle_link: geometry visual mesh filename=package://softhands_description/meshes/softhands/v1.0/commo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
- link right_hand_v1s_middle_middle_link: geometry visual mesh filename=package://softhands_description/meshes/softhands/v1.0/commo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
- link right_hand_v1s_middle_proximal_link: geometry visual mesh filename=package://softhands_description/meshes/softhands/v1.0/commo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
- link right_hand_v1s_palm_link: geometry visual mesh filename=package://softhands_description/meshes/softhands/v1.0/right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; visual mesh filename=package://softhands_description/meshes/softhands/v1.0/right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
- link right_hand_v1s_ring_distal_link: geometry visual mesh filename=package://softhands_description/meshes/softhands/v1.0/commo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
- link right_hand_v1s_ring_knuckle_link: geometry visual mesh filename=package://softhands_description/meshes/softhands/v1.0/commo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
- link right_hand_v1s_ring_middle_link: geometry visual mesh filename=package://softhands_description/meshes/softhands/v1.0/commo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
- link right_hand_v1s_ring_proximal_link: geometry visual mesh filename=package://softhands_description/meshes/softhands/v1.0/commo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
- link right_hand_v1s_thumb_distal_link: geometry visual mesh filename=package://softhands_description/meshes/softhands/v1.0/commo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
- link right_hand_v1s_thumb_knuckle_link: geometry visual mesh filename=package://softhands_description/meshes/softhands/v1.0/right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
- link right_hand_v1s_thumb_proximal_link: geometry visual mesh filename=package://softhands_description/meshes/softhands/v1.0/commo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
Joints:
- added joint camera_color_joint: type fixed, parent camera_depth_frame, child camera_color_frame, origin xyz=0 0.015 0 rpy=0 0 0
- added joint camera_color_optical_joint: type fixed, parent camera_color_frame, child camera_color_optical_frame, origin xyz=0 0 0 rpy=-1.5707963267948966 0 -1.5707963267948966
- added joint camera_depth_joint: type fixed, parent camera_link, child camera_depth_frame, origin xyz=0 0 0 rpy=0 0 0
- added joint camera_depth_optical_joint: type fixed, parent camera_depth_frame, child camera_depth_optical_frame, origin xyz=0 0 0 rpy=-1.5707963267948966 0 -1.5707963267948966
- added joint camera_joint: type fixed, parent torso_1, child camera_bottom_screw_frame, origin xyz=0.0857 0.0000476009 -0.273184 rpy=0.0009783 1.1836725 0
- added joint camera_left_ir_joint: type fixed, parent camera_depth_frame, child camera_left_ir_frame, origin xyz=0 0.0 0 rpy=0 0 0
- added joint camera_left_ir_optical_joint: type fixed, parent camera_left_ir_frame, child camera_left_ir_optical_frame, origin xyz=0 0 0 rpy=-1.5707963267948966 0 -1.5707963267948966
- added joint camera_link_joint: type fixed, parent camera_bottom_screw_frame, child camera_link, origin xyz=0 0.0175 0.0125 rpy=0 0 0
- added joint camera_right_ir_joint: type fixed, parent camera_depth_frame, child camera_right_ir_frame, origin xyz=0 -0.05 0 rpy=0 0 0
- added joint camera_right_ir_optical_joint: type fixed, parent camera_right_ir_frame, child camera_right_ir_optical_frame, origin xyz=0 0 0 rpy=-1.5707963267948966 0 -1.5707963267948966
- added joint left_hand_v1s_grasp_joint: type fixed, parent left_hand_v1s_palm_link, child left_hand_v1s_grasp_link, origin xyz=0.03 -0.06 0.10 rpy=0 0 0
- added joint right_hand_v1s_grasp_joint: type fixed, parent right_hand_v1s_palm_link, child right_hand_v1s_grasp_link, origin xyz=0.03 0.06 0.10 rpy=0 0 0
- joint left_hand_base_joint: origin xyz=0 0 -0.015 rpy=0 0.0 3.14159265359 -> xyz=0 0 0 rpy=0 0.0 1.570796326795
- joint right_hand_base_joint: origin xyz=0 -0.013900 -0.015 rpy=0 0 3.14159265359 -> xyz=0 0 0 rpy=0 0 -1.570796326795

File: repair_urdf/urdf/repair_arm_collision.urdf.xacro (robot description, xacro)
@@ -77,5 +77,5 @@
     </xacro:if>
     <xacro:unless value="${isMesh}">
-      <xacro:collision_sphere origin="0 0 0.0" radius="0.05" />
+      <xacro:collision_sphere origin="0.0 0 0.0" radius="0.07" />
       <xacro:collision_sphere origin="${rot*0.01} 0 0.14" radius="0.11" />
     </xacro:unless>

File: repair_urdf/urdf/repair_full.urdf.xacro (robot description, xacro)
@@ -18,5 +18,5 @@
     <xacro:include filename="$(find repair_urdf)/urdf/repair_hand_transmission.xacro" />
     <!-- property for enabling meshes for collision -->
-    <xacro:property name="useCollisionMesh" value="false" />
+    <xacro:property name="useCollisionMesh" value="true" />
     <link name="world"/>
     <xacro:repair_cage parent="world">
