Commit message: sliding guide working on arm_1 group

File: repair_moveit_config_v2/config/gazebo_repair_full.urdf (robot description, URDF)
Before this commit: robot repair_full, 120 links, 119 joints
Links:
- removed link left_hand_v1_2_research_grasp_link
- removed link left_hand_v1_2_research_index_distal_link
- removed link left_hand_v1_2_research_index_distal_virtual_link
- removed link left_hand_v1_2_research_index_knuckle_link
- removed link left_hand_v1_2_research_index_middle_link
- removed link left_hand_v1_2_research_index_middle_virtual_link
- removed link left_hand_v1_2_research_index_proximal_link
- removed link left_hand_v1_2_research_index_proximal_virtual_link
- removed link left_hand_v1_2_research_iso_link
- removed link left_hand_v1_2_research_little_distal_link
- removed link left_hand_v1_2_research_little_distal_virtual_link
- removed link left_hand_v1_2_research_little_knuckle_link
- removed link left_hand_v1_2_research_little_middle_link
- removed link left_hand_v1_2_research_little_middle_virtual_link
- removed link left_hand_v1_2_research_little_proximal_link
- removed link left_hand_v1_2_research_little_proximal_virtual_link
- removed link left_hand_v1_2_research_middle_distal_link
- removed link left_hand_v1_2_research_middle_distal_virtual_link
- removed link left_hand_v1_2_research_middle_knuckle_link
- removed link left_hand_v1_2_research_middle_middle_link
- removed link left_hand_v1_2_research_middle_middle_virtual_link
- removed link left_hand_v1_2_research_middle_proximal_link
- removed link left_hand_v1_2_research_middle_proximal_virtual_link
- removed link left_hand_v1_2_research_palm_link
- removed link left_hand_v1_2_research_ring_distal_link
- removed link left_hand_v1_2_research_ring_distal_virtual_link
- removed link left_hand_v1_2_research_ring_knuckle_link
- removed link left_hand_v1_2_research_ring_middle_link
- removed link left_hand_v1_2_research_ring_middle_virtual_link
- removed link left_hand_v1_2_research_ring_proximal_link
- removed link left_hand_v1_2_research_ring_proximal_virtual_link
- removed link left_hand_v1_2_research_thumb_distal_link
- removed link left_hand_v1_2_research_thumb_distal_virtual_link
- removed link left_hand_v1_2_research_thumb_knuckle_link
- removed link left_hand_v1_2_research_thumb_proximal_link
- removed link left_hand_v1_2_research_thumb_proximal_virtual_link
- added link arm_1_angle_flange; collision mesh filename=package://repair_urdf/meshes/angle_flange_90.stl scale=0.001 0.001 0.001; visual mesh filename=package://repair_urdf/meshes/angle_flange_90.stl scale=0.001 0.001 0.001
- added link arm_1_camera_mount; collision mesh filename=package://repair_urdf/meshes/camera_supp_cover_wide_left.stl scale=0.001 0.001 0.001; visual mesh filename=package://repair_urdf/meshes/camera_supp_cover_wide_left.stl scale=0.001 0.001 0.001
- added link arm_2_angle_flange; collision mesh filename=package://repair_urdf/meshes/angle_flange_90.stl scale=0.001 0.001 0.001; visual mesh filename=package://repair_urdf/meshes/angle_flange_90.stl scale=0.001 0.001 0.001
- added link arm_2_camera_mount; collision mesh filename=package://repair_urdf/meshes/camera_supp_cover_sh1p2.stl scale=0.001 0.001 0.001; visual mesh filename=package://repair_urdf/meshes/camera_supp_cover_sh1p2.stl scale=0.001 0.001 0.001
- added link left_hand_v1_wide_grasp_link
- added link left_hand_v1_wide_index_distal_link, mass 0.012475845; collision mesh filename=package://softhands_description/meshes/v1_wide/left/phalanx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 scale=0.0009 0.0009 0.0009; visual mesh filename=package://softhands_description/meshes/v1_wide/left/phalanx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 scale=0.001 0.001 0.001
- added link left_hand_v1_wide_index_distal_virtual_link, mass 0.012475845
- added link left_hand_v1_wide_index_knuckle_link, mass 7.4913242e-03; collision mesh filename=package://softhands_description/meshes/v1_wide/left/phalanx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 scale=0.0009 0.0009 0.0009; visual mesh filename=package://softhands_description/meshes/v1_wide/left/phalanx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 scale=0.001 0.001 0.001
- added link left_hand_v1_wide_index_middle_link, mass 0.024190505; collision mesh filename=package://softhands_description/meshes/v1_wide/left/phalanx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 scale=0.0009 0.0009 0.0009; visual mesh filename=package://softhands_description/meshes/v1_wide/left/phalanx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 scale=0.001 0.001 0.001
- added link left_hand_v1_wide_index_middle_virtual_link, mass 0.024190505
- added link left_hand_v1_wide_index_proximal_link, mass 0.024190505; collision mesh filename=package://softhands_description/meshes/v1_wide/left/phalanx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 scale=0.0009 0.0009 0.0009; visual mesh filename=package://softhands_description/meshes/v1_wide/left/phalanx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 scale=0.001 0.001 0.001
- added link left_hand_v1_wide_index_proximal_virtual_link, mass 0.024190505
- added link left_hand_v1_wide_little_distal_link, mass 0.012475845; collision mesh filename=package://softhands_description/meshes/v1_wide/left/phalanx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 scale=0.0009 0.0009 0.0009; visual mesh filename=package://softhands_description/meshes/v1_wide/left/phalanx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 scale=0.001 0.001 0.001
- added link left_hand_v1_wide_little_distal_virtual_link, mass 0.012475845
- added link left_hand_v1_wide_little_knuckle_link, mass 7.4913242e-03; collision mesh filename=package://softhands_description/meshes/v1_wide/left/phalanx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 scale=0.0009 0.0009 0.0009; visual mesh filename=package://softhands_description/meshes/v1_wide/left/phalanx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 scale=0.001 0.001 0.001
- added link left_hand_v1_wide_little_middle_link, mass 0.024190505; collision mesh filename=package://softhands_description/meshes/v1_wide/left/phalanx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 scale=0.0009 0.0009 0.0009; visual mesh filename=package://softhands_description/meshes/v1_wide/left/phalanx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 scale=0.001 0.001 0.001
- added link left_hand_v1_wide_little_middle_virtual_link, mass 0.024190505
- added link left_hand_v1_wide_little_proximal_link, mass 0.024190505; collision mesh filename=package://softhands_description/meshes/v1_wide/left/phalanx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 scale=0.0009 0.0009 0.0009; visual mesh filename=package://softhands_description/meshes/v1_wide/left/phalanx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 scale=0.001 0.001 0.001
- added link left_hand_v1_wide_little_proximal_virtual_link, mass 0.024190505
- added link left_hand_v1_wide_middle_distal_link, mass 0.012475845; collision mesh filename=package://softhands_description/meshes/v1_wide/left/phalanx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 scale=0.0009 0.0009 0.0009; visual mesh filename=package://softhands_description/meshes/v1_wide/left/phalanx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 scale=0.001 0.001 0.001
- added link left_hand_v1_wide_middle_distal_virtual_link, mass 0.012475845
- added link left_hand_v1_wide_middle_knuckle_link, mass 7.4913242e-03; collision mesh filename=package://softhands_description/meshes/v1_wide/left/phalanx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 scale=0.0009 0.0009 0.0009; visual mesh filename=package://softhands_description/meshes/v1_wide/left/phalanx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 scale=0.001 0.001 0.001
- added link left_hand_v1_wide_middle_middle_link, mass 0.024190505; collision mesh filename=package://softhands_description/meshes/v1_wide/left/phalanx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 scale=0.0009 0.0009 0.0009; visual mesh filename=package://softhands_description/meshes/v1_wide/left/phalanx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 scale=0.001 0.001 0.001
- added link left_hand_v1_wide_middle_middle_virtual_link, mass 0.024190505
- added link left_hand_v1_wide_middle_proximal_link, mass 0.024190505; collision mesh filename=package://softhands_description/meshes/v1_wide/left/phalanx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 scale=0.0009 0.0009 0.0009; visual mesh filename=package://softhands_description/meshes/v1_wide/left/phalanx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 scale=0.001 0.001 0.001
- added link left_hand_v1_wide_middle_proximal_virtual_link, mass 0.024190505
- added link left_hand_v1_wide_palm_central_link, mass 0.18654307333333334; collision mesh filename=package://softhands_description/meshes/v1_wide/left/palm_ce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 scale=0.0009 0.0009 0.0009; visual mesh filename=package://softhands_description/meshes/v1_wide/left/palm_ce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 scale=0.001 0.001 0.001
- added link left_hand_v1_wide_palm_central_little_link, mass 0.18654307333333334
- added link left_hand_v1_wide_palm_central_thumb_link, mass 0.18654307333333334
- added link left_hand_v1_wide_palm_little_link, mass 0.17998957; collision mesh filename=package://softhands_description/meshes/v1_wide/left/palm_li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 scale=0.0009 0.0009 0.0009; visual mesh filename=package://softhands_description/meshes/v1_wide/left/palm_li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 scale=0.001 0.001 0.001
- added link left_hand_v1_wide_palm_thumb_link, mass 0.092767; collision mesh filename=package://softhands_description/meshes/v1_wide/left/palm_th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 scale=0.001 0.001 0.001; visual mesh filename=package://softhands_description/meshes/v1_wide/left/palm_th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 scale=0.001 0.001 0.001
- added link left_hand_v1_wide_palm_thumb_support_link, mass 1.6408860e-02; collision mesh filename=package://softhands_description/meshes/v1_wide/left/thumb_s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 scale=0.0009 0.0009 0.0009; visual mesh filename=package://softhands_description/meshes/v1_wide/left/thumb_s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 scale=0.001 0.001 0.001
- added link left_hand_v1_wide_ring_distal_link, mass 0.012475845; collision mesh filename=package://softhands_description/meshes/v1_wide/left/phalanx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 scale=0.0009 0.0009 0.0009; visual mesh filename=package://softhands_description/meshes/v1_wide/left/phalanx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 scale=0.001 0.001 0.001
- added link left_hand_v1_wide_ring_distal_virtual_link, mass 0.012475845
- added link left_hand_v1_wide_ring_knuckle_link, mass 7.4913242e-03; collision mesh filename=package://softhands_description/meshes/v1_wide/left/phalanx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 scale=0.0009 0.0009 0.0009; visual mesh filename=package://softhands_description/meshes/v1_wide/left/phalanx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 scale=0.001 0.001 0.001
- added link left_hand_v1_wide_ring_middle_link, mass 0.024190505; collision mesh filename=package://softhands_description/meshes/v1_wide/left/phalanx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 scale=0.0009 0.0009 0.0009; visual mesh filename=package://softhands_description/meshes/v1_wide/left/phalanx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 scale=0.001 0.001 0.001
- added link left_hand_v1_wide_ring_middle_virtual_link, mass 0.024190505
- added link left_hand_v1_wide_ring_proximal_link, mass 0.024190505; collision mesh filename=package://softhands_description/meshes/v1_wide/left/phalanx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 scale=0.0009 0.0009 0.0009; visual mesh filename=package://softhands_description/meshes/v1_wide/left/phalanx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 scale=0.001 0.001 0.001
- added link left_hand_v1_wide_ring_proximal_virtual_link, mass 0.024190505
- added link left_hand_v1_wide_thumb_distal_link, mass 0.023674554; collision mesh filename=package://softhands_description/meshes/v1_wide/left/phalanx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 scale=0.0009 0.0009 0.0009; visual mesh filename=package://softhands_description/meshes/v1_wide/left/phalanx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 scale=0.001 0.001 0.001
- added link left_hand_v1_wide_thumb_distal_virtual_link, mass 0.023674554
- added link left_hand_v1_wide_thumb_knuckle_link, mass 2.4657976e-02; collision mesh filename=package://softhands_description/meshes/v1_wide/left/phalanx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 scale=0.0009 0.0009 0.0009; visual mesh filename=package://softhands_description/meshes/v1_wide/left/phalanx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 scale=0.001 0.001 0.001
- added link left_hand_v1_wide_thumb_proximal_link, mass 0.033679189; collision mesh filename=package://softhands_description/meshes/v1_wide/left/phalanx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 scale=0.0009 0.0009 0.0009; visual mesh filename=package://softhands_description/meshes/v1_wide/left/phalanx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 scale=0.001 0.001 0.001
- added link left_hand_v1_wide_thumb_proximal_virtual_link, mass 0.033679189
- link leg1_link: mass 0.1 -> None; geometry collision cylinder length=0.978 radius=0.02; visual cylinder length=0.978 radius=0.02
- link leg2_link: mass 0.1 -> None; geometry collision cylinder length=0.978 radius=0.02; visual cylinder length=0.978 radius=0.02
- link leg3_link: mass 0.1 -> None; geometry collision cylinder length=0.978 radius=0.02; visual cylinder length=0.978 radius=0.02
- link leg4_link: mass 0.1 -> None; geometry collision cylinder length=0.978 radius=0.02; visual cylinder length=0.978 radius=0.02
- link obar1_link: mass 0.1 -> None
- link obar2_link: mass 0.1 -> None
- link obar3_link: mass 0.1 -> None
- link obar4_link: mass 0.1 -> None
- link sliding_guide_link: mass 0.1 -> None; geometry collision box size=0.001 1.0 2.5; visual box size=0.001 0.4 2.5
- link table_top_link: mass 0.1 -> None; geometry collision box size=1.0 2.5 0.028; visual box size=1.0 2.5 0.028
- link vbar1_link: mass 0.1 -> None
- link vbar2_link: mass 0.1 -> None
- link vbar3_link: mass 0.1 -> None
- link vbar4_link: mass 0.1 -> None
Joints:
- removed joint left_hand_v1_2_research_grasp_joint
- removed joint left_hand_v1_2_research_index_distal_joint
- removed joint left_hand_v1_2_research_index_distal_virtual_joint
- removed joint left_hand_v1_2_research_index_knuckle_joint
- removed joint left_hand_v1_2_research_index_middle_joint
- removed joint left_hand_v1_2_research_index_middle_virtual_joint
- removed joint left_hand_v1_2_research_index_proximal_joint
- removed joint left_hand_v1_2_research_index_proximal_virtual_joint
- removed joint left_hand_v1_2_research_iso_joint
- removed joint left_hand_v1_2_research_little_distal_joint
- removed joint left_hand_v1_2_research_little_distal_virtual_joint
- removed joint left_hand_v1_2_research_little_knuckle_joint
- removed joint left_hand_v1_2_research_little_middle_joint
- removed joint left_hand_v1_2_research_little_middle_virtual_joint
- removed joint left_hand_v1_2_research_little_proximal_joint
- removed joint left_hand_v1_2_research_little_proximal_virtual_joint
- removed joint left_hand_v1_2_research_middle_distal_joint
- removed joint left_hand_v1_2_research_middle_distal_virtual_joint
- removed joint left_hand_v1_2_research_middle_knuckle_joint
- removed joint left_hand_v1_2_research_middle_middle_joint
- removed joint left_hand_v1_2_research_middle_middle_virtual_joint
- removed joint left_hand_v1_2_research_middle_proximal_joint
- removed joint left_hand_v1_2_research_middle_proximal_virtual_joint
- removed joint left_hand_v1_2_research_palm_joint
- removed joint left_hand_v1_2_research_ring_distal_joint
- removed joint left_hand_v1_2_research_ring_distal_virtual_joint
- removed joint left_hand_v1_2_research_ring_knuckle_joint
- removed joint left_hand_v1_2_research_ring_middle_joint
- removed joint left_hand_v1_2_research_ring_middle_virtual_joint
- removed joint left_hand_v1_2_research_ring_proximal_joint
- removed joint left_hand_v1_2_research_ring_proximal_virtual_joint
- removed joint left_hand_v1_2_research_thumb_distal_joint
- removed joint left_hand_v1_2_research_thumb_distal_virtual_joint
- removed joint left_hand_v1_2_research_thumb_knuckle_joint
- removed joint left_hand_v1_2_research_thumb_proximal_joint
- removed joint left_hand_v1_2_research_thumb_proximal_virtual_joint
- added joint arm_1_angle_flange_joint: type fixed, parent arm_1_7, child arm_1_angle_flange, origin xyz=0.0425 0 0.0430 rpy=0 1.5707963 0
- added joint arm_1_camera_mount_joint: type fixed, parent arm_1_7, child arm_1_camera_mount, origin xyz=0.17545 0.016874 -0.01 rpy=0 1.5707963 0
- added joint arm_2_angle_flange_joint: type fixed, parent arm_2_7, child arm_2_angle_flange, origin xyz=0.0425 0 0.0380 rpy=0 1.5707963 0
- added joint arm_2_camera_mount_joint: type fixed, parent arm_2_7, child arm_2_camera_mount, origin xyz=0.18145 0.00528118 -0.01350 rpy=0 1.5707963 0
- added joint left_hand_v1_wide_grasp_joint: type fixed, parent left_hand_v1_wide_palm_central_link, child left_hand_v1_wide_grasp_link, origin xyz=0.03 -0.10 0.15 rpy=0 0 0
- added joint left_hand_v1_wide_index_distal_joint: type fixed, parent left_hand_v1_wide_index_distal_virtual_link, child left_hand_v1_wide_index_distal_link, origin xyz=9e-3 0 0 rpy=0 0 0, axis 0 0 1, limit lower=0 upper=0.785398 effort=30 velocity=0.0
- added joint left_hand_v1_wide_index_distal_virtual_joint: type fixed, parent left_hand_v1_wide_index_middle_link, child left_hand_v1_wide_index_distal_virtual_link, origin xyz=41e-3 0 0 rpy=0 0 0, axis 0 0 1, limit lower=0 upper=0.785398 effort=30 velocity=0.0
- added joint left_hand_v1_wide_index_knuckle_joint: type fixed, parent left_hand_v1_wide_palm_central_link, child left_hand_v1_wide_index_knuckle_link, origin xyz=5e-3 -44.8953e-3 112.230e-3 rpy=0.1748327 0 0 , axis 0 1 0, limit lower=0.0 upper=0.01 effort=30 velocity=0.0
- added joint left_hand_v1_wide_index_middle_joint: type fixed, parent left_hand_v1_wide_index_middle_virtual_link, child left_hand_v1_wide_index_middle_link, origin xyz=9e-3 0 0 rpy=0 0 0, axis 0 0 1, limit lower=0 upper=0.785398 effort=30 velocity=0.0
- added joint left_hand_v1_wide_index_middle_virtual_joint: type fixed, parent left_hand_v1_wide_index_proximal_link, child left_hand_v1_wide_index_middle_virtual_link, origin xyz=41e-3 0 0 rpy=0 0 0, axis 0 0 1, limit lower=0 upper=0.785398 effort=30 velocity=0.0
- added joint left_hand_v1_wide_index_proximal_joint: type fixed, parent left_hand_v1_wide_index_proximal_virtual_link, child left_hand_v1_wide_index_proximal_link, origin xyz=9e-3 0 0 rpy=0 0 0, axis 0 0 1, limit lower=0 upper=0.785398 effort=30 velocity=0.0
- added joint left_hand_v1_wide_index_proximal_virtual_joint: type fixed, parent left_hand_v1_wide_index_knuckle_link, child left_hand_v1_wide_index_proximal_virtual_link, origin xyz= -6.5e-3 0 24e-3 rpy=-1.5707963 -1.5707963 0, axis 0 0 1, limit lower=0 upper=0.785398 effort=30 velocity=0.0
- added joint left_hand_v1_wide_little_distal_joint: type fixed, parent left_hand_v1_wide_little_distal_virtual_link, child left_hand_v1_wide_little_distal_link, origin xyz=9e-3 0 0 rpy=0 0 0, axis 0 0 1, limit lower=0 upper=0.785398 effort=30 velocity=0.0
- added joint left_hand_v1_wide_little_distal_virtual_joint: type fixed, parent left_hand_v1_wide_little_middle_link, child left_hand_v1_wide_little_distal_virtual_link, origin xyz=41e-3 0 0 rpy=0 0 0, axis 0 0 1, limit lower=0 upper=0.785398 effort=30 velocity=0.0
- added joint left_hand_v1_wide_little_knuckle_joint: type fixed, parent left_hand_v1_wide_palm_little_link, child left_hand_v1_wide_little_knuckle_link, origin xyz=39.2985e-3 5e-3 -34.8419e-3 rpy=2.792527 0 1.5707963 , axis 0 1 0, limit lower=0.0 upper=0.01 effort=30 velocity=0.0
- added joint left_hand_v1_wide_little_middle_joint: type fixed, parent left_hand_v1_wide_little_middle_virtual_link, child left_hand_v1_wide_little_middle_link, origin xyz=9e-3 0 0 rpy=0 0 0, axis 0 0 1, limit lower=0 upper=0.785398 effort=30 velocity=0.0
- added joint left_hand_v1_wide_little_middle_virtual_joint: type fixed, parent left_hand_v1_wide_little_proximal_link, child left_hand_v1_wide_little_middle_virtual_link, origin xyz=41e-3 0 0 rpy=0 0 0, axis 0 0 1, limit lower=0 upper=0.785398 effort=30 velocity=0.0
- added joint left_hand_v1_wide_little_proximal_joint: type fixed, parent left_hand_v1_wide_little_proximal_virtual_link, child left_hand_v1_wide_little_proximal_link, origin xyz=9e-3 0 0 rpy=0 0 0, axis 0 0 1, limit lower=0 upper=0.785398 effort=30 velocity=0.0
- added joint left_hand_v1_wide_little_proximal_virtual_joint: type fixed, parent left_hand_v1_wide_little_knuckle_link, child left_hand_v1_wide_little_proximal_virtual_link, origin xyz= -6.5e-3 0 24e-3 rpy=-1.5707963 -1.5707963 0, axis 0 0 1, limit lower=0 upper=0.785398 effort=30 velocity=0.0
- added joint left_hand_v1_wide_middle_distal_joint: type fixed, parent left_hand_v1_wide_middle_distal_virtual_link, child left_hand_v1_wide_middle_distal_link, origin xyz=9e-3 0 0 rpy=0 0 0, axis 0 0 1, limit lower=0 upper=0.785398 effort=30 velocity=0.0
- added joint left_hand_v1_wide_middle_distal_virtual_joint: type fixed, parent left_hand_v1_wide_middle_middle_link, child left_hand_v1_wide_middle_distal_virtual_link, origin xyz=41e-3 0 0 rpy=0 0 0, axis 0 0 1, limit lower=0 upper=0.785398 effort=30 velocity=0.0
- added joint left_hand_v1_wide_middle_knuckle_joint: type fixed, parent left_hand_v1_wide_palm_central_link, child left_hand_v1_wide_middle_knuckle_link, origin xyz=5e-3 -12.5e-3 115e-3 rpy=0 0 0 , axis 0 1 0, limit lower=0.0 upper=0.01 effort=30 velocity=0.0
- added joint left_hand_v1_wide_middle_middle_joint: type fixed, parent left_hand_v1_wide_middle_middle_virtual_link, child left_hand_v1_wide_middle_middle_link, origin xyz=9e-3 0 0 rpy=0 0 0, axis 0 0 1, limit lower=0 upper=0.785398 effort=30 velocity=0.0
- added joint left_hand_v1_wide_middle_middle_virtual_joint: type fixed, parent left_hand_v1_wide_middle_proximal_link, child left_hand_v1_wide_middle_middle_virtual_link, origin xyz=41e-3 0 0 rpy=0 0 0, axis 0 0 1, limit lower=0 upper=0.785398 effort=30 velocity=0.0
- added joint left_hand_v1_wide_middle_proximal_joint: type fixed, parent left_hand_v1_wide_middle_proximal_virtual_link, child left_hand_v1_wide_middle_proximal_link, origin xyz=9e-3 0 0 rpy=0 0 0, axis 0 0 1, limit lower=0 upper=0.785398 effort=30 velocity=0.0
- added joint left_hand_v1_wide_middle_proximal_virtual_joint: type fixed, parent left_hand_v1_wide_middle_knuckle_link, child left_hand_v1_wide_middle_proximal_virtual_link, origin xyz= -6.5e-3 0 24e-3 rpy=-1.5707963 -1.5707963 0, axis 0 0 1, limit lower=0 upper=0.785398 effort=30 velocity=0.0
- added joint left_hand_v1_wide_palm_central_joint: type fixed, parent arm_1_angle_flange, child left_hand_v1_wide_palm_central_link, origin xyz=0.005 0 0 rpy=0 0 3.14159265359
- added joint left_hand_v1_wide_palm_central_little_joint: type fixed, parent left_hand_v1_wide_palm_central_link, child left_hand_v1_wide_palm_central_little_link, origin xyz= -0.0000000091 10.6603e-3 66.1817e-3 rpy=3.1415927 -0.1745327 1.5707963, axis 0 0 1, limit lower=0.0 upper=0.17 effort=100 velocity=0.00
- added joint left_hand_v1_wide_palm_central_little_virtual_joint: type fixed, parent left_hand_v1_wide_palm_central_little_link, child left_hand_v1_wide_palm_little_link, origin xyz=12e-3 4.66576e-08 0 rpy=0 0 0 , axis 0 0 1, limit lower=0 upper=0.17 effort=30 velocity=0.0
- added joint left_hand_v1_wide_palm_central_thumb_joint: type fixed, parent left_hand_v1_wide_palm_central_link, child left_hand_v1_wide_palm_central_thumb_link, origin xyz= -0.0000000021 -32.5059e-3 39.6398e-3 rpy=0.3490656 0.0 0.0, axis 0 0 1, limit lower=0 upper=0.17 effort=30 velocity=0.0
- added joint left_hand_v1_wide_palm_central_thumb_virtual_joint: type fixed, parent left_hand_v1_wide_palm_central_thumb_link, child left_hand_v1_wide_palm_thumb_link, origin xyz=-0.0000454746e-3 -12e-3 0 rpy=0 0 0 , axis 0 0 1, limit lower=0 upper=0.17 effort=30 velocity=0.0
- added joint left_hand_v1_wide_palm_thumb_support_joint: type fixed, parent left_hand_v1_wide_palm_thumb_link, child left_hand_v1_wide_palm_thumb_support_link, origin xyz=5.0e-3 -24.2343e-3 9.13010e-3 rpy=1.5707963 -0.5235992 1.5707963
- added joint left_hand_v1_wide_ring_distal_joint: type fixed, parent left_hand_v1_wide_ring_distal_virtual_link, child left_hand_v1_wide_ring_distal_link, origin xyz=9e-3 0 0 rpy=0 0 0, axis 0 0 1, limit lower=0 upper=0.785398 effort=30 velocity=0.0
- added joint left_hand_v1_wide_ring_distal_virtual_joint: type fixed, parent left_hand_v1_wide_ring_middle_link, child left_hand_v1_wide_ring_distal_virtual_link, origin xyz=41e-3 0 0 rpy=0 0 0, axis 0 0 1, limit lower=0 upper=0.785398 effort=30 velocity=0.0
- added joint left_hand_v1_wide_ring_knuckle_joint: type fixed, parent left_hand_v1_wide_palm_little_link, child left_hand_v1_wide_ring_knuckle_link, origin xyz= 8.6355e-3 5e-3 -44.4863e-3 rpy=2.8797933 0 1.5707963 , axis 0 1 0, limit lower=0.0 upper=0.01 effort=30 velocity=0.0
- added joint left_hand_v1_wide_ring_middle_joint: type fixed, parent left_hand_v1_wide_ring_middle_virtual_link, child left_hand_v1_wide_ring_middle_link, origin xyz=9e-3 0 0 rpy=0 0 0, axis 0 0 1, limit lower=0 upper=0.785398 effort=30 velocity=0.0
- added joint left_hand_v1_wide_ring_middle_virtual_joint: type fixed, parent left_hand_v1_wide_ring_proximal_link, child left_hand_v1_wide_ring_middle_virtual_link, origin xyz=41e-3 0 0 rpy=0 0 0, axis 0 0 1, limit lower=0 upper=0.785398 effort=30 velocity=0.0
- added joint left_hand_v1_wide_ring_proximal_joint: type fixed, parent left_hand_v1_wide_ring_proximal_virtual_link, child left_hand_v1_wide_ring_proximal_link, origin xyz=9e-3 0 0 rpy=0 0 0, axis 0 0 1, limit lower=0 upper=0.785398 effort=30 velocity=0.0
- added joint left_hand_v1_wide_ring_proximal_virtual_joint: type fixed, parent left_hand_v1_wide_ring_knuckle_link, child left_hand_v1_wide_ring_proximal_virtual_link, origin xyz= -6.5e-3 0 24e-3 rpy=-1.5707963 -1.5707963 0, axis 0 0 1, limit lower=0 upper=0.785398 effort=30 velocity=0.0
- added joint left_hand_v1_wide_thumb_distal_joint: type fixed, parent left_hand_v1_wide_thumb_distal_virtual_link, child left_hand_v1_wide_thumb_distal_link, origin xyz=8.99947e-3 0 -0.0973875e-3 rpy=0 0.0101229 0, axis 0 0 1, limit lower=0 upper=0.785398 effort=30 velocity=0.0
- added joint left_hand_v1_wide_thumb_distal_virtual_joint: type fixed, parent left_hand_v1_wide_thumb_proximal_link, child left_hand_v1_wide_thumb_distal_virtual_link, origin xyz=41e-3 0 0 rpy=0 0 0, axis 0 0 1, limit lower=0 upper=0.785398 effort=30 velocity=0.0
- added joint left_hand_v1_wide_thumb_knuckle_joint: type fixed, parent left_hand_v1_wide_palm_thumb_support_link, child left_hand_v1_wide_thumb_knuckle_link, origin xyz=0 21.9577e-3 2.8e-3 rpy=1.5707963 0 1.5707963, axis 0 0 1, limit lower=0 upper=1.57 effort=30 velocity=0.0
- added joint left_hand_v1_wide_thumb_proximal_joint: type fixed, parent left_hand_v1_wide_thumb_knuckle_link, child left_hand_v1_wide_thumb_proximal_virtual_link, origin xyz=38.5e-3 4.82952e-3 0.000167417 rpy=1.3962638 0 0, axis 0 0 1, limit lower=0 upper=0.785398 effort=30 velocity=0.0
- added joint left_hand_v1_wide_thumb_proximal_virtual_joint: type fixed, parent left_hand_v1_wide_thumb_proximal_virtual_link, child left_hand_v1_wide_thumb_proximal_link, origin xyz=9e-3 0 0  rpy=0 0 0, axis 0 0 1, limit lower=0 upper=0.785398 effort=30 velocity=0.0
- joint leg1_joint: origin xyz=0.5 1.25 1.0 rpy=0 0 0 -> xyz=0.5 1.25 0.978 rpy=0 0 0
- joint leg2_joint: origin xyz=-0.5 1.25 1.0 rpy=0 0 0 -> xyz=-0.5 1.25 0.978 rpy=0 0 0
- joint leg3_joint: origin xyz=0.5 -1.25 1.0 rpy=0 0 0 -> xyz=0.5 -1.25 0.978 rpy=0 0 0
- joint leg4_joint: origin xyz=-0.5 -1.25 1.0 rpy=0 0 0 -> xyz=-0.5 -1.25 0.978 rpy=0 0 0
- joint right_hand_v1_2_research_iso_joint: origin xyz=0 0.0 0.00 rpy=0 0 1.570796326795 -> xyz=0.005 0 0 rpy=0 0 1.570796326795; parent arm_2_7 -> arm_2_angle_flange
