Commit message: sliding guide working on arm_1 group

File: repair_moveit_config_v2/config/repair_full.srdf.xacro (robot description, xacro)
@@ -6,5 +6,6 @@
 <robot  xmlns:xacro="http://ros.org/wiki/xacro" name="repair_full">
   <!-- QUIRINO: replaced default with arg value for xacro:if-->
-  <xacro:property name="sh_version" value="$(arg sh_version)"/>
+  <!-- <xacro:property name="sh_version" value="$(arg sh_version)"/> -->
+  <xacro:property name="sh_version" value="v1_2_research"/>
     <!--GROUPS: Representation of a set of joints and links. This can be useful for specifying DOF to plan for, defining arms, end effectors, etc-->
     <!--LINKS: When a link is specified, the parent joint of that link (if it exists) is automatically included-->
@@ -13,8 +14,8 @@
     <!--SUBGROUPS: Groups can also be formed by referencing to already defined group names-->
     <group name="arm_1">
-        <chain base_link="torso_1" tip_link="arm_1_tcp"/>
+        <chain base_link="sliding_guide_link" tip_link="arm_1_tcp"/>
     </group>
     <group name="arm_2">
-        <chain base_link="torso_1" tip_link="arm_2_tcp"/>
+        <chain base_link="sliding_guide_link" tip_link="arm_2_tcp"/>
     </group>
     <group name="both_arms">
@@ -35,6 +36,10 @@
         <joint name="j_sliding_guide" value="1"/>
     </group_state>
+    <group_state name="sliding_guide_center" group="sliding_guide">
+        <joint name="j_sliding_guide" value="0"/>
+    </group_state>
     <!--GROUP STATES: Purpose: Define a named state for a particular group, in terms of joint values. This is useful to define states like 'folded arms'-->
     <group_state name="home" group="arm_1">
+        <joint name="j_sliding_guide" value="0"/>
         <joint name="j_arm_1_1" value="0"/>
         <joint name="j_arm_1_2" value="-0.8812"/>
@@ -46,4 +51,5 @@
     </group_state>
     <group_state name="home" group="arm_2">
+        <joint name="j_sliding_guide" value="0"/>
         <joint name="j_arm_2_1" value="0"/>
         <joint name="j_arm_2_2" value="0.6156"/>
@@ -55,4 +61,5 @@
     </group_state>
     <group_state name="home" group="both_arms">
+        <joint name="j_sliding_guide" value="0"/>
         <joint name="j_arm_1_1" value="0"/>
         <joint name="j_arm_1_2" value="-0.8812"/>
@@ -69,4 +76,7 @@
         <joint name="j_arm_2_6" value="-0.3323"/>
         <joint name="j_arm_2_7" value="0"/>
+    </group_state>
+    <group_state name="home" group="sliding_guide">
+        <joint name="j_sliding_guide" value="0"/>
     </group_state>
     <!-- <group_state name="home" group="torso">
@@ -2381,4 +2391,11 @@
     <!-- IF sh_version= v1_2_research  -->
     <xacro:if value="${sh_version == 'v1_2_research'}">
+        <disable_collisions link1="arm_2_angle_flange" link2="arm_2_7" reason="Adjacent"/>
+        <disable_collisions link1="arm_2_angle_flange" link2="right_hand_v1_2_research_iso_link" reason="Adjacent"/>
+        <disable_collisions link1="right_hand_v1_2_research_palm_link" link2="arm_2_camera_mount" reason="Never"/>
+        <disable_collisions link1="arm_1_angle_flange" link2="left_hand_v1_2_research_iso_link" reason="Adjacent"/>
+        <disable_collisions link1="arm_1_angle_flange" link2="arm_1_7" reason="Adjacent"/>
+        <disable_collisions link1="left_hand_v1_2_research_palm_link" link2="arm_1_camera_mount" reason="Never"/>
+        <disable_collisions link1="sliding_guide_link" link2="left_hand_v1_2_research_thumb_knuckle_link" reason="Never"/>
         <disable_collisions link1="arm_1_1" link2="arm_1_2" reason="Adjacent"/>
         <disable_collisions link1="arm_1_1" link2="arm_1_3" reason="Never"/>

File: repair_srdf/srdf/repair.srdf.xacro (robot description, xacro)
@@ -17,4 +17,5 @@
     <!--GROUP STATES: Purpose: Define a named state for a particular group, in terms of joint values. This is useful to define states like 'folded arms'-->
     <group_state name="home" group="chains">
+        <joint name="j_sliding_guide" value="0.0"/>
         <joint name="j_arm_1_1" value="0.5"/>
         <joint name="j_arm_1_2" value="0.5"/>

File: repair_srdf/srdf/repair_full.srdf.xacro (robot description, xacro)
@@ -32,4 +32,5 @@
     <!--GROUP STATES: Purpose: Define a named state for a particular group, in terms of joint values. This is useful to define states like 'folded arms'-->
     <group_state name="home" group="chains">
+        <joint name="j_sliding_guide" value="0.0"/>
         <joint name="j_arm_1_1" value="-0.5"/>
         <joint name="j_arm_1_2" value="-0.7"/>

File: repair_urdf/urdf/repair_full.urdf (robot description, URDF)
Before this commit: robot repair_full, 128 links, 127 joints
Joints:
- joint j_sliding_guide: axis (none) -> 0 0 -1; limit (none) -> lower=-1.0 upper=1.0 effort=147 velocity=5; type fixed -> prismatic
