Commit message: [gripper] modified the version to v2s and added transmission for synergy joint

File: repair_srdf/srdf/repair_full.srdf.xacro (robot description, xacro)
@@ -13,6 +13,6 @@
         <chain base_link="base_link" tip_link="arm_2_link_7"/>
     </group>
-    <xacro:softhand side="right" type="v1s" base_link="arm_1_link_7"/>
-    <xacro:softhand side="left" type="v1s" base_link="arm_2_link_7"/>
+    <xacro:softhand side="right" type="v2s" base_link="arm_1_link_7"/>
+    <xacro:softhand side="left" type="v2s" base_link="arm_2_link_7"/>
     <group name="chains">
         <group name="sliding_guide"/>
@@ -48,6 +48,6 @@
         <joint name="arm_2_joint_7" value="-1.0"/>
         <joint name="x_joint" value="-0.05"/>
-        <xacro:softhand_homing side="right" type="v1s"/>
-        <xacro:softhand_homing side="left" type="v1s"/>
+        <xacro:softhand_homing side="right" type="v2s"/>
+        <xacro:softhand_homing side="left" type="v2s"/>
     </group_state>
 </robot>

File: repair_urdf/urdf/repair_arm.urdf.xacro (robot description, xacro)
@@ -353,5 +353,5 @@
         version="v2.0_simple"
         parent="arm_${id}_link_7"
-        useMimicTag="false"
+        useMimicTag="true"
         position="0 0 -0.015"
         orientation="0 0.0 ${PI}"

File: repair_urdf/urdf/repair_hand_transmission.xacro (robot description, xacro)
@@ -2,190 +2,201 @@
 <robot xmlns:xacro="http://www.ros.org/wiki/xacro">
   <xacro:macro name="repair_hand_transmission" params="id">
-    <transmission name="trans_${id}_hand_v1s_index_knuckle_joint">
-        <type>transmission_interface/SimpleTransmission</type>
-        <joint name="${id}_hand_v1s_index_knuckle_joint">
-            <hardwareInterface>hardware_interface/EffortJointInterface</hardwareInterface>
-        </joint>
-        <actuator name="${id}_hand_v1s_index_knuckle_joint_motor">
-            <hardwareInterface>hardware_interface/EffortJointInterface</hardwareInterface>
-            <mechanicalReduction>1</mechanicalReduction>
-        </actuator>
-    </transmission>
-    <transmission name="trans_${id}_hand_v1s_index_proximal_joint">
-        <type>transmission_interface/SimpleTransmission</type>
-        <joint name="${id}_hand_v1s_index_proximal_joint">
-            <hardwareInterface>hardware_interface/EffortJointInterface</hardwareInterface>
-        </joint>
-        <actuator name="${id}_hand_v1s_index_proximal_joint_motor">
-            <hardwareInterface>hardware_interface/EffortJointInterface</hardwareInterface>
-            <mechanicalReduction>1</mechanicalReduction>
-        </actuator>
-    </transmission>
-    <transmission name="trans_${id}_hand_v1s_index_middle_joint">
-        <type>transmission_interface/SimpleTransmission</type>
-        <joint name="${id}_hand_v1s_index_middle_joint">
-            <hardwareInterface>hardware_interface/EffortJointInterface</hardwareInterface>
-        </joint>
-        <actuator name="${id}_hand_v1s_index_middle_joint_motor">
-            <hardwareInterface>hardware_interface/EffortJointInterface</hardwareInterface>
-            <mechanicalReduction>1</mechanicalReduction>
-        </actuator>
-    </transmission>
-    <transmission name="trans_${id}_hand_v1s_index_distal_joint">
-        <type>transmission_interface/SimpleTransmission</type>
-        <joint name="${id}_hand_v1s_index_distal_joint">
-            <hardwareInterface>hardware_interface/EffortJointInterface</hardwareInterface>
-        </joint>
-        <actuator name="${id}_hand_v1s_index_distal_joint_motor">
-            <hardwareInterface>hardware_interface/EffortJointInterface</hardwareInterface>
-            <mechanicalReduction>1</mechanicalReduction>
-        </actuator>
-    </transmission>
-    <transmission name="trans_${id}_hand_v1s_middle_knuckle_joint">
-        <type>transmission_interface/SimpleTransmission</type>
-        <joint name="${id}_hand_v1s_middle_knuckle_joint">
-            <hardwareInterface>hardware_interface/EffortJointInterface</hardwareInterface>
-        </joint>
-        <actuator name="${id}_hand_v1s_middle_knuckle_joint_motor">
-            <hardwareInterface>hardware_interface/EffortJointInterface</hardwareInterface>
-            <mechanicalReduction>1</mechanicalReduction>
-        </actuator>
-    </transmission>
-    <transmission name="trans_${id}_hand_v1s_middle_proximal_joint">
-        <type>transmission_interface/SimpleTransmission</type>
-        <joint name="${id}_hand_v1s_middle_proximal_joint">
-            <hardwareInterface>hardware_interface/EffortJointInterface</hardwareInterface>
-        </joint>
-        <actuator name="${id}_hand_v1s_middle_proximal_joint_motor">
-            <hardwareInterface>hardware_interface/EffortJointInterface</hardwareInterface>
-            <mechanicalReduction>1</mechanicalReduction>
-        </actuator>
-    </transmission>
-    <transmission name="trans_${id}_hand_v1s_middle_middle_joint">
-        <type>transmission_interface/SimpleTransmission</type>
-        <joint name="${id}_hand_v1s_middle_middle_joint">
-            <hardwareInterface>hardware_interface/EffortJointInterface</hardwareInterface>
-        </joint>
-        <actuator name="${id}_hand_v1s_middle_middle_joint_motor">
-            <hardwareInterface>hardware_interface/EffortJointInterface</hardwareInterface>
-            <mechanicalReduction>1</mechanicalReduction>
-        </actuator>
-    </transmission>
-    <transmission name="trans_${id}_hand_v1s_middle_distal_joint">
-        <type>transmission_interface/SimpleTransmission</type>
-        <joint name="${id}_hand_v1s_middle_distal_joint">
-            <hardwareInterface>hardware_interface/EffortJointInterface</hardwareInterface>
-        </joint>
-        <actuator name="${id}_hand_v1s_middle_distal_joint_motor">
-            <hardwareInterface>hardware_interface/EffortJointInterface</hardwareInterface>
-            <mechanicalReduction>1</mechanicalReduction>
-        </actuator>
-    </transmission>
-    <transmission name="trans_${id}_hand_v1s_ring_knuckle_joint">
-        <type>transmission_interface/SimpleTransmission</type>
-        <joint name="${id}_hand_v1s_ring_knuckle_joint">
-            <hardwareInterface>hardware_interface/EffortJointInterface</hardwareInterface>
-        </joint>
-        <actuator name="${id}_hand_v1s_ring_knuckle_joint_motor">
-            <hardwareInterface>hardware_interface/EffortJointInterface</hardwareInterface>
-            <mechanicalReduction>1</mechanicalReduction>
-        </actuator>
-    </transmission>
-    <transmission name="trans_${id}_hand_v1s_ring_proximal_joint">
-        <type>transmission_interface/SimpleTransmission</type>
-        <joint name="${id}_hand_v1s_ring_proximal_joint">
-            <hardwareInterface>hardware_interface/EffortJointInterface</hardwareInterface>
-        </joint>
-        <actuator name="${id}_hand_v1s_ring_proximal_joint_motor">
-            <hardwareInterface>hardware_interface/EffortJointInterface</hardwareInterface>
-            <mechanicalReduction>1</mechanicalReduction>
-        </actuator>
-    </transmission>
-    <transmission name="trans_${id}_hand_v1s_ring_middle_joint">
-        <type>transmission_interface/SimpleTransmission</type>
-        <joint name="${id}_hand_v1s_ring_middle_joint">
-            <hardwareInterface>hardware_interface/EffortJointInterface</hardwareInterface>
-        </joint>
-        <actuator name="${id}_hand_v1s_ring_middle_joint_motor">
-            <hardwareInterface>hardware_interface/EffortJointInterface</hardwareInterface>
-            <mechanicalReduction>1</mechanicalReduction>
-        </actuator>
-    </transmission>
-    <transmission name="trans_${id}_hand_v1s_ring_distal_joint">
-        <type>transmission_interface/SimpleTransmission</type>
-        <joint name="${id}_hand_v1s_ring_distal_joint">
-            <hardwareInterface>hardware_interface/EffortJointInterface</hardwareInterface>
-        </joint>
-        <actuator name="${id}_hand_v1s_ring_distal_joint_motor">
-            <hardwareInterface>hardware_interface/EffortJointInterface</hardwareInterface>
-            <mechanicalReduction>1</mechanicalReduction>
-        </actuator>
-    </transmission>
-    <transmission name="trans_${id}_hand_v1s_little_knuckle_joint">
-        <type>transmission_interface/SimpleTransmission</type>
-        <joint name="${id}_hand_v1s_little_knuckle_joint">
-            <hardwareInterface>hardware_interface/EffortJointInterface</hardwareInterface>
-        </joint>
-        <actuator name="${id}_hand_v1s_little_knuckle_joint_motor">
-            <hardwareInterface>hardware_interface/EffortJointInterface</hardwareInterface>
-            <mechanicalReduction>1</mechanicalReduction>
-        </actuator>
-    </transmission>
-    <transmission name="trans_${id}_hand_v1s_little_proximal_joint">
-        <type>transmission_interface/SimpleTransmission</type>
-        <joint name="${id}_hand_v1s_little_proximal_joint">
-            <hardwareInterface>hardware_interface/EffortJointInterface</hardwareInterface>
-        </joint>
-        <actuator name="${id}_hand_v1s_little_proximal_joint_motor">
-            <hardwareInterface>hardware_interface/EffortJointInterface</hardwareInterface>
-            <mechanicalReduction>1</mechanicalReduction>
-        </actuator>
-    </transmission>
-    <transmission name="trans_${id}_hand_v1s_little_middle_joint">
-        <type>transmission_interface/SimpleTransmission</type>
-        <joint name="${id}_hand_v1s_little_middle_joint">
-            <hardwareInterface>hardware_interface/EffortJointInterface</hardwareInterface>
-        </joint>
-        <actuator name="${id}_hand_v1s_little_middle_joint_motor">
-            <hardwareInterface>hardware_interface/EffortJointInterface</hardwareInterface>
-            <mechanicalReduction>1</mechanicalReduction>
-        </actuator>
-    </transmission>
-    <transmission name="trans_${id}_hand_v1s_little_distal_joint">
-        <type>transmission_interface/SimpleTransmission</type>
-        <joint name="${id}_hand_v1s_little_distal_joint">
-            <hardwareInterface>hardware_interface/EffortJointInterface</hardwareInterface>
-        </joint>
-        <actuator name="${id}_hand_v1s_little_distal_joint_motor">
-            <hardwareInterface>hardware_interface/EffortJointInterface</hardwareInterface>
-            <mechanicalReduction>1</mechanicalReduction>
-        </actuator>
-    </transmission>
-    <transmission name="trans_${id}_hand_v1s_thumb_knuckle_joint">
-        <type>transmission_interface/SimpleTransmission</type>
-        <joint name="${id}_hand_v1s_thumb_knuckle_joint">
-            <hardwareInterface>hardware_interface/EffortJointInterface</hardwareInterface>
-        </joint>
-        <actuator name="${id}_hand_v1s_thumb_knuckle_joint_motor">
-            <hardwareInterface>hardware_interface/EffortJointInterface</hardwareInterface>
-            <mechanicalReduction>1</mechanicalReduction>
-        </actuator>
-    </transmission>
-    <transmission name="trans_${id}_hand_v1s_thumb_proximal_joint">
-        <type>transmission_interface/SimpleTransmission</type>
-        <joint name="${id}_hand_v1s_thumb_proximal_joint">
-            <hardwareInterface>hardware_interface/EffortJointInterface</hardwareInterface>
-        </joint>
-        <actuator name="${id}_hand_v1s_thumb_proximal_joint_motor">
-            <hardwareInterface>hardware_interface/EffortJointInterface</hardwareInterface>
-            <mechanicalReduction>1</mechanicalReduction>
-        </actuator>
-    </transmission>
-    <transmission name="trans_${id}_hand_v1s_thumb_distal_joint">
-        <type>transmission_interface/SimpleTransmission</type>
-        <joint name="${id}_hand_v1s_thumb_distal_joint">
-            <hardwareInterface>hardware_interface/EffortJointInterface</hardwareInterface>
-        </joint>
-        <actuator name="${id}_hand_v1s_thumb_distal_joint_motor">
+    <!-- synergy joint -->
+    <transmission name="trans_${id}_hand_v2s_synergy_joint">
+        <type>transmission_interface/SimpleTransmission</type>
+        <joint name="${id}_hand_v2s_synergy_joint">
+            <hardwareInterface>hardware_interface/PositionJointInterface</hardwareInterface>
+        </joint>
+        <actuator name="${id}_hand_v2s_synergy_joint_motor">
+            <hardwareInterface>hardware_interface/PositionJointInterface</hardwareInterface>
+            <mechanicalReduction>1</mechanicalReduction>
+        </actuator>
+    </transmission>
+    <transmission name="trans_${id}_hand_v2s_index_knuckle_joint">
+        <type>transmission_interface/SimpleTransmission</type>
+        <joint name="${id}_hand_v2s_index_knuckle_joint">
+            <hardwareInterface>hardware_interface/EffortJointInterface</hardwareInterface>
+        </joint>
+        <actuator name="${id}_hand_v2s_index_knuckle_joint_motor">
+            <hardwareInterface>hardware_interface/EffortJointInterface</hardwareInterface>
+            <mechanicalReduction>1</mechanicalReduction>
+        </actuator>
+    </transmission>
+    <transmission name="trans_${id}_hand_v2s_index_proximal_joint">
+        <type>transmission_interface/SimpleTransmission</type>
+        <joint name="${id}_hand_v2s_index_proximal_joint">
+            <hardwareInterface>hardware_interface/EffortJointInterface</hardwareInterface>
+        </joint>
+        <actuator name="${id}_hand_v2s_index_proximal_joint_motor">
+            <hardwareInterface>hardware_interface/EffortJointInterface</hardwareInterface>
+            <mechanicalReduction>1</mechanicalReduction>
+        </actuator>
+    </transmission>
+    <transmission name="trans_${id}_hand_v2s_index_middle_joint">
+        <type>transmission_interface/SimpleTransmission</type>
+        <joint name="${id}_hand_v2s_index_middle_joint">
+            <hardwareInterface>hardware_interface/EffortJointInterface</hardwareInterface>
+        </joint>
+        <actuator name="${id}_hand_v2s_index_middle_joint_motor">
+            <hardwareInterface>hardware_interface/EffortJointInterface</hardwareInterface>
+            <mechanicalReduction>1</mechanicalReduction>
+        </actuator>
+    </transmission>
+    <transmission name="trans_${id}_hand_v2s_index_distal_joint">
+        <type>transmission_interface/SimpleTransmission</type>
+        <joint name="${id}_hand_v2s_index_distal_joint">
+            <hardwareInterface>hardware_interface/EffortJointInterface</hardwareInterface>
+        </joint>
+        <actuator name="${id}_hand_v2s_index_distal_joint_motor">
+            <hardwareInterface>hardware_interface/EffortJointInterface</hardwareInterface>
+            <mechanicalReduction>1</mechanicalReduction>
+        </actuator>
+    </transmission>
+    <transmission name="trans_${id}_hand_v2s_middle_knuckle_joint">
+        <type>transmission_interface/SimpleTransmission</type>
+        <joint name="${id}_hand_v2s_middle_knuckle_joint">
+            <hardwareInterface>hardware_interface/EffortJointInterface</hardwareInterface>
+        </joint>
+        <actuator name="${id}_hand_v2s_middle_knuckle_joint_motor">
+            <hardwareInterface>hardware_interface/EffortJointInterface</hardwareInterface>
+            <mechanicalReduction>1</mechanicalReduction>
+        </actuator>
+    </transmission>
+    <transmission name="trans_${id}_hand_v2s_middle_proximal_joint">
+        <type>transmission_interface/SimpleTransmission</type>
+        <joint name="${id}_hand_v2s_middle_proximal_joint">
+            <hardwareInterface>hardware_interface/EffortJointInterface</hardwareInterface>
+        </joint>
+        <actuator name="${id}_hand_v2s_middle_proximal_joint_motor">
+            <hardwareInterface>hardware_interface/EffortJointInterface</hardwareInterface>
+            <mechanicalReduction>1</mechanicalReduction>
+        </actuator>
+    </transmission>
+    <transmission name="trans_${id}_hand_v2s_middle_middle_joint">
+        <type>transmission_interface/SimpleTransmission</type>
+        <joint name="${id}_hand_v2s_middle_middle_joint">
+            <hardwareInterface>hardware_interface/EffortJointInterface</hardwareInterface>
+        </joint>
+        <actuator name="${id}_hand_v2s_middle_middle_joint_motor">
+            <hardwareInterface>hardware_interface/EffortJointInterface</hardwareInterface>
+            <mechanicalReduction>1</mechanicalReduction>
+        </actuator>
+    </transmission>
+    <transmission name="trans_${id}_hand_v2s_middle_distal_joint">
+        <type>transmission_interface/SimpleTransmission</type>
+        <joint name="${id}_hand_v2s_middle_distal_joint">
+            <hardwareInterface>hardware_interface/EffortJointInterface</hardwareInterface>
+        </joint>
+        <actuator name="${id}_hand_v2s_middle_distal_joint_motor">
+            <hardwareInterface>hardware_interface/EffortJointInterface</hardwareInterface>
+            <mechanicalReduction>1</mechanicalReduction>
+        </actuator>
+    </transmission>
+    <transmission name="trans_${id}_hand_v2s_ring_knuckle_joint">
+        <type>transmission_interface/SimpleTransmission</type>
+        <joint name="${id}_hand_v2s_ring_knuckle_joint">
+            <hardwareInterface>hardware_interface/EffortJointInterface</hardwareInterface>
+        </joint>
+        <actuator name="${id}_hand_v2s_ring_knuckle_joint_motor">
+            <hardwareInterface>hardware_interface/EffortJointInterface</hardwareInterface>
+            <mechanicalReduction>1</mechanicalReduction>
+        </actuator>
+    </transmission>
+    <transmission name="trans_${id}_hand_v2s_ring_proximal_joint">
+        <type>transmission_interface/SimpleTransmission</type>
+        <joint name="${id}_hand_v2s_ring_proximal_joint">
+            <hardwareInterface>hardware_interface/EffortJointInterface</hardwareInterface>
+        </joint>
+        <actuator name="${id}_hand_v2s_ring_proximal_joint_motor">
+            <hardwareInterface>hardware_interface/EffortJointInterface</hardwareInterface>
+            <mechanicalReduction>1</mechanicalReduction>
+        </actuator>
+    </transmission>
+    <transmission name="trans_${id}_hand_v2s_ring_middle_joint">
+        <type>transmission_interface/SimpleTransmission</type>
+        <joint name="${id}_hand_v2s_ring_middle_joint">
+            <hardwareInterface>hardware_interface/EffortJointInterface</hardwareInterface>
+        </joint>
+        <actuator name="${id}_hand_v2s_ring_middle_joint_motor">
+            <hardwareInterface>hardware_interface/EffortJointInterface</hardwareInterface>
+            <mechanicalReduction>1</mechanicalReduction>
+        </actuator>
+    </transmission>
+    <transmission name="trans_${id}_hand_v2s_ring_distal_joint">
+        <type>transmission_interface/SimpleTransmission</type>
+        <joint name="${id}_hand_v2s_ring_distal_joint">
+            <hardwareInterface>hardware_interface/EffortJointInterface</hardwareInterface>
+        </joint>
+        <actuator name="${id}_hand_v2s_ring_distal_joint_motor">
+            <hardwareInterface>hardware_interface/EffortJointInterface</hardwareInterface>
+            <mechanicalReduction>1</mechanicalReduction>
+        </actuator>
+    </transmission>
+    <transmission name="trans_${id}_hand_v2s_little_knuckle_joint">
+        <type>transmission_interface/SimpleTransmission</type>
+        <joint name="${id}_hand_v2s_little_knuckle_joint">
+            <hardwareInterface>hardware_interface/EffortJointInterface</hardwareInterface>
+        </joint>
+        <actuator name="${id}_hand_v2s_little_knuckle_joint_motor">
+            <hardwareInterface>hardware_interface/EffortJointInterface</hardwareInterface>
+            <mechanicalReduction>1</mechanicalReduction>
+        </actuator>
+    </transmission>
+    <transmission name="trans_${id}_hand_v2s_little_proximal_joint">
+        <type>transmission_interface/SimpleTransmission</type>
+        <joint name="${id}_hand_v2s_little_proximal_joint">
+            <hardwareInterface>hardware_interface/EffortJointInterface</hardwareInterface>
+        </joint>
+        <actuator name="${id}_hand_v2s_little_proximal_joint_motor">
+            <hardwareInterface>hardware_interface/EffortJointInterface</hardwareInterface>
+            <mechanicalReduction>1</mechanicalReduction>
+        </actuator>
+    </transmission>
+    <transmission name="trans_${id}_hand_v2s_little_middle_joint">
+        <type>transmission_interface/SimpleTransmission</type>
+        <joint name="${id}_hand_v2s_little_middle_joint">
+            <hardwareInterface>hardware_interface/EffortJointInterface</hardwareInterface>
+        </joint>
+        <actuator name="${id}_hand_v2s_little_middle_joint_motor">
+            <hardwareInterface>hardware_interface/EffortJointInterface</hardwareInterface>
+            <mechanicalReduction>1</mechanicalReduction>
+        </actuator>
+    </transmission>
+    <transmission name="trans_${id}_hand_v2s_little_distal_joint">
+        <type>transmission_interface/SimpleTransmission</type>
+        <joint name="${id}_hand_v2s_little_distal_joint">
+            <hardwareInterface>hardware_interface/EffortJointInterface</hardwareInterface>
+        </joint>
+        <actuator name="${id}_hand_v2s_little_distal_joint_motor">
+            <hardwareInterface>hardware_interface/EffortJointInterface</hardwareInterface>
+            <mechanicalReduction>1</mechanicalReduction>
+        </actuator>
+    </transmission>
+    <transmission name="trans_${id}_hand_v2s_thumb_knuckle_joint">
+        <type>transmission_interface/SimpleTransmission</type>
+        <joint name="${id}_hand_v2s_thumb_knuckle_joint">
+            <hardwareInterface>hardware_interface/EffortJointInterface</hardwareInterface>
+        </joint>
+        <actuator name="${id}_hand_v2s_thumb_knuckle_joint_motor">
+            <hardwareInterface>hardware_interface/EffortJointInterface</hardwareInterface>
+            <mechanicalReduction>1</mechanicalReduction>
+        </actuator>
+    </transmission>
+    <transmission name="trans_${id}_hand_v2s_thumb_proximal_joint">
+        <type>transmission_interface/SimpleTransmission</type>
+        <joint name="${id}_hand_v2s_thumb_proximal_joint">
+            <hardwareInterface>hardware_interface/EffortJointInterface</hardwareInterface>
+        </joint>
+        <actuator name="${id}_hand_v2s_thumb_proximal_joint_motor">
+            <hardwareInterface>hardware_interface/EffortJointInterface</hardwareInterface>
+            <mechanicalReduction>1</mechanicalReduction>
+        </actuator>
+    </transmission>
+    <transmission name="trans_${id}_hand_v2s_thumb_distal_joint">
+        <type>transmission_interface/SimpleTransmission</type>
+        <joint name="${id}_hand_v2s_thumb_distal_joint">
+            <hardwareInterface>hardware_interface/EffortJointInterface</hardwareInterface>
+        </joint>
+        <actuator name="${id}_hand_v2s_thumb_distal_joint_motor">
             <hardwareInterface>hardware_interface/EffortJointInterface</hardwareInterface>
             <mechanicalReduction>1</mechanicalReduction>
