Commit message: [gripper] modified the version to v2s and added transmission for synergy joint

File: repair_urdf/urdf/xbot2.gazebo.xacro (robot description, xacro)
@@ -30,6 +30,6 @@
         </pid>
         <ignore_joints>
-            <xacro:ignore_softhand_jnts side="right" type="v1s"/>
-            <xacro:ignore_softhand_jnts side="left" type="v1s"/>
+            <xacro:ignore_softhand_jnts side="right" type="v2s"/>
+            <xacro:ignore_softhand_jnts side="left" type="v2s"/>
         </ignore_joints>
     </plugin>
