Commit message: cleaned version with softhands

File: repair_srdf/srdf/repair_full.srdf.xacro (robot description, xacro)
@@ -1,53 +1,207 @@
-<?xml version="1.0"?>
+<?xml version="1.0" encoding="UTF-8"?>
 <robot name="repair_full" xmlns:xacro="http://ros.org/wiki/xacro">
+    <!-- <xacro:include filename="$(find softhands_description)/srdf/softhands.srdf.xacro"/>
     <xacro:include filename="$(find softhands_description)/srdf/softhands.srdf.xacro"/>
-    <xacro:include filename="$(find softhands_description)/srdf/softhands.srdf.xacro"/>
-    <xacro:include filename="$(find softhands_description)/srdf/softhands_homing.srdf.xacro"/>
+    <xacro:include filename="$(find softhands_description)/srdf/softhands_homing.srdf.xacro"/> -->
     <group name="sliding_guide">
-        <chain base_link="working_surface_link" tip_link="base_link"/>
+        <chain base_link="sliding_guide_link" tip_link="torso_1"/>
     </group>
     <group name="arm1">
-        <chain base_link="base_link" tip_link="arm_1_link_7"/>
+        <chain base_link="torso_1" tip_link="arm_1_tcp"/>
     </group>
     <group name="arm2">
-        <chain base_link="base_link" tip_link="arm_2_link_7"/>
-    </group>
-    <xacro:softhand side="right" type="v2s" base_link="arm_1_link_7"/>
-    <xacro:softhand side="left" type="v2s" base_link="arm_2_link_7"/>
+        <chain base_link="torso_1" tip_link="arm_2_tcp"/>
+    </group>
     <group name="chains">
-        <group name="sliding_guide"/>
+        <group name="sliding_guide" />
         <group name="arm1"/>
         <group name="arm2"/>
-        <!-- <group name="palm_right"/> -->
-        <!-- <group name="thumb_right"/> -->
-        <!-- <group name="index_right"/> -->
-        <!-- <group name="middle_right"/> -->
-        <!-- <group name="ring_right"/> -->
-        <!-- <group name="little_right"/> -->
-        <!-- <group name="palm_left"/> -->
-        <!-- <group name="thumb_left"/> -->
-        <!-- <group name="index_left"/>
+        <!-- <group name="palm_right"/>
+        <group name="thumb_right"/>
+        <group name="index_right"/>
+        <group name="middle_right"/>
+        <group name="ring_right"/>
+        <group name="little_right"/>
+        <group name="palm_left"/>
+        <group name="thumb_left"/>
+        <group name="index_left"/>
         <group name="middle_left"/>
         <group name="ring_left"/>
         <group name="little_left"/> -->
     </group>
+    <!--GROUP STATES: Purpose: Define a named state for a particular group, in terms of joint values. This is useful to define states like 'folded arms'-->
     <group_state name="home" group="chains">
-        <joint name="arm_1_joint_1" value="0.85"/>
-        <joint name="arm_1_joint_2" value="0.72"/>
-        <joint name="arm_1_joint_3" value="0.6"/>
-        <joint name="arm_1_joint_4" value="-0.9"/>
-        <joint name="arm_1_joint_5" value="-0.5"/>
-        <joint name="arm_1_joint_6" value="0"/>
-        <joint name="arm_1_joint_7" value="1.0"/>
-        <joint name="arm_2_joint_1" value="-0.85"/>
-        <joint name="arm_2_joint_2" value="-0.72"/>
-        <joint name="arm_2_joint_3" value="-0.6"/>
-        <joint name="arm_2_joint_4" value="-0.9"/>
-        <joint name="arm_2_joint_5" value="0.5"/>
-        <joint name="arm_2_joint_6" value="0"/>
-        <joint name="arm_2_joint_7" value="-1.0"/>
-        <joint name="x_joint" value="-0.05"/>
-        <xacro:softhand_homing side="right" type="v2s"/>
-        <xacro:softhand_homing side="left" type="v2s"/>
+        <joint name="j_arm_1_1" value="-0.5"/>
+        <joint name="j_arm_1_2" value="-0.5"/>
+        <joint name="j_arm_1_3" value="0.5"/>
+        <joint name="j_arm_1_4" value="-1.0"/>
+        <joint name="j_arm_1_5" value="-0.5"/>
+        <joint name="j_arm_1_6" value="-0.5"/>
+        <joint name="j_arm_1_7" value="-1.0"/>
+        <joint name="j_arm_2_1" value="0.5"/>
+        <joint name="j_arm_2_2" value="0.5"/>
+        <joint name="j_arm_2_3" value="-0.5"/>
+        <joint name="j_arm_2_4" value="1.0"/>
+        <joint name="j_arm_2_5" value="0.5"/>
+        <joint name="j_arm_2_6" value="0.5"/>
+        <joint name="j_arm_2_7" value="1.0"/>
+        <!-- <xacro:softhand_homing side="right" type="v1s"/>
+        <xacro:softhand_homing side="left" type="v1s"/> -->
     </group_state>
+    <!-- DISABLE COLLISIONS: By default it is assumed that any link of the robot could potentially come into collision with any other link in the robot. This tag disables collision checking between a specified pair of links. -->
+    <!-- <disable_collisions link1="arm_1_link_1" link2="arm_1_link_2" reason="Adjacent"/>
+    <disable_collisions link1="arm_1_link_1" link2="arm_1_link_3" reason="Never"/>
+    <disable_collisions link1="arm_1_link_1" link2="arm_1_link_4" reason="Never"/>
+    <disable_collisions link1="arm_1_link_1" link2="arm_2_link_1" reason="Adjacent"/>
+    <disable_collisions link1="arm_1_link_1" link2="arm_2_link_2" reason="Never"/>
+    <disable_collisions link1="arm_1_link_1" link2="arm_2_link_3" reason="Never"/>
+    <disable_collisions link1="arm_1_link_1" link2="arm_2_link_4" reason="Never"/>
+    <disable_collisions link1="arm_1_link_1" link2="arm_2_link_5" reason="Never"/>
+    <disable_collisions link1="arm_1_link_1" link2="arm_2_link_7" reason="Never"/>
+    <disable_collisions link1="arm_1_link_2" link2="arm_1_link_3" reason="Adjacent"/>
+    <disable_collisions link1="arm_1_link_2" link2="arm_1_link_4" reason="Never"/>
+    <disable_collisions link1="arm_1_link_2" link2="arm_2_link_1" reason="Never"/>
+    <disable_collisions link1="arm_1_link_2" link2="arm_2_link_2" reason="Never"/>
+    <disable_collisions link1="arm_1_link_2" link2="arm_2_link_3" reason="Never"/>
+    <disable_collisions link1="arm_1_link_2" link2="arm_2_link_4" reason="Never"/>
+    <disable_collisions link1="arm_1_link_2" link2="arm_2_link_5" reason="Never"/>
+    <disable_collisions link1="arm_1_link_2" link2="arm_2_link_6" reason="Never"/>
+    <disable_collisions link1="arm_1_link_2" link2="arm_2_link_7" reason="Never"/>
+    <disable_collisions link1="arm_1_link_3" link2="arm_1_link_4" reason="Adjacent"/>
+    <disable_collisions link1="arm_1_link_3" link2="arm_2_link_1" reason="Never"/>
+    <disable_collisions link1="arm_1_link_3" link2="arm_2_link_2" reason="Never"/>
+    <disable_collisions link1="arm_1_link_3" link2="arm_2_link_3" reason="Never"/>
+    <disable_collisions link1="arm_1_link_3" link2="arm_2_link_4" reason="Never"/>
+    <disable_collisions link1="arm_1_link_4" link2="arm_1_link_5" reason="Adjacent"/>
+    <disable_collisions link1="arm_1_link_4" link2="arm_1_link_6" reason="Never"/>
+    <disable_collisions link1="arm_1_link_4" link2="arm_1_link_7" reason="Never"/>
+    <disable_collisions link1="arm_1_link_4" link2="arm_2_link_1" reason="Never"/>
+    <disable_collisions link1="arm_1_link_4" link2="arm_2_link_2" reason="Never"/>
+    <disable_collisions link1="arm_1_link_4" link2="arm_2_link_3" reason="Never"/>
+    <disable_collisions link1="arm_1_link_4" link2="arm_2_link_4" reason="Never"/>
+    <disable_collisions link1="arm_1_link_5" link2="arm_1_link_6" reason="Adjacent"/>
+    <disable_collisions link1="arm_1_link_5" link2="arm_1_link_7" reason="Never"/>
+    <disable_collisions link1="arm_1_link_5" link2="arm_2_link_1" reason="Never"/>
+    <disable_collisions link1="arm_1_link_5" link2="arm_2_link_2" reason="Never"/>
+    <disable_collisions link1="arm_1_link_6" link2="arm_1_link_7" reason="Adjacent"/>
+    <disable_collisions link1="arm_1_link_6" link2="arm_2_link_2" reason="Never"/>
+    <disable_collisions link1="arm_2_link_1" link2="arm_2_link_2" reason="Adjacent"/>
+    <disable_collisions link1="arm_2_link_1" link2="arm_2_link_4" reason="Never"/>
+    <disable_collisions link1="arm_2_link_4" link2="arm_2_link_5" reason="Adjacent"/>
+    <disable_collisions link1="arm_2_link_4" link2="arm_2_link_6" reason="Never"/>
+    <disable_collisions link1="arm_2_link_4" link2="arm_2_link_7" reason="Never"/>
+    <disable_collisions link1="arm_2_link_5" link2="arm_2_link_6" reason="Adjacent"/>
+    <disable_collisions link1="arm_2_link_5" link2="arm_2_link_7" reason="Never"/>
+    <disable_collisions link1="arm_2_link_5" link2="leg1_link" reason="Never"/>
+    <disable_collisions link1="arm_2_link_5" link2="leg3_link" reason="Never"/>
+    <disable_collisions link1="arm_2_link_5" link2="obar1_link" reason="Never"/>
+    <disable_collisions link1="arm_2_link_5" link2="obar2_link" reason="Never"/>
+    <disable_collisions link1="arm_2_link_5" link2="obar3_link" reason="Never"/>
+    <disable_collisions link1="arm_2_link_5" link2="obar4_link" reason="Never"/>
+    <disable_collisions link1="arm_2_link_5" link2="sliding_guide_link" reason="Never"/>
+    <disable_collisions link1="arm_2_link_5" link2="vbar1_link" reason="Never"/>
+    <disable_collisions link1="arm_2_link_5" link2="vbar3_link" reason="Never"/>
+    <disable_collisions link1="arm_2_link_6" link2="arm_2_link_7" reason="Adjacent"/>
+    <disable_collisions link1="arm_2_link_6" link2="leg1_link" reason="Never"/>
+    <disable_collisions link1="arm_2_link_6" link2="leg3_link" reason="Never"/>
+    <disable_collisions link1="arm_2_link_6" link2="obar3_link" reason="Never"/>
+    <disable_collisions link1="arm_2_link_6" link2="obar4_link" reason="Never"/>
+    <disable_collisions link1="arm_2_link_6" link2="vbar1_link" reason="Never"/>
+    <disable_collisions link1="arm_2_link_6" link2="vbar3_link" reason="Never"/>
+    <disable_collisions link1="arm_2_link_7" link2="leg1_link" reason="Never"/>
+    <disable_collisions link1="arm_2_link_7" link2="leg3_link" reason="Never"/>
+    <disable_collisions link1="arm_2_link_7" link2="obar3_link" reason="Never"/>
+    <disable_collisions link1="arm_2_link_7" link2="vbar1_link" reason="Never"/>
+    <disable_collisions link1="arm_2_link_7" link2="vbar3_link" reason="Never"/>
+    <disable_collisions link1="leg1_link" link2="leg2_link" reason="Never"/>
+    <disable_collisions link1="leg1_link" link2="leg3_link" reason="Never"/>
+    <disable_collisions link1="leg1_link" link2="leg4_link" reason="Never"/>
+    <disable_collisions link1="leg1_link" link2="obar1_link" reason="Never"/>
+    <disable_collisions link1="leg1_link" link2="obar2_link" reason="Never"/>
+    <disable_collisions link1="leg1_link" link2="obar3_link" reason="Never"/>
+    <disable_collisions link1="leg1_link" link2="obar4_link" reason="Never"/>
+    <disable_collisions link1="leg1_link" link2="sliding_guide_link" reason="Never"/>
+    <disable_collisions link1="leg1_link" link2="table_top_link" reason="Adjacent"/>
+    <disable_collisions link1="leg1_link" link2="vbar1_link" reason="Adjacent"/>
+    <disable_collisions link1="leg1_link" link2="vbar2_link" reason="Never"/>
+    <disable_collisions link1="leg1_link" link2="vbar3_link" reason="Never"/>
+    <disable_collisions link1="leg1_link" link2="vbar4_link" reason="Never"/>
+    <disable_collisions link1="leg2_link" link2="leg3_link" reason="Never"/>
+    <disable_collisions link1="leg2_link" link2="leg4_link" reason="Never"/>
+    <disable_collisions link1="leg2_link" link2="obar1_link" reason="Never"/>
+    <disable_collisions link1="leg2_link" link2="obar2_link" reason="Never"/>
+    <disable_collisions link1="leg2_link" link2="obar3_link" reason="Never"/>
+    <disable_collisions link1="leg2_link" link2="obar4_link" reason="Never"/>
+    <disable_collisions link1="leg2_link" link2="sliding_guide_link" reason="Never"/>
+    <disable_collisions link1="leg2_link" link2="table_top_link" reason="Adjacent"/>
+    <disable_collisions link1="leg2_link" link2="vbar1_link" reason="Never"/>
+    <disable_collisions link1="leg2_link" link2="vbar2_link" reason="Adjacent"/>
+    <disable_collisions link1="leg2_link" link2="vbar3_link" reason="Never"/>
+    <disable_collisions link1="leg2_link" link2="vbar4_link" reason="Never"/>
+    <disable_collisions link1="leg3_link" link2="leg4_link" reason="Never"/>
+    <disable_collisions link1="leg3_link" link2="obar1_link" reason="Never"/>
+    <disable_collisions link1="leg3_link" link2="obar2_link" reason="Never"/>
+    <disable_collisions link1="leg3_link" link2="obar3_link" reason="Never"/>
+    <disable_collisions link1="leg3_link" link2="obar4_link" reason="Never"/>
+    <disable_collisions link1="leg3_link" link2="sliding_guide_link" reason="Never"/>
+    <disable_collisions link1="leg3_link" link2="table_top_link" reason="Adjacent"/>
+    <disable_collisions link1="leg3_link" link2="vbar1_link" reason="Never"/>
+    <disable_collisions link1="leg3_link" link2="vbar2_link" reason="Never"/>
+    <disable_collisions link1="leg3_link" link2="vbar3_link" reason="Adjacent"/>
+    <disable_collisions link1="leg3_link" link2="vbar4_link" reason="Never"/>
+    <disable_collisions link1="leg4_link" link2="obar1_link" reason="Never"/>
+    <disable_collisions link1="leg4_link" link2="obar2_link" reason="Never"/>
+    <disable_collisions link1="leg4_link" link2="obar3_link" reason="Never"/>
+    <disable_collisions link1="leg4_link" link2="obar4_link" reason="Never"/>
+    <disable_collisions link1="leg4_link" link2="sliding_guide_link" reason="Never"/>
+    <disable_collisions link1="leg4_link" link2="table_top_link" reason="Adjacent"/>
+    <disable_collisions link1="leg4_link" link2="vbar1_link" reason="Never"/>
+    <disable_collisions link1="leg4_link" link2="vbar2_link" reason="Never"/>
+    <disable_collisions link1="leg4_link" link2="vbar3_link" reason="Never"/>
+    <disable_collisions link1="leg4_link" link2="vbar4_link" reason="Adjacent"/>
+    <disable_collisions link1="obar1_link" link2="obar2_link" reason="Never"/>
+    <disable_collisions link1="obar1_link" link2="obar3_link" reason="Default"/>
+    <disable_collisions link1="obar1_link" link2="obar4_link" reason="Default"/>
+    <disable_collisions link1="obar1_link" link2="sliding_guide_link" reason="Default"/>
+    <disable_collisions link1="obar1_link" link2="table_top_link" reason="Never"/>
+    <disable_collisions link1="obar1_link" link2="vbar1_link" reason="Adjacent"/>
+    <disable_collisions link1="obar1_link" link2="vbar2_link" reason="Default"/>
+    <disable_collisions link1="obar1_link" link2="vbar3_link" reason="Never"/>
+    <disable_collisions link1="obar1_link" link2="vbar4_link" reason="Never"/>
+    <disable_collisions link1="obar2_link" link2="obar3_link" reason="Default"/>
+    <disable_collisions link1="obar2_link" link2="obar4_link" reason="Default"/>
+    <disable_collisions link1="obar2_link" link2="sliding_guide_link" reason="Adjacent"/>
+    <disable_collisions link1="obar2_link" link2="table_top_link" reason="Never"/>
+    <disable_collisions link1="obar2_link" link2="vbar1_link" reason="Never"/>
+    <disable_collisions link1="obar2_link" link2="vbar2_link" reason="Never"/>
+    <disable_collisions link1="obar2_link" link2="vbar3_link" reason="Adjacent"/>
+    <disable_collisions link1="obar2_link" link2="vbar4_link" reason="Default"/>
+    <disable_collisions link1="obar3_link" link2="obar4_link" reason="Never"/>
+    <disable_collisions link1="obar3_link" link2="sliding_guide_link" reason="Never"/>
+    <disable_collisions link1="obar3_link" link2="table_top_link" reason="Never"/>
+    <disable_collisions link1="obar3_link" link2="vbar1_link" reason="Default"/>
+    <disable_collisions link1="obar3_link" link2="vbar2_link" reason="Never"/>
+    <disable_collisions link1="obar3_link" link2="vbar3_link" reason="Adjacent"/>
+    <disable_collisions link1="obar3_link" link2="vbar4_link" reason="Never"/>
+    <disable_collisions link1="obar4_link" link2="sliding_guide_link" reason="Never"/>
+    <disable_collisions link1="obar4_link" link2="table_top_link" reason="Never"/>
+    <disable_collisions link1="obar4_link" link2="vbar1_link" reason="Never"/>
+    <disable_collisions link1="obar4_link" link2="vbar2_link" reason="Default"/>
+    <disable_collisions link1="obar4_link" link2="vbar3_link" reason="Never"/>
+    <disable_collisions link1="obar4_link" link2="vbar4_link" reason="Adjacent"/>
+    <disable_collisions link1="sliding_guide_link" link2="table_top_link" reason="Never"/>
+    <disable_collisions link1="sliding_guide_link" link2="vbar1_link" reason="Never"/>
+    <disable_collisions link1="sliding_guide_link" link2="vbar2_link" reason="Never"/>
+    <disable_collisions link1="sliding_guide_link" link2="vbar3_link" reason="Never"/>
+    <disable_collisions link1="sliding_guide_link" link2="vbar4_link" reason="Never"/>
+    <disable_collisions link1="table_top_link" link2="vbar1_link" reason="Default"/>
+    <disable_collisions link1="table_top_link" link2="vbar2_link" reason="Default"/>
+    <disable_collisions link1="table_top_link" link2="vbar3_link" reason="Default"/>
+    <disable_collisions link1="table_top_link" link2="vbar4_link" reason="Default"/>
+    <disable_collisions link1="vbar1_link" link2="vbar2_link" reason="Never"/>
+    <disable_collisions link1="vbar1_link" link2="vbar3_link" reason="Never"/>
+    <disable_collisions link1="vbar1_link" link2="vbar4_link" reason="Never"/>
+    <disable_collisions link1="vbar2_link" link2="vbar3_link" reason="Never"/>
+    <disable_collisions link1="vbar2_link" link2="vbar4_link" reason="Never"/>
+    <disable_collisions link1="vbar3_link" link2="vbar4_link" reason="Never"/> -->
 </robot>

File: repair_urdf/urdf/gazebo/xbot.gazebo.xacro (robot description, xacro)
@@ -2,4 +2,5 @@
 <robot xmlns:xacro="http://ros.org/wiki/xacro">
 <gazebo>
+    <xacro:include filename="$(find repair_urdf)/urdf/gazebo/ignore_joint_softhand.xbot.xacro" />
     <plugin name="xbot2_joint_driver" filename="libxbot2_gz_joint_server.so">
         <pid>
@@ -23,4 +24,8 @@
             <pid name="j_arm_2_7" profile="small_mot"/>
         </pid>
+        <ignore_joints>
+            <xacro:ignore_softhand_jnts side="right" type="v1s"/>
+            <xacro:ignore_softhand_jnts side="left" type="v1s"/>
+        </ignore_joints>
     </plugin>
 </gazebo>

File: repair_urdf/urdf/repair.transmission.xacro (robot description, xacro)
@@ -2,70 +2,70 @@
 <robot xmlns:xacro="http://www.ros.org/wiki/xacro">
   <xacro:macro name="repair_arm_transmission" params="id">
-    <transmission name="trans_arm_${id}_joint_1">
+    <transmission name="trans_j_arm_${id}_1">
         <type>transmission_interface/SimpleTransmission</type>
-        <joint name="arm_${id}_joint_1">
+        <joint name="j_arm_${id}_1">
             <hardwareInterface>hardware_interface/PositionJointInterface</hardwareInterface>
         </joint>
-        <actuator name="arm_${id}_joint_1_motor">
+        <actuator name="j_arm_${id}_1_motor">
             <hardwareInterface>hardware_interface/PositionJointInterface</hardwareInterface>
             <mechanicalReduction>1</mechanicalReduction>
         </actuator>
     </transmission>
-    <transmission name="trans_arm_${id}_joint_2">
+    <transmission name="trans_j_arm_${id}_2">
         <type>transmission_interface/SimpleTransmission</type>
-        <joint name="arm_${id}_joint_2">
+        <joint name="j_arm_${id}_2">
             <hardwareInterface>hardware_interface/PositionJointInterface</hardwareInterface>
         </joint>
-        <actuator name="arm_${id}_joint_2_motor">
+        <actuator name="j_arm_${id}_2_motor">
             <hardwareInterface>hardware_interface/PositionJointInterface</hardwareInterface>
             <mechanicalReduction>1</mechanicalReduction>
         </actuator>
     </transmission>
-    <transmission name="trans_arm_${id}_joint_3">
+        <transmission name="trans_j_arm_${id}_3">
         <type>transmission_interface/SimpleTransmission</type>
-        <joint name="arm_${id}_joint_3">
+        <joint name="j_arm_${id}_3">
             <hardwareInterface>hardware_interface/PositionJointInterface</hardwareInterface>
         </joint>
-        <actuator name="arm_${id}_joint_3_motor">
+        <actuator name="j_arm_${id}_3_motor">
             <hardwareInterface>hardware_interface/PositionJointInterface</hardwareInterface>
             <mechanicalReduction>1</mechanicalReduction>
         </actuator>
     </transmission>
-    <transmission name="trans_arm_${id}_joint_4">
+    <transmission name="trans_j_arm_${id}_4">
         <type>transmission_interface/SimpleTransmission</type>
-        <joint name="arm_${id}_joint_4">
+        <joint name="j_arm_${id}_4">
             <hardwareInterface>hardware_interface/PositionJointInterface</hardwareInterface>
         </joint>
-        <actuator name="arm_${id}_joint_4_motor">
+        <actuator name="j_arm_${id}_4_motor">
             <hardwareInterface>hardware_interface/PositionJointInterface</hardwareInterface>
             <mechanicalReduction>1</mechanicalReduction>
         </actuator>
     </transmission>
-    <transmission name="trans_arm_${id}_joint_5">
+    <transmission name="trans_j_arm_${id}_5">
         <type>transmission_interface/SimpleTransmission</type>
-        <joint name="arm_${id}_joint_5">
+        <joint name="j_arm_${id}_5">
             <hardwareInterface>hardware_interface/PositionJointInterface</hardwareInterface>
         </joint>
-        <actuator name="arm_${id}_joint_5_motor">
+        <actuator name="j_arm_${id}_5_motor">
             <hardwareInterface>hardware_interface/PositionJointInterface</hardwareInterface>
             <mechanicalReduction>1</mechanicalReduction>
         </actuator>
     </transmission>
-    <transmission name="trans_arm_${id}_joint_6">
+    <transmission name="trans_j_arm_${id}_6">
         <type>transmission_interface/SimpleTransmission</type>
-        <joint name="arm_${id}_joint_6">
+        <joint name="j_arm_${id}_6">
             <hardwareInterface>hardware_interface/PositionJointInterface</hardwareInterface>
         </joint>
-        <actuator name="arm_${id}_joint_6_motor">
+        <actuator name="j_arm_${id}_6_motor">
             <hardwareInterface>hardware_interface/PositionJointInterface</hardwareInterface>
             <mechanicalReduction>1</mechanicalReduction>
         </actuator>
     </transmission>
-    <transmission name="trans_arm_${id}_joint_7">
+    <transmission name="trans_j_arm_${id}_7">
         <type>transmission_interface/SimpleTransmission</type>
-        <joint name="arm_${id}_joint_7">
+        <joint name="j_arm_${id}_7">
             <hardwareInterface>hardware_interface/PositionJointInterface</hardwareInterface>
         </joint>
-        <actuator name="arm_${id}_joint_7_motor">
+        <actuator name="j_arm_${id}_7_motor">
             <hardwareInterface>hardware_interface/PositionJointInterface</hardwareInterface>
             <mechanicalReduction>1</mechanicalReduction>
