Commit message: cleaned version with softhands

File: repair_urdf/urdf/repair_full.urdf.xacro (robot description, xacro)
@@ -1,4 +1,5 @@
 <?xml version="1.0"?>
 <robot xmlns:xacro="http://ros.org/wiki/xacro" name="repair_full">
+    <xacro:include filename="$(find softhands_description)/urdf/softhands.xacro" />
     <xacro:include filename="$(find repair_urdf)/urdf/conversions.urdf.xacro" />
     <xacro:include filename="$(find repair_urdf)/urdf/materials.urdf.xacro" />
@@ -10,4 +11,6 @@
     <xacro:include filename="$(find repair_urdf)/urdf/limits.urdf.xacro" />
     <xacro:include filename="$(find repair_urdf)/urdf/gazebo/xbot.gazebo.xacro" />
+    <!-- <xacro:include filename="$(find repair_urdf)/urdf/repair.transmission.xacro" />-->
+    <xacro:include filename="$(find repair_urdf)/urdf/common.gazebo.xacro" />
     <link name="world"/>
     <xacro:repair_cage parent="world">
@@ -25,3 +28,24 @@
                 rpy="${-Shoulder_1_roll} ${Shoulder_1_pitch} ${Shoulder_1_yaw}" />
       </xacro:repair_arm>
+    <xacro:softhands type="left"
+        version="v1.0_simple"
+        parent="arm_1_7"
+        position="0 0 -0.015"
+        orientation="0 0.0 ${PI}"
+        translation="0"
+        operation_mode="0"
+        fixed_hands="false">
+    </xacro:softhands>
+    <xacro:softhands type="right"
+        version="v1.0_simple"
+        parent="arm_2_7"
+        position="0 -0.013900 -0.015"
+        orientation="0 0 ${PI}"
+        translation="0"
+        operation_mode="0"
+        fixed_hands="false">
+    </xacro:softhands>
+    <!-- <gazebo reference="table_top_link">
+        <selfCollide> 1 </selfCollide>
+    </gazebo> -->
 </robot>

Commit message: tries for bimanual manipulation with cartesio

File: repair_srdf/srdf/repair_full.srdf.xacro (robot description, xacro)
@@ -33,17 +33,17 @@
     <group_state name="home" group="chains">
         <joint name="j_arm_1_1" value="-0.5"/>
-        <joint name="j_arm_1_2" value="-0.5"/>
+        <joint name="j_arm_1_2" value="-0.7"/>
         <joint name="j_arm_1_3" value="0.5"/>
-        <joint name="j_arm_1_4" value="-1.0"/>
+        <joint name="j_arm_1_4" value="-1.2"/>
         <joint name="j_arm_1_5" value="-0.5"/>
-        <joint name="j_arm_1_6" value="-0.5"/>
-        <joint name="j_arm_1_7" value="-1.0"/>
+        <joint name="j_arm_1_6" value="0.5"/>
+        <joint name="j_arm_1_7" value="0.5"/>
         <joint name="j_arm_2_1" value="0.5"/>
-        <joint name="j_arm_2_2" value="0.5"/>
+        <joint name="j_arm_2_2" value="0.7"/>
         <joint name="j_arm_2_3" value="-0.5"/>
-        <joint name="j_arm_2_4" value="1.0"/>
+        <joint name="j_arm_2_4" value="1.2"/>
         <joint name="j_arm_2_5" value="0.5"/>
-        <joint name="j_arm_2_6" value="0.5"/>
-        <joint name="j_arm_2_7" value="1.0"/>
+        <joint name="j_arm_2_6" value="-0.5"/>
+        <joint name="j_arm_2_7" value="-0.5"/>
         <!-- <xacro:softhand_homing side="right" type="v1s"/>
         <xacro:softhand_homing side="left" type="v1s"/> -->

File: repair_urdf/urdf/limits.urdf.xacro (robot description, xacro)
@@ -2,5 +2,5 @@
 <robot  xmlns:xacro="http://ros.org/wiki/xacro">
     <!-- Origin -->
-    <xacro:property name="j_prismatic_lower" value="${[-2]}"/>
+    <xacro:property name="j_prismatic_lower" value="${[-0.80]}"/>
     <xacro:property name="j_torso_lower" value="${[-2.6]}"/>
     <xacro:property name="j_arm_1_lower" value="${[-2.6, -2.6]}"/>
@@ -11,9 +11,9 @@
     <xacro:property name="j_arm_6_lower" value="${[-2.8, -2.1]}"/>
     <xacro:property name="j_arm_7_lower" value="${[-2.8, -2.8]}"/>
-    <xacro:property name="j_prismatic_upper" value="${[2]}"/>
+    <xacro:property name="j_prismatic_upper" value="${[0.80]}"/>
     <xacro:property name="j_torso_upper" value="${[2.6]}"/>
     <xacro:property name="j_arm_1_upper" value="${[2.6, 2.6]}"/>
+    <xacro:property name="j_arm_3_upper" value="${[2.6, 2.6]}"/>
     <xacro:property name="j_arm_2_upper" value="${[2.5, 0.1]}"/>
-    <xacro:property name="j_arm_3_upper" value="${[2.6, 2.6]}"/>
     <xacro:property name="j_arm_4_upper" value="${[2.4, 0.8]}"/>
     <xacro:property name="j_arm_5_upper" value="${[2.8, 2.8]}"/>

File: repair_urdf/urdf/repair_arm_macro.urdf.xacro (robot description, xacro)
@@ -171,5 +171,5 @@
             <origin xyz="${Shoulder_2_Ox} ${rot*Shoulder_2_Oy} ${Shoulder_2_Oz}"
             rpy="${rot*Shoulder_2_roll} ${Shoulder_2_pitch} ${Shoulder_2_yaw}" />
-            <axis xyz="0 0 1" /> <!-- -1 -->
+            <axis xyz="0 0 1" />
             <limit lower="${j_arm_2_lower[limit_index]}" upper="${j_arm_2_upper[limit_index]}"
             effort="${j_arm_2_torque[0]}" velocity="${j_arm_2_velocity[0]}" />
@@ -182,5 +182,5 @@
             <origin xyz="${Shoulder_3_Ox} ${rot*Shoulder_3_Oy} ${Shoulder_3_Oz}"
             rpy="${rot*Shoulder_3_roll} ${Shoulder_3_pitch} ${Shoulder_3_yaw}" />
-            <axis xyz="0 0 -1" /> <!-- -1 -->
+            <axis xyz="0 0 -1" />
             <limit lower="${j_arm_3_lower[limit_index]}" upper="${j_arm_3_upper[limit_index]}"
             effort="${j_arm_3_torque[0]}" velocity="${j_arm_3_velocity[0]}" />
@@ -193,5 +193,5 @@
             <origin xyz="${Elbow_1_Ox} ${rot*Elbow_1_Oy} ${Elbow_1_Oz}"
             rpy="${rot*Elbow_1_roll} ${Elbow_1_pitch} ${Elbow_1_yaw}" />
-            <axis xyz="0 0 1" /> <!-- -1 -->
+            <axis xyz="0 0 1" />
             <limit lower="${j_arm_4_lower[limit_index]}" upper="${j_arm_4_upper[limit_index]}"
             effort="${j_arm_4_torque[0]}" velocity="${j_arm_4_velocity[0]}" />
@@ -204,5 +204,5 @@
             <origin xyz="${Forearm_1_Ox} ${rot*Forearm_1_Oy} ${Forearm_1_Oz}"
             rpy="${rot*Forearm_1_roll} ${Forearm_1_pitch} ${Forearm_1_yaw}" />
-            <axis xyz="0 0 -1" /> <!-- -1 -->
+            <axis xyz="0 0 -1" />
             <limit lower="${j_arm_5_lower[limit_index]}" upper="${j_arm_5_upper[limit_index]}"
             effort="${j_arm_5_torque[0]}" velocity="${j_arm_5_velocity[0]}" />

File: repair_urdf/urdf/repair_full copy.urdf (robot description, URDF)
Before this commit: robot repair_full, 120 links, 119 joints
Links:
- removed link camera_left_ir_frame
- removed link camera_left_ir_optical_frame
- removed link camera_right_ir_frame
- removed link camera_right_ir_optical_frame
- added link arm_1_angle_flange; collision mesh filename=package://repair_urdf/meshes/angle_flange_90.stl scale=0.001 0.001 0.001; visual mesh filename=package://repair_urdf/meshes/angle_flange_90.stl scale=0.001 0.001 0.001
- added link arm_1_camera_mount; collision mesh filename=package://repair_urdf/meshes/camera_supp_cover_wide_left.stl scale=0.001 0.001 0.001; visual mesh filename=package://repair_urdf/meshes/camera_supp_cover_wide_left.stl scale=0.001 0.001 0.001
- added link arm_2_angle_flange; collision mesh filename=package://repair_urdf/meshes/angle_flange_90.stl scale=0.001 0.001 0.001; visual mesh filename=package://repair_urdf/meshes/angle_flange_90.stl scale=0.001 0.001 0.001
- added link arm_2_camera_mount; collision mesh filename=package://repair_urdf/meshes/camera_supp_cover_sh1p2.stl scale=0.001 0.001 0.001; visual mesh filename=package://repair_urdf/meshes/camera_supp_cover_sh1p2.stl scale=0.001 0.001 0.001
- added link camera_accel_frame
- added link camera_accel_optical_frame
- added link camera_gyro_frame
- added link camera_gyro_optical_frame
- added link camera_infra_frame
- added link camera_infra_optical_frame
- added link camera_lower_mount
- added link camera_upper_mount
- link arm_1_1: geometry collision mesh filename=package://repair_urdf/meshes/simplified/mesh_sh-pitch.stl scale=0.001 -0.001 0.001; visual mesh filename=package://repair_urdf/meshes/simplified/mesh_sh-pitch.stl scale=0.001 -0.001 0.001
- link arm_1_2: geometry collision mesh filename=package://repair_urdf/meshes/simplified/mesh_sh-roll.stl scale=0.001 -0.001 0.001; visual mesh filename=package://repair_urdf/meshes/simplified/mesh_sh-roll.stl scale=0.001 -0.001 0.001
- link arm_1_3: geometry collision mesh filename=package://repair_urdf/meshes/simplified/mesh_sh-yaw.stl scale=0.001 -0.001 0.001; visual mesh filename=package://repair_urdf/meshes/simplified/mesh_sh-yaw.stl scale=0.001 -0.001 0.001
- link arm_1_4: geometry collision mesh filename=package://repair_urdf/meshes/simplified/mesh_elbow.stl scale=0.001 -0.001 0.001; visual mesh filename=package://repair_urdf/meshes/simplified/mesh_elbow.stl scale=0.001 -0.001 0.001
- link arm_1_5: geometry collision mesh filename=package://repair_urdf/meshes/simplified/mesh_forearm-yaw.stl scale=0.001 -0.001 0.001; visual mesh filename=package://repair_urdf/meshes/simplified/mesh_forearm-yaw.stl scale=0.001 -0.001 0.001
- link arm_1_6: geometry collision mesh filename=package://repair_urdf/meshes/simplified/mesh_wrist-pitch.stl scale=0.001 -0.001 0.001; visual mesh filename=package://repair_urdf/meshes/simplified/mesh_wrist-pitch.stl scale=0.001 -0.001 0.001
- link arm_1_7: geometry collision mesh filename=package://repair_urdf/meshes/simplified/mesh_wrist-roll.stl scale=0.001 -0.001 0.001; visual mesh filename=package://repair_urdf/meshes/simplified/mesh_wrist-roll.stl scale=0.001 -0.001 0.001
- link arm_2_1: geometry collision mesh filename=package://repair_urdf/meshes/simplified/mesh_sh-pitch.stl scale=0.001 0.001 0.001; visual mesh filename=package://repair_urdf/meshes/simplified/mesh_sh-pitch.stl scale=0.001 0.001 0.001
- link arm_2_2: geometry collision mesh filename=package://repair_urdf/meshes/simplified/mesh_sh-roll.stl scale=0.001 0.001 0.001; visual mesh filename=package://repair_urdf/meshes/simplified/mesh_sh-roll.stl scale=0.001 0.001 0.001
- link arm_2_3: geometry collision mesh filename=package://repair_urdf/meshes/simplified/mesh_sh-yaw.stl scale=0.001 0.001 0.001; visual mesh filename=package://repair_urdf/meshes/simplified/mesh_sh-yaw.stl scale=0.001 0.001 0.001
- link arm_2_4: geometry collision mesh filename=package://repair_urdf/meshes/simplified/mesh_elbow.stl scale=0.001 0.001 0.001; visual mesh filename=package://repair_urdf/meshes/simplified/mesh_elbow.stl scale=0.001 0.001 0.001
- link arm_2_5: geometry collision mesh filename=package://repair_urdf/meshes/simplified/mesh_forearm-yaw.stl scale=0.001 0.001 0.001; visual mesh filename=package://repair_urdf/meshes/simplified/mesh_forearm-yaw.stl scale=0.001 0.001 0.001
- link arm_2_6: geometry collision mesh filename=package://repair_urdf/meshes/simplified/mesh_wrist-pitch.stl scale=0.001 0.001 0.001; visual mesh filename=package://repair_urdf/meshes/simplified/mesh_wrist-pitch.stl scale=0.001 0.001 0.001
- link arm_2_7: geometry collision mesh filename=package://repair_urdf/meshes/simplified/mesh_wrist-roll.stl scale=0.001 0.001 0.001; visual mesh filename=package://repair_urdf/meshes/simplified/mesh_wrist-roll.stl scale=0.001 0.001 0.001
- link camera_link: mass 0.564 -> 0.095; geometry collision cylinder length=0.026 radius=0.0305; visual mesh filename=package://realsense_description_l515/meshes/l515.dae
- link leg1_link: geometry collision cylinder length=0.978 radius=0.02; visual cylinder length=0.978 radius=0.02
- link leg2_link: geometry collision cylinder length=0.978 radius=0.02; visual cylinder length=0.978 radius=0.02
- link leg3_link: geometry collision cylinder length=0.978 radius=0.02; visual cylinder length=0.978 radius=0.02
- link leg4_link: geometry collision cylinder length=0.978 radius=0.02; visual cylinder length=0.978 radius=0.02
- link sliding_guide_link: geometry collision box size=0.001 1.0 2.5; visual box size=0.001 0.4 2.5
- link table_top_link: geometry collision box size=1.0 2.5 0.028; visual box size=1.0 2.5 0.028
Joints:
- removed joint camera_left_ir_joint
- removed joint camera_left_ir_optical_joint
- removed joint camera_right_ir_joint
- removed joint camera_right_ir_optical_joint
- removed joint j_torso_base
- added joint arm_1_angle_flange_joint: type fixed, parent arm_1_7, child arm_1_angle_flange, origin xyz=0.0425 0 0.0430 rpy=0 1.5707963 0
- added joint arm_1_camera_mount_joint: type fixed, parent arm_1_7, child arm_1_camera_mount, origin xyz=0.17545 0.016874 -0.01 rpy=0 1.5707963 0
- added joint arm_2_angle_flange_joint: type fixed, parent arm_2_7, child arm_2_angle_flange, origin xyz=0.0425 0 0.0380 rpy=0 1.5707963 0
- added joint arm_2_camera_mount_joint: type fixed, parent arm_2_7, child arm_2_camera_mount, origin xyz=0.18145 0.00528118 -0.01350 rpy=0 1.5707963 0
- added joint camera_accel_joint: type fixed, parent camera_color_frame, child camera_accel_frame, origin xyz=-0.00410137791186571 -0.0129784867167473 0.00256138201802969 rpy=-0.006161012 0.020193459 0.016301375
- added joint camera_accel_optical_joint: type fixed, parent camera_accel_frame, child camera_accel_optical_frame, origin xyz=0 0 0 rpy=-1.5707963267948966 0 -1.5707963267948966
- added joint camera_gyro_joint: type fixed, parent camera_color_frame, child camera_gyro_frame, origin xyz=-0.00410137791186571 -0.0129784867167473 0.00256138201802969 rpy=-0.006161012 0.020193459 0.016301375
- added joint camera_gyro_optical_joint: type fixed, parent camera_gyro_frame, child camera_gyro_optical_frame, origin xyz=0 0 0 rpy=-1.5707963267948966 0 -1.5707963267948966
- added joint camera_infra_joint: type fixed, parent camera_link, child camera_infra_frame, origin xyz=0 0.0 0 rpy=0 0 0
- added joint camera_infra_optical_joint: type fixed, parent camera_infra_frame, child camera_infra_optical_frame, origin xyz=0 0 0 rpy=-1.5707963267948966 0 -1.5707963267948966
- added joint camera_lower_mount_joint: type fixed, parent camera_bottom_screw_frame, child camera_lower_mount, origin xyz=-0.013999999999999999 0 0.01015 rpy=0 0 0
- added joint camera_upper_mount_joint: type fixed, parent camera_bottom_screw_frame, child camera_upper_mount, origin xyz=-0.013999999999999999 0 0.05015 rpy=0 0 0
- added joint j_sliding_guide: type fixed, parent sliding_guide_link, child dummy_prismatic_link, origin xyz=0 0 0 rpy=0 0 0
- joint camera_color_joint: origin xyz=0 0.015 0 rpy=0 0 0 -> xyz=0 0 0.024 rpy=0 0 0; parent camera_depth_frame -> camera_link
- joint camera_link_joint: origin xyz=0 0.0175 0.0125 rpy=0 0 0 -> xyz=0.007500000000000001 0.0 0.021150000000000002 rpy=0 0 0
- joint j_torso_1: axis 0 0 1 -> (none); limit lower=-2.6 upper=2.6 effort=147.0 velocity=3.86 -> (none); type revolute -> fixed
- joint left_hand_v1_wide_palm_central_joint: origin xyz=0 0 0.0 rpy=0 0 1.570796326795 -> xyz=0.005 0 0 rpy=0 0 3.14159265359; parent arm_1_7 -> arm_1_angle_flange
- joint leg1_joint: origin xyz=0.5 1.25 1.0 rpy=0 0 0 -> xyz=0.5 1.25 0.978 rpy=0 0 0
- joint leg2_joint: origin xyz=-0.5 1.25 1.0 rpy=0 0 0 -> xyz=-0.5 1.25 0.978 rpy=0 0 0
- joint leg3_joint: origin xyz=0.5 -1.25 1.0 rpy=0 0 0 -> xyz=0.5 -1.25 0.978 rpy=0 0 0
- joint leg4_joint: origin xyz=-0.5 -1.25 1.0 rpy=0 0 0 -> xyz=-0.5 -1.25 0.978 rpy=0 0 0
- joint right_hand_v1_2_research_iso_joint: origin xyz=0 0.0 0.00 rpy=0 0 3.14159265359 -> xyz=0.005 0 0 rpy=0 0 1.570796326795; parent arm_2_7 -> arm_2_angle_flange

File: repair_urdf/urdf/repair_full.urdf.xacro (robot description, xacro)
@@ -37,5 +37,5 @@
     <!--QUIRINO/GIANNIROS: here change the version for v1_2_research (small hand) or v1_wide (wide hand)-->
     <xacro:softhands
-        version="v1_2_research"
+        version="mixed_hands"
         position="0 0 0"
         orientation="${PI}"

File: repair_urdf/urdf/repair_torso_macro.urdf.xacro (robot description, xacro)
@@ -2,5 +2,5 @@
 <robot xmlns:xacro="http://ros.org/wiki/xacro">
     <xacro:macro name="repair_torso" params="parent *origin">
-        <!-- <link name="dummy_prismatic_link"/> -->
+        <link name="dummy_prismatic_link"/>
         <link name="torso_1">
             <inertial>
@@ -22,14 +22,14 @@
             </collision>
         </link>
-        <!-- <joint name="j_torso_base" type="fixed">
+        <joint name="j_torso_base" type="prismatic">
             <xacro:insert_block name="origin" />
             <parent link="${parent}" />
             <child link="dummy_prismatic_link"/>
             <axis xyz="0 0 1"/>
-            <limit lower="${j_prismatic_lower[0]/2}" upper= "${j_prismatic_upper[0]/2}" effort="${j_prismatic_torque[0]}" velocity="${j_prismatic_velocity[0]}"/>
-        </joint> -->
+            <limit lower="${j_prismatic_lower[0]}" upper= "${j_prismatic_upper[0]}" effort="${j_prismatic_torque[0]}" velocity="${j_prismatic_velocity[0]}"/>
+        </joint>
         <!-- torso -->
         <joint name="j_torso_1" type="revolute">
-            <parent link="${parent}" />
+            <parent link="dummy_prismatic_link" />
             <child link="torso_1" />
             <axis xyz="0 0 1" />
@@ -39,4 +39,11 @@
         </joint>
         <!-- torso  -->
+        <!-- torso -->
+        <!--<joint name="j_torso_1" type="fixed">
+            <parent link="${parent}" />
+            <child link="torso_1" />
+            <xacro:insert_block name="origin" />
+        </joint>-->
+        <!-- torso  -->
     </xacro:macro>
 </robot>
