Commit message: added sliding_guide joint to gazebo, still unable to control it

File: repair_moveit_config/config/gazebo_repair_full.urdf (robot description, URDF)
Before this commit: robot repair_full, 33 links, 32 joints
Joints:
- joint j_torso_1: axis 0 0 1 -> (none); limit lower=-2.6 upper=2.6 effort=147.0 velocity=3.86 -> (none); type revolute -> fixed

File: repair_moveit_config_v2/config/gazebo_repair_full.urdf (robot description, URDF)
Before this commit: robot repair_full, 120 links, 119 joints
Joints:
- joint j_torso_1: axis 0 0 1 -> (none); limit lower=-2.6 upper=2.6 effort=147.0 velocity=3.86 -> (none); type revolute -> fixed

File: repair_moveit_config_v2/config/repair_full.srdf.xacro (robot description, xacro)
@@ -22,7 +22,7 @@
         <group name="arm_2"/>
     </group>
-    <group name="torso">
+    <!-- <group name="torso">
         <joint name="j_torso_1"/>
-    </group>
+    </group> -->
     <group name="sliding_guide">
         <joint name="j_sliding_guide"/>
@@ -70,7 +70,7 @@
         <joint name="j_arm_2_7" value="0"/>
     </group_state>
-    <group_state name="home" group="torso">
+    <!-- <group_state name="home" group="torso">
         <joint name="j_torso_1" value="0"/>
-    </group_state>
+    </group_state> -->
     <!-- IF sh_version= v1_wide  -->
     <xacro:if value="${sh_version == 'v1_wide'}">

File: repair_srdf/srdf/repair_full.srdf.xacro (robot description, xacro)
@@ -4,7 +4,7 @@
     <xacro:include filename="$(find softhands_description)/srdf/softhands.srdf.xacro"/>
     <xacro:include filename="$(find softhands_description)/srdf/softhands_homing.srdf.xacro"/> -->
-    <!-- <group name="sliding_guide">
+    <group name="sliding_guide">
         <chain base_link="sliding_guide_link" tip_link="torso_1"/>
-    </group> -->
+    </group>
     <group name="arm1">
         <chain base_link="torso_1" tip_link="arm_1_tcp"/>
@@ -14,5 +14,5 @@
     </group>
     <group name="chains">
-        <!-- <group name="sliding_guide" /> -->
+        <group name="sliding_guide" />
         <group name="arm1"/>
         <group name="arm2"/>

File: repair_urdf/urdf/model.urdf (robot description, URDF)
Before this commit: robot repair_full, 43 links, 42 joints
Joints:
- joint j_torso_1: axis 0 0 1 -> (none); limit lower=-2.6 upper=2.6 effort=147.0 velocity=3.86 -> (none); type revolute -> fixed

File: repair_urdf/urdf/repair.transmission.xacro (robot description, xacro)
@@ -72,14 +72,24 @@
         </actuator>
     </transmission>
-        <!-- <transmission name="trans_j_torso_1">
-            <type>transmission_interface/SimpleTransmission</type>
-            <joint name="j_torso_1">
-                <hardwareInterface>hardware_interface/PositionJointInterface</hardwareInterface>
-            </joint>
-            <actuator name="j_torso_1_motor">
-                <hardwareInterface>hardware_interface/PositionJointInterface</hardwareInterface>
-                <mechanicalReduction>1</mechanicalReduction>
-            </actuator>
-        </transmission> -->
+    <transmission name="trans_j_sliding_guide">
+        <type>transmission_interface/SimpleTransmission</type>
+        <joint name="j_sliding_guide">
+            <hardwareInterface>hardware_interface/PositionJointInterface</hardwareInterface>
+        </joint>
+        <actuator name="j_sliding_guide_motor">
+            <hardwareInterface>hardware_interface/PositionJointInterface</hardwareInterface>
+            <mechanicalReduction>1</mechanicalReduction>
+        </actuator>
+    </transmission>
+    <!-- <transmission name="trans_j_torso_1">
+        <type>transmission_interface/SimpleTransmission</type>
+        <joint name="j_torso_1">
+            <hardwareInterface>hardware_interface/PositionJointInterface</hardwareInterface>
+        </joint>
+        <actuator name="j_torso_1_motor">
+            <hardwareInterface>hardware_interface/PositionJointInterface</hardwareInterface>
+            <mechanicalReduction>1</mechanicalReduction>
+        </actuator>
+    </transmission> -->
   </xacro:macro>
 </robot>

File: repair_urdf/urdf/repair_full_with_sliding_guide.urdf (robot description, URDF)
Before this commit: robot repair_full, 120 links, 119 joints
Joints:
- joint j_torso_1: axis 0 0 1 -> (none); limit lower=-2.6 upper=2.6 effort=147.0 velocity=3.86 -> (none); type revolute -> fixed

File: repair_urdf/urdf/repair_torso_macro.urdf.xacro (robot description, xacro)
@@ -2,10 +2,10 @@
 <robot xmlns:xacro="http://ros.org/wiki/xacro">
     <xacro:macro name="repair_torso" params="parent *origin">
-        <joint name="j_sliding_guide" type="fixed">
+        <joint name="j_sliding_guide" type="prismatic">
             <origin xyz="0 0 0" rpy="0 0 0" />
             <parent link="${parent}" />
             <child link="dummy_prismatic_link"/>
-            <!-- <axis xyz="0 0 -1"/> -->
-            <!-- <limit lower="${j_prismatic_lower[0]/2}" upper= "${j_prismatic_upper[0]/2}" effort="${j_prismatic_torque[0]}" velocity="${j_prismatic_velocity[0]}"/> -->
+            <axis xyz="0 0 -1"/>
+            <limit lower="${j_prismatic_lower[0]/2}" upper= "${j_prismatic_upper[0]/2}" effort="${j_prismatic_torque[0]}" velocity="${j_prismatic_velocity[0]}"/>
         </joint>
         <link name="dummy_prismatic_link"/>
@@ -36,19 +36,10 @@
             <limit lower="${j_prismatic_lower[0]/2}" upper= "${j_prismatic_upper[0]/2}" effort="${j_prismatic_torque[0]}" velocity="${j_prismatic_velocity[0]}"/>
         </joint> -->
-        <joint name="j_torso_base" type="prismatic">
-        <!-- <xacro:insert_block name="origin" /> -->
-        <origin rpy="0.0 0.0 0.0" xyz="0.0 0.0 0.0"/>
-        <parent link="sliding_guide_link"/>
-                <child link="dummy_prismatic_link"/>
-                <axis xyz="0 0 1"/>
-        <limit effort="147" lower="-0.8" upper="0.8" velocity="2.2"/>
-            </joint>
-        <!-- torso -->
-        <joint name="j_torso_1" type="revolute">
+        <joint name="j_torso_1" type="fixed">
             <parent link="dummy_prismatic_link"/>
             <child link="torso_1"/>
-            <axis xyz="0 0 1"/>
+            <!-- <axis xyz="0 0 1"/> -->
             <origin rpy="1.570796326795 0.0 1.570796326795" xyz="0.0 0.0 0.0"/>
-            <limit effort="147.0" lower="-2.6" upper="2.6" velocity="2.0"/>
+            <!-- <limit effort="147.0" lower="-2.6" upper="2.6" velocity="2.0"/> -->
         </joint>
     </xacro:macro>
