Commit message: changes to xacro and urdf in files for gazebo and stuff

File: repair_moveit_config_v3/config/gazebo_repair_full.urdf (robot description, URDF)
Before this commit: robot repair_full, 124 links, 123 joints
Links:
- added link arm_1_angle_flange; collision mesh filename=package://repair_urdf/meshes/angle_flange_90.stl scale=0.001 0.001 0.001; visual mesh filename=package://repair_urdf/meshes/angle_flange_90.stl scale=0.001 0.001 0.001
- added link arm_1_camera_mount; collision mesh filename=package://repair_urdf/meshes/camera_supp_cover_wide_left.stl scale=0.001 0.001 0.001; visual mesh filename=package://repair_urdf/meshes/camera_supp_cover_wide_left.stl scale=0.001 0.001 0.001
- added link arm_2_angle_flange; collision mesh filename=package://repair_urdf/meshes/angle_flange_90.stl scale=0.001 0.001 0.001; visual mesh filename=package://repair_urdf/meshes/angle_flange_90.stl scale=0.001 0.001 0.001
- added link arm_2_camera_mount; collision mesh filename=package://repair_urdf/meshes/camera_supp_cover_sh1p2.stl scale=0.001 0.001 0.001; visual mesh filename=package://repair_urdf/meshes/camera_supp_cover_sh1p2.stl scale=0.001 0.001 0.001
- link dummy_prismatic_link: mass None -> 0.1
- link leg1_link: mass 0.1 -> None; geometry collision cylinder length=0.978 radius=0.02; visual cylinder length=0.978 radius=0.02
- link leg2_link: mass 0.1 -> None; geometry collision cylinder length=0.978 radius=0.02; visual cylinder length=0.978 radius=0.02
- link leg3_link: mass 0.1 -> None; geometry collision cylinder length=0.978 radius=0.02; visual cylinder length=0.978 radius=0.02
- link leg4_link: mass 0.1 -> None; geometry collision cylinder length=0.978 radius=0.02; visual cylinder length=0.978 radius=0.02
- link obar1_link: mass 0.1 -> None
- link obar2_link: mass 0.1 -> None
- link obar3_link: mass 0.1 -> None
- link obar4_link: mass 0.1 -> None
- link sliding_guide_link: mass 0.1 -> None; geometry collision box size=0.001 1.0 2.5; visual box size=0.001 0.4 2.5
- link table_top_link: mass 0.1 -> None; geometry collision box size=1.0 2.5 0.028; visual box size=1.0 2.5 0.028
- link vbar1_link: mass 0.1 -> None
- link vbar2_link: mass 0.1 -> None
- link vbar3_link: mass 0.1 -> None
- link vbar4_link: mass 0.1 -> None
Joints:
- removed joint j_sliding_guide
- added joint arm_1_angle_flange_joint: type fixed, parent arm_1_7, child arm_1_angle_flange, origin xyz=0.0425 0 0.0430 rpy=0 1.5707963 0
- added joint arm_1_camera_mount_joint: type fixed, parent arm_1_7, child arm_1_camera_mount, origin xyz=0.17545 0.016874 -0.01 rpy=0 1.5707963 0
- added joint arm_2_angle_flange_joint: type fixed, parent arm_2_7, child arm_2_angle_flange, origin xyz=0.0425 0 0.0380 rpy=0 1.5707963 0
- added joint arm_2_camera_mount_joint: type fixed, parent arm_2_7, child arm_2_camera_mount, origin xyz=0.18145 0.00528118 -0.01350 rpy=0 1.5707963 0
- added joint j_torso_base: type prismatic, parent sliding_guide_link, child dummy_prismatic_link, origin xyz=0.0 0.0 0.0 rpy=0.0 0.0 0.0, axis 0 0 1, limit lower=-0.8 upper=0.8 effort=147.0 velocity=0.25
- joint j_arm_1_7: origin xyz=0.0 -0.062877 0.05 rpy=1.570796326795 0.3316123 0.0 -> xyz=0.0 -0.062877 0.05 rpy=1.570796326795 0.0 0.0
- joint j_arm_2_7: origin xyz=0.0 0.062877 0.05 rpy=-1.570796326795 0.3316123 0.0 -> xyz=0.0 0.062877 0.05 rpy=-1.570796326795 0.0 0.0
- joint j_torso_1: axis (none) -> 0 0 1; limit (none) -> lower=-2.6 upper=2.6 effort=147.0 velocity=2.0; type fixed -> revolute
- joint left_hand_v1_wide_palm_central_joint: origin xyz=0 0 0.0 rpy=0 0 3.14159265359 -> xyz=0.005 0 0 rpy=0 0 3.14159265359; parent arm_1_7 -> arm_1_angle_flange
- joint leg1_joint: origin xyz=0.5 1.25 1.0 rpy=0 0 0 -> xyz=0.5 1.25 0.978 rpy=0 0 0
- joint leg2_joint: origin xyz=-0.5 1.25 1.0 rpy=0 0 0 -> xyz=-0.5 1.25 0.978 rpy=0 0 0
- joint leg3_joint: origin xyz=0.5 -1.25 1.0 rpy=0 0 0 -> xyz=0.5 -1.25 0.978 rpy=0 0 0
- joint leg4_joint: origin xyz=-0.5 -1.25 1.0 rpy=0 0 0 -> xyz=-0.5 -1.25 0.978 rpy=0 0 0
- joint right_hand_v1_2_research_iso_joint: origin xyz=0 0.0 0.00 rpy=0 0 1.570796326795 -> xyz=0.005 0 0 rpy=0 0 1.570796326795; parent arm_2_7 -> arm_2_angle_flange

File: repair_urdf/urdf/common.gazebo.xacro (robot description, xacro)
@@ -3,6 +3,6 @@
   <gazebo>
     <plugin name="ros_control" filename="libgazebo_ros_control.so">
-      <!--robotNamespace>/</robotNamespace-->
-      <!--robotSimType>gazebo_ros_control/DefaultRobotHWSim</robotSimType-->
+      <!-- <robotNamespace>/repair</robotNamespace> -->
+      <robotSimType>gazebo_ros_control/DefaultRobotHWSim</robotSimType>
     </plugin>
   </gazebo>

File: repair_urdf/urdf/repair.transmission.xacro (robot description, xacro)
@@ -72,14 +72,24 @@
         </actuator>
     </transmission>
-        <!-- <transmission name="trans_j_torso_1">
-            <type>transmission_interface/SimpleTransmission</type>
-            <joint name="j_torso_1">
-                <hardwareInterface>hardware_interface/PositionJointInterface</hardwareInterface>
-            </joint>
-            <actuator name="j_torso_1_motor">
-                <hardwareInterface>hardware_interface/PositionJointInterface</hardwareInterface>
-                <mechanicalReduction>1</mechanicalReduction>
-            </actuator>
-        </transmission> -->
+    <transmission name="trans_j_torso_1">
+        <type>transmission_interface/SimpleTransmission</type>
+        <joint name="j_torso_1">
+            <hardwareInterface>hardware_interface/PositionJointInterface</hardwareInterface>
+        </joint>
+        <actuator name="j_torso_1_motor">
+            <hardwareInterface>hardware_interface/PositionJointInterface</hardwareInterface>
+            <mechanicalReduction>1</mechanicalReduction>
+        </actuator>
+    </transmission>
+    <transmission name="trans_j_torso_base">
+        <type>transmission_interface/SimpleTransmission</type>
+        <joint name="j_torso_base">
+            <hardwareInterface>hardware_interface/PositionJointInterface</hardwareInterface>
+        </joint>
+        <actuator name="j_torso_base_motor">
+            <hardwareInterface>hardware_interface/PositionJointInterface</hardwareInterface>
+            <mechanicalReduction>1</mechanicalReduction>
+        </actuator>
+    </transmission>
   </xacro:macro>
 </robot>

File: repair_urdf/urdf/repair_cage_macro.urdf.xacro (robot description, xacro)
@@ -2,23 +2,4 @@
 <robot xmlns:xacro="http://ros.org/wiki/xacro">
   <xacro:macro name="repair_cage" params="parent">
-  <link name="sand_bed_b1_link">
-    <visual>
-      <origin xyz="${Table_x} ${Table_y} ${Table_z+table_height+table_top_thickness/2}" />
-      <geometry>
-        <box size="2.0 0.035  0.035" />
-      </geometry>
-      <material name="wood" />
-    </visual>
-    <collision>
-      <origin xyz="${Table_x} ${Table_y} ${Table_z+table_height+table_top_thickness/2}" />
-      <geometry>
-        <box size="2.0 0.035  0.035" />
-      </geometry>
-    </collision>
-  </link>
-  <joint name="sand_bed_b1_joint" type="fixed" >
-    <parent link="table_top_link" />
-    <child link="sand_bed_b1_link" />
-  </joint>
   <link name="table_top_link">
     <visual>
@@ -36,4 +17,7 @@
     </collision>
   </link>
+  <gazebo reference="table_top_link">
+    <material>Gazebo/Wood</material>
+  </gazebo>
   <joint name="table_top_link_joint" type="fixed" >
     <parent link="${parent}" />
@@ -160,4 +144,97 @@
     </collision>
   </link>
+  <!-- Adding wood boundary for Sand -->
+  <!-- small 1 -->
+  <link name="sand_bed_b1_link">
+    <visual>
+      <origin xyz="${Table_x} ${Table_y-Cage_y/2} ${Table_z+table_height+table_top_thickness/2}" />
+      <geometry>
+        <box size="${Cage_x} 0.035  0.035"/>
+      </geometry>
+      <material name="wood" />
+    </visual>
+    <collision>
+      <origin xyz="${Table_x} ${Table_y-Cage_y/2} ${Table_z+table_height+table_top_thickness/2}" />
+      <geometry>
+        <box size="${Cage_x} 0.035  0.035" />
+      </geometry>
+    </collision>
+  </link>
+  <gazebo reference="sand_bed_b1_link">
+    <material>Gazebo/Wood</material>
+  </gazebo>
+  <joint name="sand_bed_b1_joint" type="fixed" >
+    <parent link="table_top_link" />
+    <child link="sand_bed_b1_link" />
+  </joint>
+  <!-- small 2 -->
+  <link name="sand_bed_b2_link">
+    <visual>
+      <origin xyz="${Table_x} ${Table_y+Cage_y/2} ${Table_z+table_height+table_top_thickness/2}" />
+      <geometry>
+        <box size="${Cage_x} 0.035  0.035"/>
+      </geometry>
+      <material name="wood" />
+    </visual>
+    <collision>
+      <origin xyz="${Table_x} ${Table_y-Cage_y/2} ${Table_z+table_height+table_top_thickness/2}" />
+      <geometry>
+        <box size="${Cage_x} 0.035  0.035" />
+      </geometry>
+    </collision>
+  </link>
+  <gazebo reference="sand_bed_b2_link">
+    <material>Gazebo/Wood</material>
+  </gazebo>
+  <joint name="sand_bed_b2_joint" type="fixed" >
+    <parent link="table_top_link" />
+    <child link="sand_bed_b2_link" />
+  </joint>
+  <!-- long 1 -->
+  <link name="sand_bed_b3_link">
+    <visual>
+      <origin xyz="${Table_x+Cage_x/2} ${Table_y} ${Table_z+table_height+table_top_thickness/2}" />
+      <geometry>
+        <box size="0.035 ${Cage_y} 0.035"/>
+      </geometry>
+      <material name="wood" />
+    </visual>
+    <collision>
+      <origin xyz="${Table_x-Cage_x/2} ${Table_y} ${Table_z+table_height+table_top_thickness/2}" />
+      <geometry>
+        <box size="0.035 ${Cage_y} 0.035" />
+      </geometry>
+    </collision>
+  </link>
+  <gazebo reference="sand_bed_b3_link">
+    <material>Gazebo/Wood</material>
+  </gazebo>
+  <joint name="sand_bed_b3_joint" type="fixed" >
+    <parent link="table_top_link" />
+    <child link="sand_bed_b3_link" />
+  </joint>
+  <!-- long 2 -->
+  <link name="sand_bed_b4_link">
+    <visual>
+      <origin xyz="${Table_x-Cage_x/2} ${Table_y} ${Table_z+table_height+table_top_thickness/2}" />
+      <geometry>
+        <box size="0.035 ${Cage_y} 0.035"/>
+      </geometry>
+      <material name="wood" />
+    </visual>
+    <collision>
+      <origin xyz="${Table_x-Cage_x/2} ${Table_y} ${Table_z+table_height+table_top_thickness/2}" />
+      <geometry>
+        <box size="0.035 ${Cage_y} 0.035" />
+      </geometry>
+    </collision>
+  </link>
+  <gazebo reference="sand_bed_b4_link">
+    <material>Gazebo/Wood</material>
+  </gazebo>
+  <joint name="sand_bed_b4_joint" type="fixed" >
+    <parent link="table_top_link" />
+    <child link="sand_bed_b4_link" />
+  </joint>
   <joint name="leg4_joint" type="fixed" >
     <parent link="table_top_link" />

File: repair_urdf/urdf/repair_full.urdf (robot description, URDF)
Before this commit: robot repair_full, 128 links, 128 joints
Links:
- link dummy_prismatic_link: mass None -> 0.1
Joints:
- removed joint j_sliding_guide
- joint j_arm_1_7: origin xyz=0.0 -0.062877 0.05 rpy=1.570796326795 0.03316123 0.0 -> xyz=0.0 -0.062877 0.05 rpy=1.570796326795 0.0 0.0
- joint j_arm_2_7: origin xyz=0.0 0.062877 0.05 rpy=-1.570796326795 0.03316123 0.0 -> xyz=0.0 0.062877 0.05 rpy=-1.570796326795 0.0 0.0
- joint j_torso_1: axis (none) -> 0 0 1; type fixed -> revolute
- joint j_torso_base: limit lower=-0.8 upper=0.8 effort=147 velocity=0.35 -> lower=-0.8 upper=0.8 effort=147.0 velocity=0.25; origin xyz=0.0 0.0 0.07 rpy=0.0 0.0 0.0 -> xyz=0.0 0.0 0.0 rpy=0.0 0.0 0.0; type fixed -> prismatic

File: repair_urdf/urdf/repair_full.urdf.xacro (robot description, xacro)
@@ -28,6 +28,8 @@
         <origin xyz="0.0857 0.0000476009 -0.273184" rpy="0.0009783 1.1836725 0" />
     </xacro:sensor_d435> -->
-    <xacro:sensor_l515 parent='torso_1' use_nominal_extrinsics='true'>
-        <!-- <origin xyz="0.0857 0.0000476009 -0.273184" rpy="0.0009783 1.1836725 0" /> -->
+    <!-- <xacro:sensor_l515 parent='torso_1' use_nominal_extrinsics='true'>
+        <origin xyz="0.0857 0.0000476009 -0.273184" rpy="0.0009783 1.1836725 0" />
+    </xacro:sensor_l515> -->
+    <xacro:sensor_l515 name="camera" topics_ns="camera" parent="torso_1" use_nominal_extrinsics="true" publish_pointcloud="true" add_plug="false" use_mesh="true">
         <origin xyz="0.0857 0.0000476009 -0.273184" rpy="0.0009783 1.1836725 0" />
     </xacro:sensor_l515>
@@ -139,5 +141,5 @@
         <selfCollide>0</selfCollide>
     </gazebo>
-    <!-- <xacro:repair_hand_transmission id="left" />
-    <xacro:repair_hand_transmission id="right" /> -->
+    <!-- <xacro:repair_hand_transmission id="left" /> -->
+    <!-- <xacro:repair_hand_transmission id="right" /> -->
 </robot>

File: repair_urdf/urdf/repair_torso_macro.urdf_old.xacro (robot description, xacro)
@@ -10,14 +10,14 @@
         </joint>-->
         <!-- <link name="dummy_prismatic_link"/> -->
-        <link name="dummy_prismatic_link">
+        <!-- <link name="dummy_prismatic_link">
             <inertial>
-                <origin xyz="0.0 0.0 0.0" rpy="0 0 0"/>
-                <mass value="0.1"/>
+                <origin xyz="0 0 0" rpy="0 0 0"/>
+                <mass value="0.001"/>
                 <inertia
-                ixx="0.0" ixy="0.0" ixz="0.0"
-                iyy="0.0" iyz="0.0"
-                izz="0.0"/>
+                ixx="1e-6" ixy="0.0" ixz="0.0"
+                iyy="1e-6" iyz="0.0"
+                izz="1e-6"/>
             </inertial>
-        </link>
+        </link> -->
         <link name="torso_1">
             <inertial>
@@ -40,15 +40,13 @@
         </link>
         <!-- <joint name="j_torso_base" type="prismatic"> -->
-        <!-- <limit effort="147.0" lower="-0.8" upper="0.8" velocity="0.25"/> -->
-        <joint name="j_torso_base" type="prismatic">
-        <origin rpy="0.0 0.0 0.0" xyz="0.0 0.0 0.0"/>
+        <!-- <joint name="j_torso_base" type="fixed">
+        <origin rpy="0.0 0.0 0.0" xyz="0.0 0.0 0.07"/>
         <parent link="${parent}"/>
                 <child link="dummy_prismatic_link"/>
                 <axis xyz="0 0 1"/>
-        <limit effort="147.0" lower="-0.8" upper="0.8" velocity="0.25"/>
-        </joint>
+        <limit effort="147" lower="-0.8" upper="0.8" velocity="0.25"/>
+        </joint> -->
         <!-- torso -->
-        <!-- revolute -->
-        <joint name="j_torso_1" type="revolute">
+        <!-- <joint name="j_torso_1" type="revolute">
             <parent link="dummy_prismatic_link"/>
             <child link="torso_1"/>
@@ -56,6 +54,6 @@
             <origin rpy="1.570796326795 0.0 1.570796326795" xyz="0.0 0.0 0.0"/>
             <limit effort="147.0" lower="-2.6" upper="2.6" velocity="2.0"/>
-        </joint>
-        <!-- <joint name="j_torso_1" type="revolute">
+        </joint> -->
+        <joint name="j_torso_1" type="revolute">
             <parent link="${parent}"/>
             <child link="torso_1"/>
@@ -64,5 +62,5 @@
             <limit lower="${j_torso_lower[0]}" upper="${j_torso_upper[0]}"
             effort="${j_torso_torque[0]}" velocity="${j_torso_velocity[0]}" />
-        </joint> -->
+        </joint>
     </xacro:macro>
 </robot>

Commit message: latest working code

File: repair_moveit_config_v3/config/gazebo_repair_full.urdf (robot description, URDF)
Before this commit: robot repair_full, 128 links, 127 joints
Joints:
- joint j_torso_base: origin xyz=0.0 0.0 0.0 rpy=0.0 0.0 0.0 -> xyz=0.0 0.0 0.07 rpy=0.0 0.0 0.0
- joint left_hand_v1_wide_grasp_joint: origin xyz=0.03 -0.10 0.15 rpy=0 0 0 -> xyz=0.05 -0.06 0.12 rpy=0 0 0
- joint right_hand_v1_2_research_grasp_joint: origin xyz=-0.06 0.03 0.16 rpy=0 0 1.57 -> xyz=0.0 0.03 0.12 rpy=0 0 1.57

File: repair_urdf/urdf/repair_full.urdf (robot description, URDF)
Before this commit: robot repair_full, 128 links, 127 joints
Joints:
- joint left_hand_v1_wide_grasp_joint: origin xyz=0.05 0 0.12 rpy=0 0 0 -> xyz=0.05 -0.06 0.12 rpy=0 0 0

File: repair_urdf/urdf/repair_torso_macro.urdf.xacro (robot description, xacro)
@@ -42,9 +42,9 @@
         <!-- <limit effort="147.0" lower="-0.8" upper="0.8" velocity="0.25"/> -->
         <joint name="j_torso_base" type="prismatic">
-        <origin rpy="0.0 0.0 0.0" xyz="0.0 0.0 0.0"/>
+        <origin rpy="0.0 0.0 0.0" xyz="0.0 0.0 0.07"/>
         <parent link="${parent}"/>
                 <child link="dummy_prismatic_link"/>
                 <axis xyz="0 0 1"/>
-        <limit effort="147.0" lower="-0.8" upper="0.8" velocity="0.25"/>
+        <limit effort="147.0" lower="-0.75" upper="0.75" velocity="0.25"/>
         </joint>
         <!-- torso -->
